File: power/power.sch (KiCad schematic (older format))
At the start: 14 parts, among them P1 CONN_2, U1 KPS-5, U2 RB-0515S, U3 RB-0515S, U4 RB-0512D, U5 RB-0505D

Commit message: [power] drill files
Parts:
- gave numbers to parts that had none: 1
Changed lines of the file:
@@
 	6700 3400 6700 3700
 $Comp
-L CONN_5X2 P?
+L CONN_5X2 P2
 U 1 1 52E7B775
 P 8000 3900
-F 0 "P?" H 8000 4200 60  0000 C CNN
+F 0 "P2" H 8000 4200 60  0000 C CNN
 F 1 "CONN_5X2" V 8000 3900 50  0000 C CNN
 F 2 "~" H 8000 3900 60  0000 C CNN
