File: test-op/test-op.sch (KiCad schematic (older format))
At the start: 0 parts

Commit message: [test-op] sch
Parts:
- added C1, C2: 1u, ~, symbol C
- added P1, P2, P3, P4, P5: SMA, symbol SMA
- added P6: CONN_5X2, ~, symbol CONN_5X2
- added R1: 1k, ~, symbol R
- added R2: 100, ~, symbol R
- added R3: 100k, ~, symbol R
- added RV1: 100k, ~, symbol POT
- added RV2: 10k, ~, symbol POT
- added U1: HOLD, ~, symbol DG467
- added U2: INT, ~, symbol OPA827
- added U3: RST1, ~, symbol DG468
- added U4: VG, ~, symbol LMH6505
- added U5: RST2, ~, symbol DG468
Connections:
- new net: RV2.2, U4.2 (Vin), U5.1 (NO)
- new net: R2.2, U4.3 (Rg)
- new net: C2.1, R1.1, U4.6 (Vout)
- new net: R1.2, U4.7 (I-)
- new net: C2.2, RV1.2, RV1.3, U2.2 (-In), U3.1 (NO)
- new net: R3.1, RV2.1
- new net: RV1.1, U1.6 (COM)
- new net +15V: P6.1, U1.5 (V+), U2.7 (V+), U3.5 (V+), U5.5 (V+)
- new net +6V: P6.9, U4.8 (V+)
- new net -15V: P6.2, U1.2 (V-), U2.4 (V-), U3.2 (V-), U5.2 (V-)
- new net -6V: P6.7, U4.5 (V-)
- new net GND: C1.2, P1.2 (GND1), P1.3 (GND2), P1.4 (GND3), P1.5 (GND4), P2.2 (GND1), P2.3 (GND2), P2.4 (GND3), P2.5 (GND4), P3.2 (GND1), P3.3 (GND2), P3.4 (GND3), P3.5 (GND4), P4.2 (GND1), P4.3 (GND2), P4.4 (GND3), P4.5 (GND4), P5.2 (GND1), P5.3 (GND2), P5.4 (GND3), P5.5 (GND4), P6.10, R2.1, RV2.3, U1.4 (GND), U2.3 (+In), U3.4 (GND), U4.4 (GND), U5.4 (GND), U5.6 (COM)
- new net HOLD: P2.1 (V), U1.3 (IN)
- new net In: P1.1 (V), U1.1 (NC)
- new net OUT: P4.1 (V), R3.2, U2.6 (Out), U3.6 (COM)
- new net RST: P3.1 (V), U3.3 (IN), U5.3 (IN)
- new net VG: C1.1, P5.1 (V), U4.1 (Vg)
- no-connect marks 0 -> 5

Commit message: [test-op] routing
Parts:
- added C10, C11, C13, C14, C15, C16, C17, C18, C19, C20, C3, C4, C5, C6, C7, C8, C9: 1u, ~, symbol C
- added C12, C21: 0.1u, ~, symbol C
- added P7: IN2, symbol SMA
- added P8: VG2, symbol SMA
- added P9: OUT2, symbol SMA
- added R4, R7: 10k, ~, symbol R
- added R5: 100, ~, symbol R
- added R6: 1k, ~, symbol R
- added RV3, RV4: 10k, ~, symbol POT
- added U6: VG2, ~, symbol LMH6505
- P1: value SMA -> IN
- P2: value SMA -> HOLD
- P3: value SMA -> RST
- P4: value SMA -> OUT
- P5: value SMA -> VG
Connections:
- net +15V: now also C3.1, C5.1, C7.1, C9.1
- net +6V: now also C13.1, C15.1, C17.1, C19.1, RV3.1, RV4.3, U6.8 (V+)
- net -15V: now also C10.2, C4.2, C6.2, C8.2
- net -6V: now also C14.2, C16.2, C18.2, C20.2, RV3.3, RV4.1, U6.5 (V-)
- net GND: now also C10.1, C11.2, C12.2, C13.2, C14.1, C15.2, C16.1, C17.2, C18.1, C19.2, C20.1, C21.2, C3.2, C4.1, C5.2, C6.1, C7.2, C8.1, C9.2, P7.2 (GND1), P7.3 (GND2), P7.4 (GND3), P7.5 (GND4), P8.2 (GND1), P8.3 (GND2), P8.4 (GND3), P8.5 (GND4), P9.2 (GND1), P9.3 (GND2), P9.4 (GND3), P9.5 (GND4), R5.2, U6.4 (GND)
- new net: C12.1, R4.2, RV3.2
- new net: R4.1, R5.1, U6.3 (Rg)
- new net: R6.1, R7.1, U6.7 (I-)
- new net: C21.1, R7.2, RV4.2
- new net IN2: P7.1 (V), U6.2 (Vin)
- new net OUT2: P9.1 (V), R6.2, U6.6 (Vout)
- new net VG2: C11.1, P8.1 (V), U6.1 (Vg)
