File: test-op/test-op.kicad_pcb (KiCad board)
At the start: 2 copper layers, 0 parts

Commit message: [test-op] routing
Parts:
- added C1: 1u, C1206C, F.Cu at (161.4, 101.7)
- added C10: 1u, C1206C, F.Cu at (171.6, 110.4)
- added C11: 1u, C1206C, F.Cu at (137.8, 107.6)
- added C12: 0.1u, C1206C, F.Cu at (141.6, 104.8)
- added C13: 1u, C1206C, F.Cu at (122.0, 104.0)
- added C14: 1u, C1206C, F.Cu at (125.9, 93.6)
- added C15: 1u, C1206C, F.Cu at (149.5, 108.8)
- added C16: 1u, C1206C, F.Cu at (149.2, 97.7)
- added C17: 1u, C1206C, F.Cu at (133.2, 106.3)
- added C18: 1u, C1206C, F.Cu at (134.2, 98.2)
- added C19: 1u, C1206C, F.Cu at (161.4, 107.3)
- added C2: 1u, C1206C, F.Cu at (161.9, 111.4)
- added C20: 1u, C1206C, F.Cu at (153.5, 107.3)
- added C21: 0.1u, C1206C, F.Cu at (126.1, 105.0)
- added C3: 1u, C1206C, F.Cu at (175.6, 110.1)
- added C4: 1u, C1206C, F.Cu at (183.0, 111.1)
- added C5: 1u, C1206C, F.Cu at (153.4, 97.2)
- added C6: 1u, C1206C, F.Cu at (160.4, 95.5)
- added C7: 1u, C1206C, F.Cu at (170.3, 99.4)
- added C8: 1u, C1206C, F.Cu at (173.9, 106.0)
- added C9: 1u, C1206C, F.Cu at (165.2, 103.5)
- added P1: IN, 1814832, F.Cu at (180.2, 118.2)
- added P2: HOLD, 1814832, F.Cu at (180.5, 103.3)
- added P3: RST, 1814832, F.Cu at (163.2, 118.2)
- added P4: OUT, 1814832, F.Cu at (180.5, 90.8)
- added P5: VG, 1814832, F.Cu at (166.5, 90.8)
- added P6: CONN_5X2, VASCH5x2, F.Cu at (113.9, 104.8)
- added P7: IN2, 1814832, F.Cu at (146.7, 118.2)
- added P8: VG2, 1814832, F.Cu at (131.7, 118.2)
- added P9: OUT2, 1814832, F.Cu at (141.6, 90.8)
- added R1: 1k, RMCF0603, F.Cu at (157.6, 110.9)
- added R2: 100, RMCF0603, F.Cu at (156.3, 101.5)
- added R3: 100k, RMCF0603, F.Cu at (168.3, 103.5)
- added R4: 10k, RMCF0603, F.Cu at (141.6, 101.7)
- added R5: 100, RMCF0603, F.Cu at (139.1, 101.0)
- added R6: 1k, RMCF0603, F.Cu at (129.7, 102.2)
- added R7: 10k, RMCF0603, F.Cu at (127.1, 102.7)
- added RV1: 100k, 84WR, F.Cu at (172.1, 116.5)
- added RV2: 10k, 84WR, F.Cu at (165.2, 98.7)
- added RV3: 10k, 84WR, F.Cu at (146.7, 103.3)
- added RV4: 10k, 84WR, F.Cu at (125.1, 99.4)
- added U1: HOLD, TSOP-6, F.Cu at (178.9, 111.6)
- added U2: INT, so-8, F.Cu at (167.5, 108.6)
- added U3: RST1, TSOP-6, F.Cu at (171.8, 102.7)
- added U4: VG, so-8, F.Cu at (157.6, 106.0)
- added U5: RST2, TSOP-6, F.Cu at (157.1, 98.7)
- added U6: VG2, so-8, F.Cu at (134.5, 102.2)
Routing:
- net +15V: track 0.00 -> 166.0 mm
- net -15V: track 0.00 -> 129.3 mm, vias 0 -> 5
- net GND: track 0.00 -> 123.0 mm, vias 0 -> 3
- net -6V: track 0.00 -> 107.0 mm, vias 0 -> 2
- net +6V: track 0.00 -> 80.6 mm, vias 0 -> 2
- net RST: track 0.00 -> 68.2 mm
- net N-0000024: track 0.00 -> 23.3 mm
- net OUT: track 0.00 -> 22.5 mm
- net OUT2: track 0.00 -> 20.3 mm
- net IN2: track 0.00 -> 20.1 mm
- net VG2: track 0.00 -> 17.1 mm
- net VG: track 0.00 -> 16.4 mm
- net N-0000021: track 0.00 -> 8.71 mm
- net HOLD: track 0.00 -> 7.54 mm
- net N-0000015: track 0.00 -> 6.76 mm
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- added copper zone on B.Cu, net GND
- added copper zone on F.Cu, net GND
Other:
- board outline added: 79.5 x 38.9 mm

Commit message: [test-op] ground
Routing:
- net GND: track 123.0 -> 168.2 mm, vias 3 -> 7
Changed lines of the file:
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@@
     (links 128)
     (no_connects 0)
-    (area 110.224999 98.38055 146.315001 177.125)
+    (area 107.137999 84.785999 186.740001 123.748001)
     (thickness 1.6)
     (drawings 5)
-    (tracks 412)
+    (tracks 428)
     (zones 0)
     (modules 47)
@@
   (segment (start 139.4234 98.1817) (end 137.4792 96.2375) (width 0.254) (layer F.Cu) (net 4))
   (segment (start 149.225 98.1817) (end 139.4234 98.1817) (width 0.254) (layer F.Cu) (net 4))
+  (segment (start 142.3035 108.2675) (end 142.3035 108.3035) (width 0.254) (layer F.Cu) (net 5))
+  (segment (start 158.697 115.697) (end 160.655 115.697) (width 0.254) (layer F.Cu) (net 5) (status 800000))
+  (segment (start 158 115) (end 158.697 115.697) (width 0.254) (layer F.Cu) (net 5))
+  (via (at 158 115) (size 0.889) (layers F.Cu B.Cu) (net 5))
+  (segment (start 156 117) (end 158 115) (width 0.254) (layer B.Cu) (net 5))
+  (via (at 156 117) (size 0.889) (layers F.Cu B.Cu) (net 5))
+  (segment (start 152 113) (end 156 117) (width 0.254) (layer F.Cu) (net 5))
+  (segment (start 147 113) (end 152 113) (width 0.254) (layer F.Cu) (net 5))
+  (segment (start 142.3035 108.3035) (end 147 113) (width 0.254) (layer F.Cu) (net 5))
+  (segment (start 144.145 93.345) (end 148.655 93.345) (width 0.254) (layer F.Cu) (net 5) (status 400000))
+  (segment (start 154.265 88.265) (end 163.957 88.265) (width 0.254) (layer F.Cu) (net 5) (status 800000))
+  (segment (start 154 88) (end 154.265 88.265) (width 0.254) (layer F.Cu) (net 5))
+  (via (at 154 88) (size 0.889) (layers F.Cu B.Cu) (net 5))
+  (segment (start 151 91) (end 154 88) (width 0.254) (layer B.Cu) (net 5))
+  (via (at 151 91) (size 0.889) (layers F.Cu B.Cu) (net 5))
+  (segment (start 148.655 93.345) (end 151 91) (width 0.254) (layer F.Cu) (net 5))
   (segment (start 139.065 100.315) (end 143.400676 100.315) (width 0.254) (layer F.Cu) (net 5))
   (segment (start 146.558 104.013) (end 142.3035 108.2675) (width 0.254) (layer F.Cu) (net 5))
