File: test-op2-tweak/test-op2-tweak.kicad_pcb (KiCad board)
At the start: 2 copper layers, 98.4 x 57.8 mm, 114 parts, among them P1 CONN_13X2, P2 CONN_5X2

Commit message: [test-op2-tweak] tweak
Routing:
- net GND: track 562.8 -> 564.6 mm
- net Off4_3: track 30.8 -> 29.6 mm
- net Ctrl2_3: track 46.6 -> 45.6 mm

Commit message: [test-op2-tweak] tweak
Parts:
- P2: footprint VASCH5x2 -> VASCH5x2-2
Routing:
- net GND: track 564.6 -> 798.2 mm, vias 11 -> 39
- net +5V: track 416.3 -> 414.9 mm
