File: pid/pid.kicad_pcb (KiCad board)
At the start: 2 copper layers, 0 parts

Commit message: [pid] more capacitors, layout
Parts:
- added C1: 10u, SM1206, F.Cu at (91.9, 243.6)
- added C10: 10u, SM1206, F.Cu at (73.8, 245.4)
- added C100: 10u, SM1206, F.Cu at (25.4, 104.1)
- added C101: 10u, SM1206, F.Cu at (82.5, 96.5)
- added C102: 10u, SM1206, F.Cu at (68.6, 96.5)
- added C103: 10u, SM1206, F.Cu at (111.8, 108.0)
- added C104: 10u, SM1206, F.Cu at (118.1, 108.0)
- added C105: 0.01u, SM1206, F.Cu at (125.7, 104.1)
- added C106: 0.01u, SM1206, F.Cu at (96.5, 108.0)
- added C107: 10u, SM1206, F.Cu at (82.5, 108.0)
- added C108: 10u, SM1206, F.Cu at (76.2, 108.0)
- added C109: 10p, SM1206, F.Cu at (40.6, 104.1)
- added C11: 10u, SM1206, F.Cu at (106.4, 238.8)
- added C110: 10u, SM1206, F.Cu at (125.7, 100.3)
- added C111: 10u, SM1206, F.Cu at (111.8, 100.3)
- added C112: 10u, SM1206, F.Cu at (82.5, 100.3)
- added C113: 10p, SM1206, F.Cu at (90.2, 108.0)
- added C114: 10u, SM1206, F.Cu at (61.0, 108.0)
- added C115: 10u, SM1206, F.Cu at (54.6, 108.0)
- added C116: 10u, SM1206, F.Cu at (47.0, 108.0)
- added C117: 10u, SM1206, F.Cu at (40.6, 108.0)
- added C118: 10u, SM1206, F.Cu at (68.6, 100.3)
- added C119: 10u, SM1206, F.Cu at (125.7, 96.5)
- added C12: 10u, SM1206, F.Cu at (101.0, 238.8)
- added C120: 10u, SM1206, F.Cu at (118.1, 96.5)
- added C121: 10u, SM1206, F.Cu at (111.8, 96.5)
- added C122: 10u, SM1206, F.Cu at (104.1, 96.5)
- added C123: 10u, SM1206, F.Cu at (96.5, 96.5)
- added C124: 10u, SM1206, F.Cu at (132.1, 96.5)
- added C125: 10u, SM1206, F.Cu at (139.7, 96.5)
- added C126: 10u, SM1206, F.Cu at (25.4, 100.3)
- added C127: 10u, SM1206, F.Cu at (33.0, 100.3)
- added C128: 10u, SM1206, F.Cu at (40.6, 100.3)
- added C129: 10u, SM1206, F.Cu at (47.0, 100.3)
- added C13: 10u, SM1206, F.Cu at (101.0, 231.1)
- added C130: 10u, SM1206, F.Cu at (90.2, 96.5)
- added C131: 10u, SM1206, F.Cu at (61.0, 100.3)
- added C132: 10u, SM1206, F.Cu at (3.56, 4.32)
- added C133: 10u, SM1206, F.Cu at (-2.41, 5.84)
- added C134: 10u, SM1206, F.Cu at (2.92, -3.68)
- added C135: 10u, SM1206, F.Cu at (6.73, 0.89)
- added C136: 10u, SM1206, F.Cu at (158.4, 156.6)
- added C137: 10u, SM1206, F.Cu at (159.9, 150.5)
- added C138: 10u, SM1206, F.Cu at (-2.79, -3.43)
- added C139: 10u, SM1206, F.Cu at (-2.03, -0.13)
- added C14: 10u, SM1206, F.Cu at (101.0, 241.4)
- added C15: 10u, SM1206, F.Cu at (106.4, 231.0)
- added C16: 10u, SM1206, F.Cu at (33.0, 108.0)
- added C17: 10u, SM1206, F.Cu at (61.0, 88.9)
- added C18: 10u, SM1206, F.Cu at (54.6, 88.9)
- added C19: 0.01u, SM1206, F.Cu at (33.0, 104.1)
- added C2: 10u, SM1206, F.Cu at (91.9, 251.5)
- added C20: 0.01u, SM1206, F.Cu at (139.7, 108.0)
- added C21: 10u, SM1206, F.Cu at (61.0, 96.5)
- added C22: 10u, SM1206, F.Cu at (40.6, 88.9)
- added C23: 10u, SM1206, F.Cu at (25.4, 111.8)
- added C24: 10u, SM1206, F.Cu at (47.0, 88.9)
- added C25: 1u, SM1206, F.Cu at (111.8, 92.7)
- added C26: 1p, SM1206, F.Cu at (96.5, 92.7)
- added C27: 1p, SM1206, F.Cu at (90.2, 92.7)
- added C28: 0.1u, SM1206, F.Cu at (132.1, 100.3)
- added C29: 10u, SM1206, F.Cu at (118.1, 92.7)
- added C3: 0.1u, SM1206, F.Cu at (85.0, 245.2)
- added C30: 0.01u, SM1206, F.Cu at (132.1, 92.7)
- added C31: 10u, SM1206, F.Cu at (132.1, 88.9)
- added C32: 10u, SM1206, F.Cu at (47.0, 96.5)
- added C33: 10u, SM1206, F.Cu at (54.6, 96.5)
- added C34: 10u, SM1206, F.Cu at (90.2, 88.9)
- added C35: 10u, SM1206, F.Cu at (118.1, 88.9)
- added C36: 10u, SM1206, F.Cu at (40.6, 92.7)
- added C37: 10u, SM1206, F.Cu at (139.7, 88.9)
- added C38: 10u, SM1206, F.Cu at (25.4, 92.7)
- added C39: 10u, SM1206, F.Cu at (76.2, 88.9)
- added C4: 1u, SM1206, F.Cu at (89.0, 241.0)
- added C40: 10u, SM1206, F.Cu at (47.0, 104.1)
- added C41: 10u, SM1206, F.Cu at (54.6, 104.1)
- added C42: 10u, SM1206, F.Cu at (118.1, 85.1)
- added C43: 10u, SM1206, F.Cu at (68.6, 104.1)
- added C44: 10u, SM1206, F.Cu at (76.2, 104.1)
- added C45: 10u, SM1206, F.Cu at (104.1, 104.1)
- added C46: 10u, SM1206, F.Cu at (124.5, 76.2)
- added C47: 10u, SM1206, F.Cu at (130.8, 76.2)
- added C48: 0.01u, SM1206, F.Cu at (110.5, 76.2)
- added C49: 0.01u, SM1206, F.Cu at (61.0, 85.1)
- added C5: 1p, SM1206, F.Cu at (87.6, 245.2)
- added C50: 10u, SM1206, F.Cu at (102.9, 76.2)
- added C51: 10u, SM1206, F.Cu at (88.9, 76.2)
- added C52: 10u, SM1206, F.Cu at (37.5, 203.3)
- added C53: 10u, SM1206, F.Cu at (37.5, 210.9)
- added C54: 10u, SM1206, F.Cu at (111.8, 192.9)
- added C55: 10u, SM1206, F.Cu at (111.8, 200.5)
- added C56: 1p, SM1206, F.Cu at (107.7, 191.4)
- added C57: 10u, SM1206, F.Cu at (97.9, 187.5)
- added C58: 10u, SM1206, F.Cu at (102.0, 188.8)
- added C59: 10u, SM1206, F.Cu at (102.0, 196.5)
- added C6: 10u, SM1206, F.Cu at (75.2, 236.0)
- added C60: 10u, SM1206, F.Cu at (102.0, 186.2)
- added C61: 10u, SM1206, F.Cu at (96.5, 196.8)
- added C62: 10u, SM1206, F.Cu at (129.0, 187.8)
- added C63: 10u, SM1206, F.Cu at (123.6, 187.8)
- added C64: 10u, SM1206, F.Cu at (123.6, 180.2)
- added C65: 10u, SM1206, F.Cu at (123.6, 190.5)
- added C66: 10u, SM1206, F.Cu at (129.0, 180.1)
- added C67: 10u, SM1206, F.Cu at (164.0, 148.8)
- added C68: 10u, SM1206, F.Cu at (159.9, 147.8)
- added C69: 10u, SM1206, F.Cu at (82.5, 85.1)
- added C7: 10u, SM1206, F.Cu at (79.2, 237.4)
- added C70: 0.01u, SM1206, F.Cu at (163.8, 156.6)
- added C71: 0.01u, SM1206, F.Cu at (111.8, 85.1)
- added C72: 10u, SM1206, F.Cu at (57.5, 207.1)
- added C73: 10u, SM1206, F.Cu at (52.7, 214.8)
- added C74: 10u, SM1206, F.Cu at (53.7, 199.5)
- added C75: 10u, SM1206, F.Cu at (52.2, 207.1)
- added C76: 10p, SM1206, F.Cu at (50.2, 197.9)
- added C77: 100p, SM1206, F.Cu at (50.2, 219.1)
- added C78: 10u, SM1206, F.Cu at (96.5, 104.1)
- added C79: 10u, SM1206, F.Cu at (90.2, 104.1)
- added C8: 10u, SM1206, F.Cu at (79.2, 245.0)
- added C80: 10u, SM1206, F.Cu at (25.4, 88.9)
- added C81: 10u, SM1206, F.Cu at (139.7, 85.1)
- added C82: 10u, SM1206, F.Cu at (125.7, 85.1)
- added C83: 10u, SM1206, F.Cu at (61.0, 104.1)
- added C84: 10p, SM1206, F.Cu at (47.0, 92.7)
- added C85: 10u, SM1206, F.Cu at (33.0, 92.7)
- added C86: 10u, SM1206, F.Cu at (82.5, 88.9)
- added C87: 10u, SM1206, F.Cu at (111.8, 88.9)
- added C88: 10u, SM1206, F.Cu at (104.1, 88.9)
- added C89: 10u, SM1206, F.Cu at (139.7, 92.7)
- added C9: 10u, SM1206, F.Cu at (85.0, 239.8)
- added C90: 10u, SM1206, F.Cu at (68.6, 85.1)
- added C91: 1p, SM1206, F.Cu at (95.2, 76.2)
- added C92: 10u, SM1206, F.Cu at (76.2, 92.7)
- added C93: 10u, SM1206, F.Cu at (33.0, 96.5)
- added C94: 10u, SM1206, F.Cu at (25.4, 96.5)
- added C95: 10u, SM1206, F.Cu at (104.1, 92.7)
- added C96: 10u, SM1206, F.Cu at (139.7, 100.3)
- added C97: 10u, SM1206, F.Cu at (33.0, 111.8)
- added C98: 10u, SM1206, F.Cu at (40.6, 111.8)
- added C99: 10u, SM1206, F.Cu at (47.0, 111.8)
- added D1: DIODE, sc70, F.Cu at (64.8, 111.8)
- added D2: DIODE, sc70, F.Cu at (61.0, 111.8)
- added P1: CONN_13X2, VASCH13x2, F.Cu at (43.2, 25.4)
- added P2: SMA, 1814832, F.Cu at (23.7, 217.3)
- added P3: SMA, 1814832, F.Cu at (23.7, 204.1)
- added P4: SMA, 1814832, F.Cu at (87.6, 24.1)
- added P5: SMA, 1814832, F.Cu at (78.7, 24.1)
- added P6: SMA, 1814832, F.Cu at (68.6, 24.1)
- added R1: 200, SM0603, F.Cu at (24.1, 128.3)
- added R10: 100, SM0603, F.Cu at (82.8, 244.0)
- added R100: 100, SM0603, F.Cu at (110.5, 190.6)
- added R101: 200, SM0603, F.Cu at (117.5, 196.6)
- added R102: 10k, SM0603, F.Cu at (94.6, 194.2)
- added R103: 5k, SM0603, F.Cu at (95.8, 188.3)
- added R104: 100, SM0603, F.Cu at (96.4, 194.2)
- added R105: 1k, SM0603, F.Cu at (105.5, 192.7)
- added R106: 10k, SM0603, F.Cu at (105.5, 190.0)
- added R107: 100k, SM0603, F.Cu at (110.2, 180.8)
- added R108: 100k, SM0603, F.Cu at (105.7, 179.3)
- added R109: 2k, SM0603, F.Cu at (112.5, 181.6)
- added R11: 10, SM0603, F.Cu at (92.7, 240.9)
- added R110: 2k, SM0603, F.Cu at (114.6, 185.9)
- added R111: 100k, SM0603, F.Cu at (103.4, 205.6)
- added R112: 100k, SM0603, F.Cu at (104.9, 201.3)
- added R113: 2k, SM0603, F.Cu at (100.7, 206.5)
- added R114: 2k, SM0603, F.Cu at (96.0, 207.8)
- added R115: 10k, SM0603, F.Cu at (130.9, 182.8)
- added R116: 5k, SM0603, F.Cu at (125.0, 177.9)
- added R117: 100, SM0603, F.Cu at (129.2, 182.8)
- added R118: 1k, SM0603, F.Cu at (120.0, 184.0)
- added R119: 10k, SM0603, F.Cu at (120.0, 186.8)
- added R12: 100, SM0603, F.Cu at (93.7, 238.0)
- added R120: 100k, SM0603, F.Cu at (116.8, 173.5)
- added R121: 100k, SM0603, F.Cu at (115.3, 177.9)
- added R122: 2k, SM0603, F.Cu at (117.5, 170.6)
- added R123: 2k, SM0603, F.Cu at (121.9, 169.0)
- added R124: 100k, SM0603, F.Cu at (135.6, 173.1)
- added R125: 100k, SM0603, F.Cu at (130.8, 171.6)
- added R126: 2k, SM0603, F.Cu at (138.2, 173.5)
- added R127: 2k, SM0603, F.Cu at (139.7, 177.9)
- added R128: 100k, SM0603, F.Cu at (64.8, 120.7)
- added R129: 2k, SM0603, F.Cu at (156.2, 150.5)
- added R13: 200, SM0603, F.Cu at (97.5, 247.5)
- added R130: 2k, SM0603, F.Cu at (97.8, 118.1)
- added R131: 2k, SM0603, F.Cu at (86.4, 118.1)
- added R132: 2k, SM0603, F.Cu at (40.6, 120.7)
- added R133: 2k, SM0603, F.Cu at (94.0, 118.1)
- added R134: 20k, SM0603, F.Cu at (163.2, 153.2)
- added R135: 20k, SM0603, F.Cu at (77.5, 118.1)
- added R136: 20k, SM0603, F.Cu at (165.4, 152.7)
- added R137: 20k, SM0603, F.Cu at (53.3, 120.7)
- added R138: 1k, SM0603, F.Cu at (41.5, 206.4)
- added R139: 510, SM0603, F.Cu at (49.1, 202.1)
- added R14: 10k, SM0603, F.Cu at (72.0, 242.7)
- added R140: 510, SM0603, F.Cu at (54.1, 197.2)
- added R141: 100, SM0603, F.Cu at (51.6, 216.9)
- added R142: 510, SM0603, F.Cu at (54.4, 216.9)
- added R143: 51, SM0603, F.Cu at (58.8, 211.7)
- added R144: 200k, SM0603, F.Cu at (134.6, 118.1)
- added R145: 5k, SM0603, F.Cu at (27.9, 120.7)
- added R146: 510, SM0603, F.Cu at (134.6, 110.5)
- added R147: 200k, SM0603, F.Cu at (24.1, 115.6)
- added R148: 5k, SM0603, F.Cu at (127.0, 118.1)
- added R149: 510, SM0603, F.Cu at (138.4, 110.5)
- added R15: 5k, SM0603, F.Cu at (73.0, 238.3)
- added R150: 100, SM0603, F.Cu at (123.2, 123.2)
- added R151: 100, SM0603, F.Cu at (114.3, 123.2)
- added R152: 200, SM0603, F.Cu at (110.5, 123.2)
- added R153: 10k, SM0603, F.Cu at (90.2, 123.2)
- added R154: 5k, SM0603, F.Cu at (69.8, 118.1)
- added R155: 100, SM0603, F.Cu at (81.3, 123.2)
- added R156: 1k, SM0603, F.Cu at (130.8, 115.6)
- added R157: 10k, SM0603, F.Cu at (64.8, 118.1)
- added R158: 100k, SM0603, F.Cu at (44.5, 120.7)
- added R159: 100k, SM0603, F.Cu at (57.1, 120.7)
- added R16: 100, SM0603, F.Cu at (73.7, 242.7)
- added R160: 2k, SM0603, F.Cu at (77.5, 120.7)
- added R161: 2k, SM0603, F.Cu at (101.6, 118.1)
- added R162: 100k, SM0603, F.Cu at (73.7, 120.7)
- added R163: 100k, SM0603, F.Cu at (69.8, 120.7)
- added R164: 2k, SM0603, F.Cu at (40.6, 118.1)
- added R165: 2k, SM0603, F.Cu at (27.9, 118.1)
- added R166: 10k, SM0603, F.Cu at (57.1, 118.1)
- added R167: 5k, SM0603, F.Cu at (106.7, 123.2)
- added R168: 100, SM0603, F.Cu at (118.1, 110.5)
- added R169: 1k, SM0603, F.Cu at (73.7, 123.2)
- added R17: 1k, SM0603, F.Cu at (82.8, 241.2)
- added R170: 10k, SM0603, F.Cu at (77.5, 123.2)
- added R171: 100k, SM0603, F.Cu at (139.7, 123.2)
- added R172: 100k, SM0603, F.Cu at (33.0, 120.7)
- added R173: 2k, SM0603, F.Cu at (134.6, 123.2)
- added R174: 2k, SM0603, F.Cu at (64.8, 123.2)
- added R175: 100k, SM0603, F.Cu at (69.8, 123.2)
- added R176: 100k, SM0603, F.Cu at (125.7, 110.5)
- added R177: 2k, SM0603, F.Cu at (130.8, 110.5)
- added R178: 2k, SM0603, F.Cu at (105.4, 110.5)
- added R179: 100k, SM0603, F.Cu at (142.2, 110.5)
- added R18: 10k, SM0603, F.Cu at (82.8, 238.4)
- added R180: 2k, SM0603, F.Cu at (27.9, 115.6)
- added R181: 2k, SM0603, F.Cu at (123.2, 118.1)
- added R182: 2k, SM0603, F.Cu at (130.8, 118.1)
- added R183: 2k, SM0603, F.Cu at (114.3, 118.1)
- added R184: 2k, SM0603, F.Cu at (118.1, 118.1)
- added R185: 20k, SM0603, F.Cu at (139.7, 118.1)
- added R186: 20k, SM0603, F.Cu at (106.7, 118.1)
- added R187: 20k, SM0603, F.Cu at (24.1, 120.7)
- added R188: 20k, SM0603, F.Cu at (36.8, 120.7)
- added R189: 510, SM0603, F.Cu at (94.0, 123.2)
- added R19: 100k, SM0603, F.Cu at (87.6, 230.9)
- added R190: 510, SM0603, F.Cu at (86.4, 123.2)
- added R191: 2k, SM0603, F.Cu at (101.6, 123.2)
- added R192: 1k, SM0603, F.Cu at (90.2, 118.1)
- added R193: 1k, SM0603, F.Cu at (48.3, 120.7)
- added R2: 200, SM0603, F.Cu at (95.8, 192.0)
- added R20: 100k, SM0603, F.Cu at (82.9, 229.4)
- added R21: 2k, SM0603, F.Cu at (90.3, 231.5)
- added R22: 2k, SM0603, F.Cu at (91.8, 236.0)
- added R23: 100k, SM0603, F.Cu at (65.2, 250.1)
- added R24: 100k, SM0603, F.Cu at (70.1, 252.2)
- added R25: 2k, SM0603, F.Cu at (62.4, 250.1)
- added R26: 2k, SM0603, F.Cu at (61.2, 245.9)
- added R27: 10k, SM0603, F.Cu at (108.3, 233.7)
- added R28: 5k, SM0603, F.Cu at (102.4, 228.9)
- added R29: 100, SM0603, F.Cu at (106.6, 233.7)
- added R3: 200, SM0603, F.Cu at (73.2, 240.5)
- added R30: 1k, SM0603, F.Cu at (97.4, 234.9)
- added R31: 10k, SM0603, F.Cu at (97.4, 237.7)
- added R32: 100k, SM0603, F.Cu at (94.2, 224.4)
- added R33: 100k, SM0603, F.Cu at (92.7, 228.9)
- added R34: 2k, SM0603, F.Cu at (94.9, 221.5)
- added R35: 2k, SM0603, F.Cu at (99.3, 220.0)
- added R36: 100k, SM0603, F.Cu at (113.0, 224.0)
- added R37: 100k, SM0603, F.Cu at (108.2, 222.5)
- added R38: 2k, SM0603, F.Cu at (115.6, 224.4)
- added R39: 2k, SM0603, F.Cu at (117.1, 228.9)
- added R4: 200, SM0603, F.Cu at (73.7, 115.6)
- added R40: 100k, SM0603, F.Cu at (69.8, 128.3)
- added R41: 2k, SM0603, F.Cu at (73.7, 128.3)
- added R42: 2k, SM0603, F.Cu at (106.7, 128.3)
- added R43: 2k, SM0603, F.Cu at (110.5, 128.3)
- added R44: 2k, SM0603, F.Cu at (118.1, 123.2)
- added R45: 2k, SM0603, F.Cu at (97.8, 128.3)
- added R46: 20k, SM0603, F.Cu at (114.3, 128.3)
- added R47: 20k, SM0603, F.Cu at (90.2, 128.3)
- added R48: 20k, SM0603, F.Cu at (123.2, 128.3)
- added R49: 20k, SM0603, F.Cu at (81.3, 128.3)
- added R5: 2k, SM0603, F.Cu at (123.2, 125.7)
- added R50: 100, SM0603, F.Cu at (127.0, 128.3)
- added R51: 10, SM0603, F.Cu at (123.2, 120.7)
- added R52: 200k, SM0603, F.Cu at (36.8, 125.7)
- added R53: 10, SM0603, F.Cu at (57.1, 125.7)
- added R54: 0, SM0603, F.Cu at (40.6, 125.7)
- added R55: 100, SM0603, F.Cu at (27.9, 125.7)
- added R56: 510, SM0603, F.Cu at (53.3, 125.7)
- added R57: 1M, SM0603, F.Cu at (90.2, 120.7)
- added R58: 200, SM0603, F.Cu at (130.8, 128.3)
- added R59: 510, SM0603, F.Cu at (86.4, 120.7)
- added R6: 2k, SM0603, F.Cu at (48.3, 115.6)
- added R60: 10k, SM0603, F.Cu at (94.0, 120.7)
- added R61: 5k, SM0603, F.Cu at (110.5, 120.7)
- added R62: 100, SM0603, F.Cu at (97.8, 120.7)
- added R63: 1k, SM0603, F.Cu at (101.6, 120.7)
- added R64: 10k, SM0603, F.Cu at (106.7, 120.7)
- added R65: 100k, SM0603, F.Cu at (24.1, 125.7)
- added R66: 100k, SM0603, F.Cu at (130.8, 120.7)
- added R67: 2k, SM0603, F.Cu at (118.1, 120.7)
- added R68: 2k, SM0603, F.Cu at (114.3, 120.7)
- added R69: 100k, SM0603, F.Cu at (33.0, 123.2)
- added R7: 2k, SM0603, F.Cu at (44.5, 115.6)
- added R70: 100k, SM0603, F.Cu at (36.8, 123.2)
- added R71: 2k, SM0603, F.Cu at (27.9, 123.2)
- added R72: 2k, SM0603, F.Cu at (24.1, 123.2)
- added R73: 10k, SM0603, F.Cu at (40.6, 123.2)
- added R74: 5k, SM0603, F.Cu at (53.3, 123.2)
- added R75: 100, SM0603, F.Cu at (44.5, 123.2)
- added R76: 1k, SM0603, F.Cu at (48.3, 123.2)
- added R77: 10k, SM0603, F.Cu at (94.0, 128.3)
- added R78: 100k, SM0603, F.Cu at (134.6, 125.7)
- added R79: 100k, SM0603, F.Cu at (94.0, 115.6)
- added R8: 2k, SM0603, F.Cu at (27.9, 128.3)
- added R80: 2k, SM0603, F.Cu at (90.2, 115.6)
- added R81: 2k, SM0603, F.Cu at (61.0, 123.2)
- added R82: 100k, SM0603, F.Cu at (110.5, 115.6)
- added R83: 100k, SM0603, F.Cu at (114.3, 115.6)
- added R84: 2k, SM0603, F.Cu at (106.7, 115.6)
- added R85: 2k, SM0603, F.Cu at (101.6, 115.6)
- added R86: 100k, SM0603, F.Cu at (118.1, 115.6)
- added R87: 2k, SM0603, F.Cu at (123.2, 115.6)
- added R88: 2k, SM0603, F.Cu at (97.8, 110.5)
- added R89: 2k, SM0603, F.Cu at (92.7, 110.5)
- added R9: 20, SM0603, F.Cu at (118.1, 125.7)
- added R90: 2k, SM0603, F.Cu at (114.3, 110.5)
- added R91: 2k, SM0603, F.Cu at (72.4, 110.5)
- added R92: 20k, SM0603, F.Cu at (88.9, 110.5)
- added R93: 20k, SM0603, F.Cu at (68.6, 110.5)
- added R94: 20k, SM0603, F.Cu at (81.3, 110.5)
- added R95: 20k, SM0603, F.Cu at (109.2, 110.5)
- added R96: 16.67k, sot23, F.Cu at (29.8, 205.1)
- added R97: 16.67k, sot23, F.Cu at (29.8, 210.4)
- added R98: 200, SM0603, F.Cu at (31.9, 207.1)
- added R99: 100, SM0603, F.Cu at (106.3, 194.9)
- added RV1: 200, 84WR, F.Cu at (100.8, 247.5)
- added RV10: 20k, 84WR, F.Cu at (111.8, 62.2)
- added RV11: 20k, 84WR, F.Cu at (83.8, 34.3)
- added RV12: 200k, 84WR, F.Cu at (102.9, 62.2)
- added RV13: 200k, 84WR, F.Cu at (45.7, 43.2)
- added RV14: 100k, 84WR, F.Cu at (120.7, 62.2)
- added RV15: 200, 84WR, F.Cu at (92.7, 62.2)
- added RV16: 100k, 84WR, F.Cu at (45.7, 62.2)
- added RV17: 10k, 84WR, F.Cu at (54.6, 62.2)
- added RV18: 100k, 84WR, F.Cu at (111.8, 34.3)
- added RV19: 10k, 84WR, F.Cu at (26.7, 62.2)
- added RV2: 100k, 84WR, F.Cu at (82.9, 232.5)
- added RV20: 100k, 84WR, F.Cu at (54.6, 52.1)
- added RV21: 10k, 84WR, F.Cu at (139.7, 52.1)
- added RV22: 100k, 84WR, F.Cu at (73.7, 52.1)
- added RV23: 10k, 84WR, F.Cu at (64.8, 52.1)
- added RV24: 20k, 84WR, F.Cu at (102.9, 52.1)
- added RV25: 20k, 84WR, F.Cu at (92.7, 52.1)
- added RV26: 200k, 84WR, F.Cu at (111.8, 52.1)
- added RV27: 200k, 84WR, F.Cu at (83.8, 52.1)
- added RV28: 200, 84WR, F.Cu at (120.9, 196.6)
- added RV29: 100k, 84WR, F.Cu at (105.7, 182.5)
- added RV3: 10k, 84WR, F.Cu at (88.6, 236.0)
- added RV30: 10k, 84WR, F.Cu at (111.4, 185.9)
- added RV31: 100k, 84WR, F.Cu at (101.7, 201.3)
- added RV32: 10k, 84WR, F.Cu at (96.0, 204.6)
- added RV33: 100k, 84WR, F.Cu at (118.5, 177.9)
- added RV34: 10k, 84WR, F.Cu at (121.9, 172.2)
- added RV35: 100k, 84WR, F.Cu at (130.8, 174.8)
- added RV36: 10k, 84WR, F.Cu at (136.5, 177.9)
- added RV37: 20k, 84WR, F.Cu at (45.7, 52.1)
- added RV38: 20k, 84WR, F.Cu at (45.7, 34.3)
- added RV39: 200k, 84WR, F.Cu at (169.2, 154.4)
- added RV4: 100k, 84WR, F.Cu at (70.1, 249.0)
- added RV40: 200k, 84WR, F.Cu at (36.8, 34.3)
- added RV41: 200, 84WR, F.Cu at (45.3, 206.9)
- added RV42: 200, 84WR, F.Cu at (36.8, 62.2)
- added RV43: 100k, 84WR, F.Cu at (64.8, 62.2)
- added RV44: 10k, 84WR, F.Cu at (130.8, 43.2)
- added RV45: 100k, 84WR, F.Cu at (83.8, 62.2)
- added RV46: 10k, 84WR, F.Cu at (73.7, 62.2)
- added RV47: 100k, 84WR, F.Cu at (130.8, 52.1)
- added RV48: 10k, 84WR, F.Cu at (54.6, 43.2)
- added RV49: 100k, 84WR, F.Cu at (26.7, 43.2)
- added RV5: 10k, 84WR, F.Cu at (64.4, 245.7)
- added RV50: 10k, 84WR, F.Cu at (36.8, 43.2)
- added RV51: 20k, 84WR, F.Cu at (83.8, 43.2)
- added RV52: 20k, 84WR, F.Cu at (120.7, 34.3)
- added RV53: 200k, 84WR, F.Cu at (64.8, 43.2)
- added RV54: 200k, 84WR, F.Cu at (73.7, 34.3)
- added RV6: 100k, 84WR, F.Cu at (95.9, 228.9)
- added RV7: 10k, 84WR, F.Cu at (99.3, 223.1)
- added RV8: 100k, 84WR, F.Cu at (108.2, 225.7)
- added RV9: 10k, 84WR, F.Cu at (113.9, 228.9)
- added U1: LM7171, so-8, F.Cu at (93.0, 247.5)
- added U10: DG468, TSOP-6, F.Cu at (78.7, 77.5)
- added U11: MAX44251, MSOP_8, F.Cu at (64.8, 77.5)
- added U12: DG468, TSOP-6, F.Cu at (73.7, 77.5)
- added U13: AD8421, so-8, F.Cu at (36.4, 207.1)
- added U14: LM7171, so-8, F.Cu at (112.9, 196.7)
- added U15: LMH6505, so-8, F.Cu at (101.0, 192.7)
- added U16: LMH6505, so-8, F.Cu at (124.6, 184.0)
- added U17: MAX44251, MSOP_8, F.Cu at (159.1, 153.5)
- added U18: LM7171, so-8, F.Cu at (53.7, 203.3)
- added U19: LM7171, so-8, F.Cu at (53.7, 210.9)
- added U2: LMH6505, so-8, F.Cu at (78.2, 241.2)
- added U20: DG469, so-8, F.Cu at (96.5, 69.8)
- added U21: DG469, so-8, F.Cu at (102.9, 69.8)
- added U22: DG469, so-8, F.Cu at (110.5, 69.8)
- added U23: LM7171, so-8, F.Cu at (116.8, 69.8)
- added U24: DG469, so-8, F.Cu at (129.5, 69.8)
- added U25: LM7171, so-8, F.Cu at (142.2, 61.0)
- added U26: LMH6505, so-8, F.Cu at (129.5, 61.0)
- added U27: LMH6505, so-8, F.Cu at (83.8, 69.8)
- added U28: MAX44251, MSOP_8, F.Cu at (59.7, 77.5)
- added U29: DG469, so-8, F.Cu at (31.8, 69.8)
- added U3: LMH6505, so-8, F.Cu at (102.0, 234.9)
- added U30: LM7171, so-8, F.Cu at (38.1, 69.8)
- added U31: LM7171, so-8, F.Cu at (25.4, 78.7)
- added U32: DG469, so-8, F.Cu at (135.9, 69.8)
- added U33: DG469, so-8, F.Cu at (38.1, 78.7)
- added U34: DG468, TSOP-6, F.Cu at (68.6, 77.5)
- added U4: MAX44251, MSOP_8, F.Cu at (54.6, 77.5)
- added U5: LM7171, so-8, F.Cu at (77.5, 69.8)
- added U6: LM7171, so-8, F.Cu at (71.1, 69.8)
- added U7: LMH6505, so-8, F.Cu at (52.1, 69.8)
- added U8: LMH6505, so-8, F.Cu at (123.2, 69.8)
- added U9: DG467, TSOP-6, F.Cu at (82.5, 77.5)
Routing:
- net GND: track 0.00 -> 100.6 mm
- net +5V: track 0.00 -> 48.1 mm
- net /Comp_P/Off4: track 0.00 -> 24.0 mm
- net /Comp_D/Off4: track 0.00 -> 24.0 mm
- net -5V: track 0.00 -> 19.7 mm
- net /Comp_P/VarAmp2/In: track 0.00 -> 15.5 mm
- net /Comp_P/VarAmp2/Out: track 0.00 -> 15.3 mm
- net /Comp_D/VarAmp2/In: track 0.00 -> 14.2 mm
- net N-0000060: track 0.00 -> 12.0 mm
- net /Comp_P/Off1: track 0.00 -> 11.8 mm
- net N-00000139: track 0.00 -> 11.7 mm
- net N-00000119: track 0.00 -> 11.7 mm
- net N-0000096: track 0.00 -> 11.4 mm
- net N-0000094: track 0.00 -> 11.4 mm
- net N-0000095: track 0.00 -> 11.0 mm
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
Commit message: [pid] layout
Parts:
- C102, C103, C104, C105, C106, C124, C125, C126, C127, C128, C129, C130, C131, C132, C133, C134, C135, C136, C137, C138, C139, C16, C17, C18, C19, C20, C45, C46, C47, C48, C49, C67, C68, C69, C70, C71, R128, R129, R130, R131, R132, R133, R134, R135, R136, R137, R179, R180, R181, R182, R183, R184, R185, R186, R187, R188, R40, R41, R42, R43, R44, R45, R46, R47, R48, R49, R86, R87, R88, R89, R90, R91, R92, R93, R94, R95, RV10, RV11, RV12, RV13, RV24, RV25, RV26, RV27, RV37, RV38, RV39, RV40, RV51, RV52, RV53, RV54, U11, U17, U28, U4: moved to B.Cu
- moved C135 182.8 mm to (138.6, 127.5), turned to 180 degrees
- moved C134 182.1 mm to (135.3, 121.3)
- moved C133 181.6 mm to (149.0, 106.1), turned to 180 degrees
- moved C132 171.3 mm to (145.7, 99.9)
- moved U31 166.1 mm to (190.3, 99.0), turned to 180 degrees
- moved C80 162.9 mm to (174.3, 154.9)
- moved C1 154.7 mm to (159.8, 104.6)
- moved C10 154.7 mm to (141.7, 106.4)
- moved C15 154.7 mm to (174.3, 92.0)
- moved C2 154.7 mm to (159.8, 112.5)
- moved C6 154.7 mm to (143.1, 97.0)
- moved C8 154.7 mm to (147.1, 106.0)
- moved C9 154.7 mm to (152.8, 100.8)
- moved R10 154.7 mm to (150.7, 105.0)
- moved R11 154.7 mm to (160.6, 101.9)
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Connections:
- C27 pad 1: /Comp_I/Reset1/NO -> /Comp_I/Reset1/COM
- C28 pad 2: /Comp_I/Reset1/NO -> /Comp_I/Reset1/COM
- C30 pad 2: /Comp_I/Reset1/COM -> /Comp_I/Reset1/NO
- R51 pad 2: /Comp_I/Reset1/NO -> /Comp_I/Reset1/COM
- R52 pad 2: /Comp_I/Reset1/NO -> /Comp_I/Reset1/COM
- R54 pad 1: /Comp_I/Reset1/NO -> /Comp_I/Reset1/COM
- R57 pad 1: /Comp_I/Reset1/COM -> /Comp_I/Reset1/NO
- U10 pad 1: /Comp_I/Reset1/COM -> /Comp_I/Reset1/NO
- U5 pad 3: /Comp_I/Reset1/NO -> /Comp_I/Reset1/COM
Routing:
- net GND: track 100.6 -> 1568.9 mm, vias 0 -> 84
- net -5V: track 19.7 -> 827.3 mm, vias 0 -> 28
- net +5V: track 48.1 -> 795.9 mm, vias 0 -> 37
- net -15V: track 1.96 -> 437.4 mm, vias 0 -> 17
- net +15V: track 1.96 -> 426.6 mm, vias 0 -> 14
- net /ScaleOutput/Inv: track 0.00 -> 147.8 mm, vias 0 -> 2
- net /P_Switch/IN: track 0.00 -> 138.1 mm, vias 0 -> 1
- net /ScaleOutput/Limit_H: track 0.00 -> 130.3 mm, vias 0 -> 1
- net /ScaleOutput/Offset: track 0.00 -> 123.4 mm, vias 0 -> 1
- net /Comp_P/Ctrl: track 0.00 -> 112.2 mm, vias 0 -> 1
- net /Comp_D/Ctrl: track 0.00 -> 111.6 mm, vias 0 -> 1
- net /ScaleOutput/Limit_L: track 0.00 -> 110.4 mm, vias 0 -> 1
- net /FF_Switch/IN: track 0.00 -> 93.8 mm, vias 0 -> 2
- net /ScaleOutput/In: track 0.00 -> 91.5 mm
- net /Comp_FF/Ctrl: track 0.00 -> 91.3 mm, vias 0 -> 1
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- added copper zone on B.Cu, net GND
- added copper zone on F.Cu, net GND
- added copper zone on Inner1.Cu, net GND
- added copper zone on Inner2.Cu, net GND
Other:
- board outline added: 108.5 x 107.7 mm
- copper layers 2 -> 4
- net class Default: via_dia 0.889 -> 0.7874; via_drill 0.635 -> 0.4064
- rule via_min_drill: 0.508 -> 0.4064
- rule via_min_size: 0.889 -> 0.7874
