File: pid/pid.kicad_pcb (KiCad board)
At the start: 4 copper layers, 108.5 x 107.7 mm, 428 parts, among them P1 CONN_13X2, P2 SMA, P3 SMA, P4 SMA, P5 SMA, P6 SMA, U1 LM7171, U10 DG468, U11 MAX44251, U12 DG468, U13 AD8421, U14 LM7171, U15 LMH6505, U16 LMH6505, U17 MAX44251, U18 LM7171, U19 LM7171, U2 LMH6505, U20 DG469, U21 DG469, U22 DG469, U23 LM7171, U24 DG469, U25 LM7171, U26 LMH6505, U27 LMH6505, U28 MAX44251, U29 DG469, U3 LMH6505, U30 LM7171, U31 LM7171, U32 DG469, U33 DG469, U34 DG468, U4 MAX44251, U5 LM7171, U6 LM7171, U7 LMH6505, U8 LMH6505, U9 DG467

Commit message: [pid] show values on board
Parts:
- C1, C10, C100, C101, C102, C103, C104, C105, C106, C107, C108, C109, C11, C110, C111, C112, C113, C114, C115, C116, C117, C118, C119, C12, C120, C121, C122, C123, C124, C125, C126, C127, C128, C129, C13, C130, C131, C132, C133, C134, C135, C136, C137, C138, C139, C14, C15, C16, C17, C18, C19, C2, C20, C21, C22, C23, C24, C25, C26, C27, C28, C29, C3, C30, C31, C32, C33, C34, C35, C36, C37, C38, C39, C4, C40, C41, C42, C43, C44, C45, C46, C47, C48, C49, C5, C50, C51, C52, C53, C54, C55, C56, C57, C58, C59, C6, C60, C61, C62, C63, C64, C65, C66, C67, C68, C69, C7, C70, C71, C72, C73, C74, C75, C76, C77, C78, C79, C8, C80, C81, C82, C83, C84, C85, C86, C87, C88, C89, C9, C90, C91, C92, C93, C94, C95, C96, C97, C98, C99: footprint SM1206 -> SM1206_V
- R1, R10, R100, R101, R102, R103, R104, R105, R106, R107, R108, R109, R11, R110, R111, R112, R113, R114, R115, R116, R117, R118, R119, R12, R120, R121, R122, R123, R124, R125, R126, R127, R128, R129, R13, R130, R131, R132, R133, R134, R135, R136, R137, R138, R139, R14, R140, R141, R142, R143, R144, R145, R146, R147, R148, R149, R15, R150, R151, R152, R153, R154, R155, R156, R157, R158, R159, R16, R160, R161, R162, R163, R164, R165, R166, R167, R168, R169, R17, R170, R171, R172, R173, R174, R175, R176, R177, R178, R179, R18, R180, R181, R182, R183, R184, R185, R186, R187, R188, R189, R19, R190, R191, R192, R193, R2, R20, R21, R22, R23, R24, R25, R26, R27, R28, R29, R3, R30, R31, R32, R33, R34, R35, R36, R37, R38, R39, R4, R40, R41, R42, R43, R44, R45, R46, R47, R48, R49, R5, R50, R51, R52, R53, R54, R55, R56, R57, R58, R59, R6, R60, R61, R62, R63, R64, R65, R66, R67, R68, R69, R7, R70, R71, R72, R73, R74, R75, R76, R77, R78, R79, R8, R80, R81, R82, R83, R84, R85, R86, R87, R88, R89, R9, R90, R91, R92, R93, R94, R95, R98, R99: footprint SM0603 -> SM0603_V
