File: pid/pid.sch (KiCad schematic (older format))
At the start: 0 parts

Commit message: [pid] comp amps
Parts:
- added P1: In1, symbol SMA
- added P10: Out2, symbol SMA
- added P11: Out3, symbol SMA
- added P12: Out4, symbol SMA
- added P13: CONN_13X2, ~, symbol CONN_13X2
- added P14: CONN_5X2, ~, symbol CONN_5X2
- added P2: In2, symbol SMA
- added P3: In3, symbol SMA
- added P4: In4, symbol SMA
- added P9: Out1, symbol SMA
Connections:
- net labels added: +15V, +5V, -15V, -5V, GND, In1, In2, In3, In4, Out1, Out2, Out3, Out4
- net labels removed: Measure, Setpoint
- wire segments 0 -> 26

Commit message: [pid] -
Parts:
- removed P1: In1, symbol SMA
- removed P10: Out2, symbol SMA
- removed P11: Out3, symbol SMA
- removed P12: Out4, symbol SMA
- removed P2: In2, symbol SMA
- removed P3: In3, symbol SMA
- removed P4: In4, symbol SMA
- removed P9: Out1, symbol SMA
- added R1, R2, R3, R?: 200, ~, symbol R
- added R4, R5, R6, R?: 2k, ~, symbol R
- renumbered P13 to P1, P14 to P2
Connections:
- net labels added: D_Ctrl, D_On, FF_Ctrl, FF_On, FF_Select, FeedForward, Hold, I_Ctrl, I_On, Measure, Monitor, P_Ctrl, P_On, Reset, SetPoint
- net labels removed: In1, In2, In3, In4, Out1, Out2, Out3, Out4
- wire segments 26 -> 73
- no-connect marks 0 -> 2

Commit message: [pid] -
Parts:
- removed P2: CONN_5X2, ~, symbol CONN_5X2
- added R9: 20, ~, symbol R
- gave numbers to parts that had none: 2
- renumbered R1 to R2, R2 to R3, R3 to R4, R4 to R6, R5 to R7, R6 to R8
Connections:
- net labels added: I_Off1, I_Off2, Invert, Limit_H, Limit_L, Out, Out_Offset, Out_On
- wire segments 73 -> 126
- no-connect marks 2 -> 0
Other:
- moved on the sheet: P1, R1, R2, R3, R4, R5, R6, R7, R8

Commit message: [pid] net list
Parts:
- added C124, C125, C126, C127, C128, C129, C130, C131: 10u, ~, symbol C
Connections:
- net +15V: now also C126.1, C130.1
- net +5V: now also C124.1, C128.1
- net -15V: now also C127.2, C131.2
- net -5V: now also C125.2, C129.2
- net GND: now also C124.2, C125.1, C126.2, C127.1, C128.2, C129.1, C130.2, C131.1
Changed lines of the file:
@@
 Wire Wire Line
 	7150 2450 7300 2450
+Text GLabel 2900 1100 2    60   Input ~ 0
++5V
+Text GLabel 2900 2100 2    60   Input ~ 0
+-5V
+$Comp
+L C C124
+U 1 1 5363D8B6
+P 2850 1350
+F 0 "C124" H 2850 1450 40  0000 L CNN
+F 1 "10u" H 2856 1265 40  0000 L CNN
+F 2 "~" H 2888 1200 30  0000 C CNN
+F 3 "~" H 2850 1350 60  0000 C CNN
+	1    2850 1350
+	1    0    0    -1
+$EndComp
+$Comp
+L C C125
+U 1 1 5363D8BC
+P 2850 1850
+F 0 "C125" H 2850 1950 40  0000 L CNN
+F 1 "10u" H 2856 1765 40  0000 L CNN
+F 2 "~" H 2888 1700 30  0000 C CNN
+F 3 "~" H 2850 1850 60  0000 C CNN
+	1    2850 1850
+	1    0    0    -1
+$EndComp
+$Comp
+L GND #PWR09
+U 1 1 5363D8C2
+P 2950 1650
+F 0 "#PWR09" H 2950 1650 30  0001 C CNN
+F 1 "GND" H 2950 1580 30  0001 C CNN
+F 2 "" H 2950 1650 60  0000 C CNN
+F 3 "" H 2950 1650 60  0000 C CNN
+	1    2950 1650
+	1    0    0    -1
+$EndComp
+Wire Wire Line
+	2900 1100 2850 1100
+Wire Wire Line
+	2850 1100 2850 1150
+Wire Wire Line
+	2850 1550 2850 1650
+Wire Wire Line
+	2850 1600 2950 1600
+Wire Wire Line
+	2950 1600 2950 1650
+Connection ~ 2850 1600
+Wire Wire Line
+	2850 2050 2850 2100
+Wire Wire Line
+	2850 2100 2900 2100
+Text GLabel 3550 1100 2    60   Input ~ 0
++15V
+Text GLabel 3550 2100 2    60   Input ~ 0
+-15V
+$Comp
+L C C126
+U 1 1 5363D8D2
+P 3500 1350
+F 0 "C126" H 3500 1450 40  0000 L CNN
+F 1 "10u" H 3506 1265 40  0000 L CNN
+F 2 "~" H 3538 1200 30  0000 C CNN
+F 3 "~" H 3500 1350 60  0000 C CNN
+	1    3500 1350
+	1    0    0    -1
+$EndComp
+$Comp
+L C C127
+U 1 1 5363D8D8
+P 3500 1850
+F 0 "C127" H 3500 1950 40  0000 L CNN
+F 1 "10u" H 3506 1765 40  0000 L CNN
+F 2 "~" H 3538 1700 30  0000 C CNN
+F 3 "~" H 3500 1850 60  0000 C CNN
+	1    3500 1850
+	1    0    0    -1
+$EndComp
+$Comp
+L GND #PWR010
+U 1 1 5363D8DE
+P 3600 1650
+F 0 "#PWR010" H 3600 1650 30  0001 C CNN
+F 1 "GND" H 3600 1580 30  0001 C CNN
+F 2 "" H 3600 1650 60  0000 C CNN
+F 3 "" H 3600 1650 60  0000 C CNN
+	1    3600 1650
+	1    0    0    -1
+$EndComp
+Wire Wire Line
+	3550 1100 3500 1100
+Wire Wire Line
+	3500 1100 3500 1150
+Wire Wire Line
+	3500 1550 3500 1650
+Wire Wire Line
+	3500 1600 3600 1600
+Wire Wire Line
+	3600 1600 3600 1650
+Connection ~ 3500 1600
+Wire Wire Line
+	3500 2050 3500 2100
+Wire Wire Line
+	3500 2100 3550 2100
+Text GLabel 4250 1100 2    60   Input ~ 0
++5V
+Text GLabel 4250 2100 2    60   Input ~ 0
+-5V
+$Comp
+L C C128
+U 1 1 5363DBA6
+P 4200 1350
+F 0 "C128" H 4200 1450 40  0000 L CNN
+F 1 "10u" H 4206 1265 40  0000 L CNN
+F 2 "~" H 4238 1200 30  0000 C CNN
+F 3 "~" H 4200 1350 60  0000 C CNN
+	1    4200 1350
+	1    0    0    -1
+$EndComp
+$Comp
+L C C129
+U 1 1 5363DBAC
+P 4200 1850
+F 0 "C129" H 4200 1950 40  0000 L CNN
+F 1 "10u" H 4206 1765 40  0000 L CNN
+F 2 "~" H 4238 1700 30  0000 C CNN
+F 3 "~" H 4200 1850 60  0000 C CNN
+	1    4200 1850
+	1    0    0    -1
+$EndComp
+$Comp
+L GND #PWR011
+U 1 1 5363DBB2
+P 4300 1650
+F 0 "#PWR011" H 4300 1650 30  0001 C CNN
+F 1 "GND" H 4300 1580 30  0001 C CNN
+F 2 "" H 4300 1650 60  0000 C CNN
+F 3 "" H 4300 1650 60  0000 C CNN
+	1    4300 1650
+	1    0    0    -1
+$EndComp
+Wire Wire Line
+	4250 1100 4200 1100
+Wire Wire Line
+	4200 1100 4200 1150
+Wire Wire Line
+	4200 1550 4200 1650
+Wire Wire Line
+	4200 1600 4300 1600
+Wire Wire Line
+	4300 1600 4300 1650
+Connection ~ 4200 1600
+Wire Wire Line
+	4200 2050 4200 2100
+Wire Wire Line
+	4200 2100 4250 2100
+Text GLabel 4900 1100 2    60   Input ~ 0
++15V
+Text GLabel 4900 2100 2    60   Input ~ 0
+-15V
+$Comp
+L C C130
+U 1 1 5363DBC2
+P 4850 1350
+F 0 "C130" H 4850 1450 40  0000 L CNN
+F 1 "10u" H 4856 1265 40  0000 L CNN
+F 2 "~" H 4888 1200 30  0000 C CNN
+F 3 "~" H 4850 1350 60  0000 C CNN
+	1    4850 1350
+	1    0    0    -1
+$EndComp
+$Comp
+L C C131
+U 1 1 5363DBC8
+P 4850 1850
+F 0 "C131" H 4850 1950 40  0000 L CNN
+F 1 "10u" H 4856 1765 40  0000 L CNN
+F 2 "~" H 4888 1700 30  0000 C CNN
+F 3 "~" H 4850 1850 60  0000 C CNN
+	1    4850 1850
+	1    0    0    -1
+$EndComp
+$Comp
+L GND #PWR012
+U 1 1 5363DBCE
+P 4950 1650
+F 0 "#PWR012" H 4950 1650 30  0001 C CNN
+F 1 "GND" H 4950 1580 30  0001 C CNN
+F 2 "" H 4950 1650 60  0000 C CNN
+F 3 "" H 4950 1650 60  0000 C CNN
+	1    4950 1650
+	1    0    0    -1
+$EndComp
+Wire Wire Line
+	4900 1100 4850 1100
+Wire Wire Line
+	4850 1100 4850 1150
+Wire Wire Line
+	4850 1550 4850 1650
+Wire Wire Line
+	4850 1600 4950 1600
+Wire Wire Line
+	4950 1600 4950 1650
+Connection ~ 4850 1600
+Wire Wire Line
+	4850 2050 4850 2100
+Wire Wire Line
+	4850 2100 4900 2100
 $EndSCHEMATC
