File: pid/Comp_D.sch (KiCad schematic (older format))
At the start: 11 parts, among them U1 LM7171

Commit message: [pid] -
Parts:
- removed C4: 1p, ~, symbol C
- removed R1, R2: 100, ~, symbol R
- added C5: 1p, ~, symbol C
- added R7, R9: 100, ~, symbol R
- gave numbers to parts that had none: 2
- renumbered R3 to R10
Connections:
- net GND: now also C5.2
- net VarAmp/Out: now also R7.1
- net VarAmp2/Out: now also R9.1
- net at C3.1: now also R7.2
- net at C3.2, R8.2, U1.2 (-In): now also C5.1
- net at C4.2, R8.1: now also R9.2
Changed lines of the file:
@@
 LIBS:rb-0524s
 LIBS:max44251
+LIBS:r_div
 LIBS:pid-cache
 EELAYER 27 0
@@
 $Descr A4 11693 8268
 encoding utf-8
-Sheet 28 27
+Sheet 28 47
 Title ""
-Date "22 apr 2014"
+Date "1 may 2014"
 Rev ""
 Comp ""
@@
 $Sheet
 S 2250 2700 700  500
-U 531E6F48
+U 53598F1D
 F0 "VarAmp" 50
 F1 "VarAmp.sch" 50
@@
 Off2
 $Comp
-L R R1
-U 1 1 531EACE1
+L R R7
+U 1 1 53598F1E
 P 3350 2800
-AR Path="/531E9A87/531EACE1" Ref="R1"  Part="1"
-AR Path="/531FFF34/531EACE1" Ref="R48"  Part="1"
-AR Path="/5355B409/531EACE1" Ref="R1"  Part="1"
-F 0 "R1" V 3430 2800 40  0000 C CNN
+F 0 "R7" V 3430 2800 40  0000 C CNN
 F 1 "100" V 3357 2801 40  0000 C CNN
 F 2 "~" V 3280 2800 30  0000 C CNN
@@
 $Comp
 L LM7171 U1
-U 1 1 531EAD57
+U 1 1 53598F1F
 P 4850 2900
-AR Path="/531E9A87/531EAD57" Ref="U1"  Part="1"
-AR Path="/531FFF34/531EAD57" Ref="U15"  Part="1"
-AR Path="/5355B409/531EAD57" Ref="U1"  Part="1"
 F 0 "U1" H 5150 3100 60  0000 C CNN
 F 1 "LM7171" H 4950 2900 60  0000 C CNN
@@
 $EndComp
 $Comp
-L R R2
-U 1 1 531EAE22
+L R R9
+U 1 1 53598F20
 P 4550 2100
-AR Path="/531E9A87/531EAE22" Ref="R2"  Part="1"
-AR Path="/531FFF34/531EAE22" Ref="R49"  Part="1"
-AR Path="/5355B409/531EAE22" Ref="R2"  Part="1"
-F 0 "R2" V 4630 2100 40  0000 C CNN
+F 0 "R9" V 4630 2100 40  0000 C CNN
 F 1 "100" V 4557 2101 40  0000 C CNN
 F 2 "~" V 4480 2100 30  0000 C CNN
@@
 U 1 1 531EAE28
 P 3950 2800
-AR Path="/531E9A87/531EAE28" Ref="C3"  Part="1"
-AR Path="/531FFF34/531EAE28" Ref="C60"  Part="1"
-AR Path="/5355B409/531EAE28" Ref="C3"  Part="1"
 F 0 "C3" H 3950 2900 40  0000 L CNN
 F 1 "0.1u" H 3956 2715 40  0000 L CNN
@@
 -5V
 $Comp
-L GND #PWR07
+L GND #PWR04
 U 1 1 531EC8D5
 P 4400 3100
-AR Path="/531E9A87/531EC8D5" Ref="#PWR07"  Part="1"
-AR Path="/531FFF34/531EC8D5" Ref="#PWR062"  Part="1"
-AR Path="/5355B409/531EC8D5" Ref="#PWR07"  Part="1"
-F 0 "#PWR07" H 4400 3100 30  0001 C CNN
+F 0 "#PWR04" H 4400 3100 30  0001 C CNN
 F 1 "GND" H 4400 3030 30  0001 C CNN
 F 2 "" H 4400 3100 60  0000 C CNN
@@
 $EndComp
 $Comp
-L R R3
+L R R10
 U 1 1 531ECB0B
 P 5850 2650
-AR Path="/531E9A87/531ECB0B" Ref="R3"  Part="1"
-AR Path="/531FFF34/531ECB0B" Ref="R50"  Part="1"
-AR Path="/5355B409/531ECB0B" Ref="R3"  Part="1"
-F 0 "R3" V 5930 2650 40  0000 C CNN
+F 0 "R10" V 5930 2650 40  0000 C CNN
 F 1 "200" V 5857 2651 40  0000 C CNN
 F 2 "~" V 5780 2650 30  0000 C CNN
@@
 U 1 1 531ECB11
 P 5850 2100
-AR Path="/531E9A87/531ECB11" Ref="RV1"  Part="1"
-AR Path="/531FFF34/531ECB11" Ref="RV4"  Part="1"
-AR Path="/5355B409/531ECB11" Ref="RV1"  Part="1"
 F 0 "RV1" H 5850 2000 50  0000 C CNN
 F 1 "200" H 5850 2100 50  0000 C CNN
@@
 $EndComp
 $Comp
-L GND #PWR08
+L GND #PWR05
 U 1 1 531ED061
 P 6050 1900
-AR Path="/531E9A87/531ED061" Ref="#PWR08"  Part="1"
-AR Path="/531FFF34/531ED061" Ref="#PWR063"  Part="1"
-AR Path="/5355B409/531ED061" Ref="#PWR08"  Part="1"
-F 0 "#PWR08" H 6050 1900 30  0001 C CNN
+F 0 "#PWR05" H 6050 1900 30  0001 C CNN
 F 1 "GND" H 6050 1830 30  0001 C CNN
 F 2 "" H 6050 1900 60  0000 C CNN
@@
 $Comp
 L C C1
-U 1 1 531EE90B
+U 1 1 53598F26
 P 3100 1350
-AR Path="/531E9A87/531EE90B" Ref="C1"  Part="1"
-AR Path="/531FFF34/531EE90B" Ref="C58"  Part="1"
-AR Path="/5355B409/531EE90B" Ref="C1"  Part="1"
 F 0 "C1" H 3100 1450 40  0000 L CNN
 F 1 "10u" H 3106 1265 40  0000 L CNN
@@
 $Comp
 L C C2
-U 1 1 531EE911
+U 1 1 53598F27
 P 3100 1850
-AR Path="/531E9A87/531EE911" Ref="C2"  Part="1"
-AR Path="/531FFF34/531EE911" Ref="C59"  Part="1"
-AR Path="/5355B409/531EE911" Ref="C2"  Part="1"
 F 0 "C2" H 3100 1950 40  0000 L CNN
 F 1 "10u" H 3106 1765 40  0000 L CNN
@@
 $EndComp
 $Comp
-L GND #PWR09
+L GND #PWR06
 U 1 1 531EE917
 P 3200 1650
-AR Path="/531E9A87/531EE917" Ref="#PWR09"  Part="1"
-AR Path="/531FFF34/531EE917" Ref="#PWR064"  Part="1"
-AR Path="/5355B409/531EE917" Ref="#PWR09"  Part="1"
-F 0 "#PWR09" H 3200 1650 30  0001 C CNN
+F 0 "#PWR06" H 3200 1650 30  0001 C CNN
 F 1 "GND" H 3200 1580 30  0001 C CNN
 F 2 "" H 3200 1650 60  0000 C CNN
@@
 $EndComp
 $Comp
-L C C4
-U 1 1 531FE94B
+L C C5
+U 1 1 53598F2D
 P 4300 3250
-AR Path="/531E9A87/531FE94B" Ref="C4"  Part="1"
-AR Path="/531FFF34/531FE94B" Ref="C61"  Part="1"
-AR Path="/5355B409/531FE94B" Ref="C4"  Part="1"
-F 0 "C4" H 4300 3350 40  0000 L CNN
+F 0 "C5" H 4300 3350 40  0000 L CNN
 F 1 "1p" H 4306 3165 40  0000 L CNN
 F 2 "~" H 4338 3100 30  0000 C CNN
@@
 $EndComp
 $Comp
-L GND #PWR010
+L GND #PWR07
 U 1 1 531FE951
 P 4300 3500
-AR Path="/531E9A87/531FE951" Ref="#PWR010"  Part="1"
-AR Path="/531FFF34/531FE951" Ref="#PWR065"  Part="1"
-AR Path="/5355B409/531FE951" Ref="#PWR010"  Part="1"
-F 0 "#PWR010" H 4300 3500 30  0001 C CNN
+F 0 "#PWR07" H 4300 3500 30  0001 C CNN
 F 1 "GND" H 4300 3430 30  0001 C CNN
 F 2 "" H 4300 3500 60  0000 C CNN
@@
 $Sheet
 S 3850 1100 600  200
-U 53555E75
+U 53598F2F
 F0 "CtrlConvert" 50
 F1 "CtrlConvert.sch" 50
@@
 Ctrl1
 $Comp
-L R R?
+L R R8
 U 1 1 5355A894
 P 4300 2450
-F 0 "R?" V 4380 2450 40  0000 C CNN
+F 0 "R8" V 4380 2450 40  0000 C CNN
 F 1 "10" V 4307 2451 40  0000 C CNN
 F 2 "~" V 4230 2450 30  0000 C CNN
@@
 $EndComp
 $Comp
-L C C?
+L C C4
 U 1 1 5355A89A
 P 4000 2100
-F 0 "C?" H 4000 2200 40  0000 L CNN
+F 0 "C4" H 4000 2200 40  0000 L CNN
 F 1 "1u" H 4006 2015 40  0000 L CNN
 F 2 "~" H 4038 1950 30  0000 C CNN
@@
 $EndComp
 $Comp
-L GND #PWR?
+L GND #PWR08
 U 1 1 5355A8A0
 P 3750 2150
-F 0 "#PWR?" H 3750 2150 30  0001 C CNN
+F 0 "#PWR08" H 3750 2150 30  0001 C CNN
 F 1 "GND" H 3750 2080 30  0001 C CNN
 F 2 "" H 3750 2150 60  0000 C CNN

Commit message: [pid] -
Parts:
- renumbered R7 to R10, R8 to R11, R9 to R12, R10 to R13
Changed lines of the file:
@@
 $Descr A4 11693 8268
 encoding utf-8
-Sheet 28 47
+Sheet 2 53
 Title ""
-Date "1 may 2014"
+Date "2 may 2014"
 Rev ""
 Comp ""
@@
 Off2
 $Comp
-L R R7
+L R R10
 U 1 1 53598F1E
 P 3350 2800
-F 0 "R7" V 3430 2800 40  0000 C CNN
+F 0 "R10" V 3430 2800 40  0000 C CNN
 F 1 "100" V 3357 2801 40  0000 C CNN
 F 2 "~" V 3280 2800 30  0000 C CNN
@@
 $EndComp
 $Comp
-L R R9
+L R R12
 U 1 1 53598F20
 P 4550 2100
-F 0 "R9" V 4630 2100 40  0000 C CNN
+F 0 "R12" V 4630 2100 40  0000 C CNN
 F 1 "100" V 4557 2101 40  0000 C CNN
 F 2 "~" V 4480 2100 30  0000 C CNN
@@
 -5V
 $Comp
-L GND #PWR04
+L GND #PWR09
 U 1 1 531EC8D5
 P 4400 3100
-F 0 "#PWR04" H 4400 3100 30  0001 C CNN
+F 0 "#PWR09" H 4400 3100 30  0001 C CNN
 F 1 "GND" H 4400 3030 30  0001 C CNN
 F 2 "" H 4400 3100 60  0000 C CNN
@@
 $EndComp
 $Comp
-L R R10
+L R R13
 U 1 1 531ECB0B
 P 5850 2650
-F 0 "R10" V 5930 2650 40  0000 C CNN
+F 0 "R13" V 5930 2650 40  0000 C CNN
 F 1 "200" V 5857 2651 40  0000 C CNN
 F 2 "~" V 5780 2650 30  0000 C CNN
@@
 $EndComp
 $Comp
-L GND #PWR05
+L GND #PWR010
 U 1 1 531ED061
 P 6050 1900
-F 0 "#PWR05" H 6050 1900 30  0001 C CNN
+F 0 "#PWR010" H 6050 1900 30  0001 C CNN
 F 1 "GND" H 6050 1830 30  0001 C CNN
 F 2 "" H 6050 1900 60  0000 C CNN
@@
 $EndComp
 $Comp
-L GND #PWR06
+L GND #PWR011
 U 1 1 531EE917
 P 3200 1650
-F 0 "#PWR06" H 3200 1650 30  0001 C CNN
+F 0 "#PWR011" H 3200 1650 30  0001 C CNN
 F 1 "GND" H 3200 1580 30  0001 C CNN
 F 2 "" H 3200 1650 60  0000 C CNN
@@
 $EndComp
 $Comp
-L GND #PWR07
+L GND #PWR012
 U 1 1 531FE951
 P 4300 3500
-F 0 "#PWR07" H 4300 3500 30  0001 C CNN
+F 0 "#PWR012" H 4300 3500 30  0001 C CNN
 F 1 "GND" H 4300 3430 30  0001 C CNN
 F 2 "" H 4300 3500 60  0000 C CNN
@@
 Ctrl1
 $Comp
-L R R8
+L R R11
 U 1 1 5355A894
 P 4300 2450
-F 0 "R8" V 4380 2450 40  0000 C CNN
+F 0 "R11" V 4380 2450 40  0000 C CNN
 F 1 "10" V 4307 2451 40  0000 C CNN
 F 2 "~" V 4230 2450 30  0000 C CNN
@@
 $EndComp
 $Comp
-L GND #PWR08
+L GND #PWR013
 U 1 1 5355A8A0
 P 3750 2150
-F 0 "#PWR08" H 3750 2150 30  0001 C CNN
+F 0 "#PWR013" H 3750 2150 30  0001 C CNN
 F 1 "GND" H 3750 2080 30  0001 C CNN
 F 2 "" H 3750 2150 60  0000 C CNN
