File: pid/Comp_P.sch (KiCad schematic (older format))
At the start: 8 parts, among them U1 LM7171

Commit message: [pid] -
Parts:
- removed R3: 200, ~, symbol R
- removed RV1: 200, ~, symbol POT
- added R98: 200, ~, symbol R
- added RV28: 200, ~, symbol POT
- renumbered C1 to C54, C2 to C55, C4 to C56, R1 to R96, R2 to R97, U1 to U14
Connections:
- net GND: now also RV28.3
- net Out: now also R98.1
- net VarAmp2/In: now also RV28.2
- new net: R98.2, RV28.1
Changed lines of the file:
@@
 LIBS:rb-0524s
 LIBS:max44251
+LIBS:r_div
 LIBS:pid-cache
 EELAYER 27 0
@@
 $Descr A4 11693 8268
 encoding utf-8
-Sheet 20 27
+Sheet 23 47
 Title ""
-Date "22 apr 2014"
+Date "1 may 2014"
 Rev ""
 Comp ""
@@
 	3650 3100 3850 3100
 $Comp
-L R R1
+L R R96
 U 1 1 531EACE1
 P 4050 2800
-AR Path="/531E9A87/531EACE1" Ref="R1"  Part="1"
-AR Path="/531FFF34/531EACE1" Ref="R48"  Part="1"
-AR Path="/5355C3A0/531EACE1" Ref="R1"  Part="1"
-F 0 "R1" V 4130 2800 40  0000 C CNN
+F 0 "R96" V 4130 2800 40  0000 C CNN
 F 1 "100" V 4057 2801 40  0000 C CNN
 F 2 "~" V 3980 2800 30  0000 C CNN
@@
 $EndComp
 $Comp
-L LM7171 U1
+L LM7171 U14
 U 1 1 531EAD57
 P 4850 2900
-AR Path="/531E9A87/531EAD57" Ref="U1"  Part="1"
-AR Path="/531FFF34/531EAD57" Ref="U15"  Part="1"
-AR Path="/5355C3A0/531EAD57" Ref="U1"  Part="1"
-F 0 "U1" H 5150 3100 60  0000 C CNN
+F 0 "U14" H 5150 3100 60  0000 C CNN
 F 1 "LM7171" H 4950 2900 60  0000 C CNN
 F 2 "~" H 4850 2900 60  0000 C CNN
@@
 $EndComp
 $Comp
-L R R2
+L R R97
 U 1 1 531EAE22
 P 4450 2350
-AR Path="/531E9A87/531EAE22" Ref="R2"  Part="1"
-AR Path="/531FFF34/531EAE22" Ref="R49"  Part="1"
-AR Path="/5355C3A0/531EAE22" Ref="R2"  Part="1"
-F 0 "R2" V 4530 2350 40  0000 C CNN
+F 0 "R97" V 4530 2350 40  0000 C CNN
 F 1 "100" V 4457 2351 40  0000 C CNN
 F 2 "~" V 4380 2350 30  0000 C CNN
@@
 $Sheet
 S 4850 1700 700  500
-U 531EB865
+U 53598F21
 F0 "VarAmp2" 50
 F1 "VarAmp.sch" 50
@@
 	4950 3350 5000 3350
 $Comp
-L GND #PWR07
-U 1 1 531EC8D5
+L GND #PWR061
+U 1 1 53598F22
 P 4400 3100
-AR Path="/531E9A87/531EC8D5" Ref="#PWR07"  Part="1"
-AR Path="/531FFF34/531EC8D5" Ref="#PWR062"  Part="1"
-AR Path="/5355C3A0/531EC8D5" Ref="#PWR07"  Part="1"
-F 0 "#PWR07" H 4400 3100 30  0001 C CNN
+F 0 "#PWR061" H 4400 3100 30  0001 C CNN
 F 1 "GND" H 4400 3030 30  0001 C CNN
 F 2 "" H 4400 3100 60  0000 C CNN
@@
 	4400 3000 4400 3100
 $Comp
-L R R3
-U 1 1 531ECB0B
+L R R98
+U 1 1 53598F23
 P 5850 2650
-AR Path="/531E9A87/531ECB0B" Ref="R3"  Part="1"
-AR Path="/531FFF34/531ECB0B" Ref="R50"  Part="1"
-AR Path="/5355C3A0/531ECB0B" Ref="R3"  Part="1"
-F 0 "R3" V 5930 2650 40  0000 C CNN
+F 0 "R98" V 5930 2650 40  0000 C CNN
 F 1 "200" V 5857 2651 40  0000 C CNN
 F 2 "~" V 5780 2650 30  0000 C CNN
@@
 $EndComp
 $Comp
-L POT RV1
-U 1 1 531ECB11
+L POT RV28
+U 1 1 53598F24
 P 5850 2100
-AR Path="/531E9A87/531ECB11" Ref="RV1"  Part="1"
-AR Path="/531FFF34/531ECB11" Ref="RV4"  Part="1"
-AR Path="/5355C3A0/531ECB11" Ref="RV1"  Part="1"
-F 0 "RV1" H 5850 2000 50  0000 C CNN
+F 0 "RV28" H 5850 2000 50  0000 C CNN
 F 1 "200" H 5850 2100 50  0000 C CNN
 F 2 "~" H 5850 2100 60  0000 C CNN
@@
 	5850 2350 5850 2400
 $Comp
-L GND #PWR08
-U 1 1 531ED061
+L GND #PWR062
+U 1 1 53598F25
 P 6050 1900
-AR Path="/531E9A87/531ED061" Ref="#PWR08"  Part="1"
-AR Path="/531FFF34/531ED061" Ref="#PWR063"  Part="1"
-AR Path="/5355C3A0/531ED061" Ref="#PWR08"  Part="1"
-F 0 "#PWR08" H 6050 1900 30  0001 C CNN
+F 0 "#PWR062" H 6050 1900 30  0001 C CNN
 F 1 "GND" H 6050 1830 30  0001 C CNN
 F 2 "" H 6050 1900 60  0000 C CNN
@@
 -5V
 $Comp
-L C C1
+L C C54
 U 1 1 531EE90B
 P 3100 1350
-AR Path="/531E9A87/531EE90B" Ref="C1"  Part="1"
-AR Path="/531FFF34/531EE90B" Ref="C58"  Part="1"
-AR Path="/5355C3A0/531EE90B" Ref="C1"  Part="1"
-F 0 "C1" H 3100 1450 40  0000 L CNN
+F 0 "C54" H 3100 1450 40  0000 L CNN
 F 1 "10u" H 3106 1265 40  0000 L CNN
 F 2 "~" H 3138 1200 30  0000 C CNN
@@
 $EndComp
 $Comp
-L C C2
+L C C55
 U 1 1 531EE911
 P 3100 1850
-AR Path="/531E9A87/531EE911" Ref="C2"  Part="1"
-AR Path="/531FFF34/531EE911" Ref="C59"  Part="1"
-AR Path="/5355C3A0/531EE911" Ref="C2"  Part="1"
-F 0 "C2" H 3100 1950 40  0000 L CNN
+F 0 "C55" H 3100 1950 40  0000 L CNN
 F 1 "10u" H 3106 1765 40  0000 L CNN
 F 2 "~" H 3138 1700 30  0000 C CNN
@@
 $EndComp
 $Comp
-L GND #PWR09
-U 1 1 531EE917
+L GND #PWR063
+U 1 1 53598F28
 P 3200 1650
-AR Path="/531E9A87/531EE917" Ref="#PWR09"  Part="1"
-AR Path="/531FFF34/531EE917" Ref="#PWR064"  Part="1"
-AR Path="/5355C3A0/531EE917" Ref="#PWR09"  Part="1"
-F 0 "#PWR09" H 3200 1650 30  0001 C CNN
+F 0 "#PWR063" H 3200 1650 30  0001 C CNN
 F 1 "GND" H 3200 1580 30  0001 C CNN
 F 2 "" H 3200 1650 60  0000 C CNN
@@
 	5450 2900 6000 2900
 $Comp
-L C C4
+L C C56
 U 1 1 531FE94B
 P 4300 3250
-AR Path="/531E9A87/531FE94B" Ref="C4"  Part="1"
-AR Path="/531FFF34/531FE94B" Ref="C61"  Part="1"
-AR Path="/5355C3A0/531FE94B" Ref="C4"  Part="1"
-F 0 "C4" H 4300 3350 40  0000 L CNN
+F 0 "C56" H 4300 3350 40  0000 L CNN
 F 1 "1p" H 4306 3165 40  0000 L CNN
 F 2 "~" H 4338 3100 30  0000 C CNN
@@
 $EndComp
 $Comp
-L GND #PWR010
-U 1 1 531FE951
+L GND #PWR064
+U 1 1 53598F2E
 P 4300 3500
-AR Path="/531E9A87/531FE951" Ref="#PWR010"  Part="1"
-AR Path="/531FFF34/531FE951" Ref="#PWR065"  Part="1"
-AR Path="/5355C3A0/531FE951" Ref="#PWR010"  Part="1"
-F 0 "#PWR010" H 4300 3500 30  0001 C CNN
+F 0 "#PWR064" H 4300 3500 30  0001 C CNN
 F 1 "GND" H 4300 3430 30  0001 C CNN
 F 2 "" H 4300 3500 60  0000 C CNN
@@
 $Sheet
 S 3850 1100 600  200
-U 53555E75
+U 53598F30
 F0 "CtrlConvert" 50
 F1 "CtrlConvert.sch" 50

Commit message: [pid] -
Parts:
- renumbered R97 to R100, R98 to R101, R96 to R99
Changed lines of the file:
@@
 $Descr A4 11693 8268
 encoding utf-8
-Sheet 23 47
+Sheet 23 53
 Title ""
-Date "1 may 2014"
+Date "2 may 2014"
 Rev ""
 Comp ""
@@
 	3650 3100 3850 3100
 $Comp
-L R R96
+L R R99
 U 1 1 531EACE1
 P 4050 2800
-F 0 "R96" V 4130 2800 40  0000 C CNN
+AR Path="/5355C3A0/531EACE1" Ref="R99"  Part="1"
+AR Path="/5362BBC7/531EACE1" Ref="R150"  Part="1"
+F 0 "R99" V 4130 2800 40  0000 C CNN
 F 1 "100" V 4057 2801 40  0000 C CNN
 F 2 "~" V 3980 2800 30  0000 C CNN
@@
 U 1 1 531EAD57
 P 4850 2900
+AR Path="/5355C3A0/531EAD57" Ref="U14"  Part="1"
+AR Path="/5362BBC7/531EAD57" Ref="U25"  Part="1"
 F 0 "U14" H 5150 3100 60  0000 C CNN
 F 1 "LM7171" H 4950 2900 60  0000 C CNN
@@
 $EndComp
 $Comp
-L R R97
+L R R100
 U 1 1 531EAE22
 P 4450 2350
-F 0 "R97" V 4530 2350 40  0000 C CNN
+AR Path="/5355C3A0/531EAE22" Ref="R100"  Part="1"
+AR Path="/5362BBC7/531EAE22" Ref="R151"  Part="1"
+F 0 "R100" V 4530 2350 40  0000 C CNN
 F 1 "100" V 4457 2351 40  0000 C CNN
 F 2 "~" V 4380 2350 30  0000 C CNN
@@
 	4950 3350 5000 3350
 $Comp
-L GND #PWR061
+L GND #PWR066
 U 1 1 53598F22
 P 4400 3100
-F 0 "#PWR061" H 4400 3100 30  0001 C CNN
+AR Path="/5355C3A0/53598F22" Ref="#PWR066"  Part="1"
+AR Path="/5362BBC7/53598F22" Ref="#PWR0104"  Part="1"
+F 0 "#PWR066" H 4400 3100 30  0001 C CNN
 F 1 "GND" H 4400 3030 30  0001 C CNN
 F 2 "" H 4400 3100 60  0000 C CNN
@@
 	4400 3000 4400 3100
 $Comp
-L R R98
+L R R101
 U 1 1 53598F23
 P 5850 2650
-F 0 "R98" V 5930 2650 40  0000 C CNN
+AR Path="/5355C3A0/53598F23" Ref="R101"  Part="1"
+AR Path="/5362BBC7/53598F23" Ref="R152"  Part="1"
+F 0 "R101" V 5930 2650 40  0000 C CNN
 F 1 "200" V 5857 2651 40  0000 C CNN
 F 2 "~" V 5780 2650 30  0000 C CNN
@@
 U 1 1 53598F24
 P 5850 2100
+AR Path="/5355C3A0/53598F24" Ref="RV28"  Part="1"
+AR Path="/5362BBC7/53598F24" Ref="RV42"  Part="1"
 F 0 "RV28" H 5850 2000 50  0000 C CNN
 F 1 "200" H 5850 2100 50  0000 C CNN
@@
 	5850 2350 5850 2400
 $Comp
-L GND #PWR062
+L GND #PWR067
 U 1 1 53598F25
 P 6050 1900
-F 0 "#PWR062" H 6050 1900 30  0001 C CNN
+AR Path="/5355C3A0/53598F25" Ref="#PWR067"  Part="1"
+AR Path="/5362BBC7/53598F25" Ref="#PWR0105"  Part="1"
+F 0 "#PWR067" H 6050 1900 30  0001 C CNN
 F 1 "GND" H 6050 1830 30  0001 C CNN
 F 2 "" H 6050 1900 60  0000 C CNN
@@
 U 1 1 531EE90B
 P 3100 1350
+AR Path="/5355C3A0/531EE90B" Ref="C54"  Part="1"
+AR Path="/5362BBC7/531EE90B" Ref="C89"  Part="1"
 F 0 "C54" H 3100 1450 40  0000 L CNN
 F 1 "10u" H 3106 1265 40  0000 L CNN
@@
 U 1 1 531EE911
 P 3100 1850
+AR Path="/5355C3A0/531EE911" Ref="C55"  Part="1"
+AR Path="/5362BBC7/531EE911" Ref="C90"  Part="1"
 F 0 "C55" H 3100 1950 40  0000 L CNN
 F 1 "10u" H 3106 1765 40  0000 L CNN
@@
 $EndComp
 $Comp
-L GND #PWR063
+L GND #PWR068
 U 1 1 53598F28
 P 3200 1650
-F 0 "#PWR063" H 3200 1650 30  0001 C CNN
+AR Path="/5355C3A0/53598F28" Ref="#PWR068"  Part="1"
+AR Path="/5362BBC7/53598F28" Ref="#PWR0106"  Part="1"
+F 0 "#PWR068" H 3200 1650 30  0001 C CNN
 F 1 "GND" H 3200 1580 30  0001 C CNN
 F 2 "" H 3200 1650 60  0000 C CNN
@@
 U 1 1 531FE94B
 P 4300 3250
+AR Path="/5355C3A0/531FE94B" Ref="C56"  Part="1"
+AR Path="/5362BBC7/531FE94B" Ref="C91"  Part="1"
 F 0 "C56" H 4300 3350 40  0000 L CNN
 F 1 "1p" H 4306 3165 40  0000 L CNN
@@
 $EndComp
 $Comp
-L GND #PWR064
+L GND #PWR069
 U 1 1 53598F2E
 P 4300 3500
-F 0 "#PWR064" H 4300 3500 30  0001 C CNN
+AR Path="/5355C3A0/53598F2E" Ref="#PWR069"  Part="1"
+AR Path="/5362BBC7/53598F2E" Ref="#PWR0107"  Part="1"
+F 0 "#PWR069" H 4300 3500 30  0001 C CNN
 F 1 "GND" H 4300 3430 30  0001 C CNN
 F 2 "" H 4300 3500 60  0000 C CNN

Commit message: [pid] more capacitors, layout
Changed lines of the file:
@@
 AR Path="/5355C3A0/531EACE1" Ref="R99"  Part="1"
 AR Path="/5362BBC7/531EACE1" Ref="R150"  Part="1"
-F 0 "R99" V 4130 2800 40  0000 C CNN
+F 0 "R150" V 4130 2800 40  0000 C CNN
 F 1 "100" V 4057 2801 40  0000 C CNN
 F 2 "~" V 3980 2800 30  0000 C CNN
@@
 AR Path="/5355C3A0/531EAD57" Ref="U14"  Part="1"
 AR Path="/5362BBC7/531EAD57" Ref="U25"  Part="1"
-F 0 "U14" H 5150 3100 60  0000 C CNN
+F 0 "U25" H 5150 3100 60  0000 C CNN
 F 1 "LM7171" H 4950 2900 60  0000 C CNN
 F 2 "~" H 4850 2900 60  0000 C CNN
@@
 AR Path="/5355C3A0/531EAE22" Ref="R100"  Part="1"
 AR Path="/5362BBC7/531EAE22" Ref="R151"  Part="1"
-F 0 "R100" V 4530 2350 40  0000 C CNN
+F 0 "R151" V 4530 2350 40  0000 C CNN
 F 1 "100" V 4457 2351 40  0000 C CNN
 F 2 "~" V 4380 2350 30  0000 C CNN
@@
 	4950 3350 5000 3350
 $Comp
-L GND #PWR070
+L GND #PWR74
 U 1 1 53598F22
 P 4400 3100
-AR Path="/5355C3A0/53598F22" Ref="#PWR070"  Part="1"
-AR Path="/5362BBC7/53598F22" Ref="#PWR0108"  Part="1"
-F 0 "#PWR0108" H 4400 3100 30  0001 C CNN
+AR Path="/5355C3A0/53598F22" Ref="#PWR74"  Part="1"
+AR Path="/5362BBC7/53598F22" Ref="#PWR113"  Part="1"
+F 0 "#PWR113" H 4400 3100 30  0001 C CNN
 F 1 "GND" H 4400 3030 30  0001 C CNN
 F 2 "" H 4400 3100 60  0000 C CNN
@@
 AR Path="/5355C3A0/53598F23" Ref="R101"  Part="1"
 AR Path="/5362BBC7/53598F23" Ref="R152"  Part="1"
-F 0 "R101" V 5930 2650 40  0000 C CNN
+F 0 "R152" V 5930 2650 40  0000 C CNN
 F 1 "200" V 5857 2651 40  0000 C CNN
 F 2 "~" V 5780 2650 30  0000 C CNN
@@
 AR Path="/5355C3A0/53598F24" Ref="RV28"  Part="1"
 AR Path="/5362BBC7/53598F24" Ref="RV42"  Part="1"
-F 0 "RV28" H 5850 2000 50  0000 C CNN
+F 0 "RV42" H 5850 2000 50  0000 C CNN
 F 1 "200" H 5850 2100 50  0000 C CNN
 F 2 "~" H 5850 2100 60  0000 C CNN
@@
 	5850 2350 5850 2400
 $Comp
-L GND #PWR071
+L GND #PWR75
 U 1 1 53598F25
 P 6050 1900
-AR Path="/5355C3A0/53598F25" Ref="#PWR071"  Part="1"
-AR Path="/5362BBC7/53598F25" Ref="#PWR0109"  Part="1"
-F 0 "#PWR0109" H 6050 1900 30  0001 C CNN
+AR Path="/5355C3A0/53598F25" Ref="#PWR75"  Part="1"
+AR Path="/5362BBC7/53598F25" Ref="#PWR114"  Part="1"
+F 0 "#PWR114" H 6050 1900 30  0001 C CNN
 F 1 "GND" H 6050 1830 30  0001 C CNN
 F 2 "" H 6050 1900 60  0000 C CNN
@@
 AR Path="/5355C3A0/531EE90B" Ref="C54"  Part="1"
 AR Path="/5362BBC7/531EE90B" Ref="C89"  Part="1"
-F 0 "C54" H 3100 1450 40  0000 L CNN
+F 0 "C89" H 3100 1450 40  0000 L CNN
 F 1 "10u" H 3106 1265 40  0000 L CNN
 F 2 "~" H 3138 1200 30  0000 C CNN
@@
 AR Path="/5355C3A0/531EE911" Ref="C55"  Part="1"
 AR Path="/5362BBC7/531EE911" Ref="C90"  Part="1"
-F 0 "C55" H 3100 1950 40  0000 L CNN
+F 0 "C90" H 3100 1950 40  0000 L CNN
 F 1 "10u" H 3106 1765 40  0000 L CNN
 F 2 "~" H 3138 1700 30  0000 C CNN
@@
 $EndComp
 $Comp
-L GND #PWR072
+L GND #PWR72
 U 1 1 53598F28
 P 3200 1650
-AR Path="/5355C3A0/53598F28" Ref="#PWR072"  Part="1"
-AR Path="/5362BBC7/53598F28" Ref="#PWR0110"  Part="1"
-F 0 "#PWR0110" H 3200 1650 30  0001 C CNN
+AR Path="/5355C3A0/53598F28" Ref="#PWR72"  Part="1"
+AR Path="/5362BBC7/53598F28" Ref="#PWR111"  Part="1"
+F 0 "#PWR111" H 3200 1650 30  0001 C CNN
 F 1 "GND" H 3200 1580 30  0001 C CNN
 F 2 "" H 3200 1650 60  0000 C CNN
@@
 AR Path="/5355C3A0/531FE94B" Ref="C56"  Part="1"
 AR Path="/5362BBC7/531FE94B" Ref="C91"  Part="1"
-F 0 "C56" H 4300 3350 40  0000 L CNN
+F 0 "C91" H 4300 3350 40  0000 L CNN
 F 1 "1p" H 4306 3165 40  0000 L CNN
 F 2 "~" H 4338 3100 30  0000 C CNN
@@
 $EndComp
 $Comp
-L GND #PWR073
+L GND #PWR73
 U 1 1 53598F2E
 P 4300 3500
-AR Path="/5355C3A0/53598F2E" Ref="#PWR073"  Part="1"
-AR Path="/5362BBC7/53598F2E" Ref="#PWR0111"  Part="1"
-F 0 "#PWR0111" H 4300 3500 30  0001 C CNN
+AR Path="/5355C3A0/53598F2E" Ref="#PWR73"  Part="1"
+AR Path="/5362BBC7/53598F2E" Ref="#PWR112"  Part="1"
+F 0 "#PWR112" H 4300 3500 30  0001 C CNN
 F 1 "GND" H 4300 3430 30  0001 C CNN
 F 2 "" H 4300 3500 60  0000 C CNN

Commit message: [pid] layout
Changed lines of the file:
@@
 Sheet 23 53
 Title ""
-Date "2 may 2014"
+Date "5 may 2014"
 Rev ""
 Comp ""
@@
 AR Path="/5355C3A0/531EACE1" Ref="R99"  Part="1"
 AR Path="/5362BBC7/531EACE1" Ref="R150"  Part="1"
-F 0 "R150" V 4130 2800 40  0000 C CNN
+F 0 "R99" V 4130 2800 40  0000 C CNN
 F 1 "100" V 4057 2801 40  0000 C CNN
 F 2 "~" V 3980 2800 30  0000 C CNN
@@
 AR Path="/5355C3A0/531EAD57" Ref="U14"  Part="1"
 AR Path="/5362BBC7/531EAD57" Ref="U25"  Part="1"
-F 0 "U25" H 5150 3100 60  0000 C CNN
+F 0 "U14" H 5150 3100 60  0000 C CNN
 F 1 "LM7171" H 4950 2900 60  0000 C CNN
 F 2 "~" H 4850 2900 60  0000 C CNN
@@
 AR Path="/5355C3A0/531EAE22" Ref="R100"  Part="1"
 AR Path="/5362BBC7/531EAE22" Ref="R151"  Part="1"
-F 0 "R151" V 4530 2350 40  0000 C CNN
+F 0 "R100" V 4530 2350 40  0000 C CNN
 F 1 "100" V 4457 2351 40  0000 C CNN
 F 2 "~" V 4380 2350 30  0000 C CNN
@@
 	4950 3350 5000 3350
 $Comp
-L GND #PWR74
+L GND #PWR072
 U 1 1 53598F22
 P 4400 3100
-AR Path="/5355C3A0/53598F22" Ref="#PWR74"  Part="1"
-AR Path="/5362BBC7/53598F22" Ref="#PWR113"  Part="1"
-F 0 "#PWR113" H 4400 3100 30  0001 C CNN
+AR Path="/5355C3A0/53598F22" Ref="#PWR072"  Part="1"
+AR Path="/5362BBC7/53598F22" Ref="#PWR0111"  Part="1"
+F 0 "#PWR072" H 4400 3100 30  0001 C CNN
 F 1 "GND" H 4400 3030 30  0001 C CNN
 F 2 "" H 4400 3100 60  0000 C CNN
@@
 AR Path="/5355C3A0/53598F23" Ref="R101"  Part="1"
 AR Path="/5362BBC7/53598F23" Ref="R152"  Part="1"
-F 0 "R152" V 5930 2650 40  0000 C CNN
+F 0 "R101" V 5930 2650 40  0000 C CNN
 F 1 "200" V 5857 2651 40  0000 C CNN
 F 2 "~" V 5780 2650 30  0000 C CNN
@@
 AR Path="/5355C3A0/53598F24" Ref="RV28"  Part="1"
 AR Path="/5362BBC7/53598F24" Ref="RV42"  Part="1"
-F 0 "RV42" H 5850 2000 50  0000 C CNN
+F 0 "RV28" H 5850 2000 50  0000 C CNN
 F 1 "200" H 5850 2100 50  0000 C CNN
 F 2 "~" H 5850 2100 60  0000 C CNN
@@
 	5850 2350 5850 2400
 $Comp
-L GND #PWR75
+L GND #PWR073
 U 1 1 53598F25
 P 6050 1900
-AR Path="/5355C3A0/53598F25" Ref="#PWR75"  Part="1"
-AR Path="/5362BBC7/53598F25" Ref="#PWR114"  Part="1"
-F 0 "#PWR114" H 6050 1900 30  0001 C CNN
+AR Path="/5355C3A0/53598F25" Ref="#PWR073"  Part="1"
+AR Path="/5362BBC7/53598F25" Ref="#PWR0112"  Part="1"
+F 0 "#PWR073" H 6050 1900 30  0001 C CNN
 F 1 "GND" H 6050 1830 30  0001 C CNN
 F 2 "" H 6050 1900 60  0000 C CNN
@@
 AR Path="/5355C3A0/531EE90B" Ref="C54"  Part="1"
 AR Path="/5362BBC7/531EE90B" Ref="C89"  Part="1"
-F 0 "C89" H 3100 1450 40  0000 L CNN
+F 0 "C54" H 3100 1450 40  0000 L CNN
 F 1 "10u" H 3106 1265 40  0000 L CNN
 F 2 "~" H 3138 1200 30  0000 C CNN
@@
 AR Path="/5355C3A0/531EE911" Ref="C55"  Part="1"
 AR Path="/5362BBC7/531EE911" Ref="C90"  Part="1"
-F 0 "C90" H 3100 1950 40  0000 L CNN
+F 0 "C55" H 3100 1950 40  0000 L CNN
 F 1 "10u" H 3106 1765 40  0000 L CNN
 F 2 "~" H 3138 1700 30  0000 C CNN
@@
 $EndComp
 $Comp
-L GND #PWR72
+L GND #PWR074
 U 1 1 53598F28
 P 3200 1650
-AR Path="/5355C3A0/53598F28" Ref="#PWR72"  Part="1"
-AR Path="/5362BBC7/53598F28" Ref="#PWR111"  Part="1"
-F 0 "#PWR111" H 3200 1650 30  0001 C CNN
+AR Path="/5355C3A0/53598F28" Ref="#PWR074"  Part="1"
+AR Path="/5362BBC7/53598F28" Ref="#PWR0113"  Part="1"
+F 0 "#PWR074" H 3200 1650 30  0001 C CNN
 F 1 "GND" H 3200 1580 30  0001 C CNN
 F 2 "" H 3200 1650 60  0000 C CNN
@@
 AR Path="/5355C3A0/531FE94B" Ref="C56"  Part="1"
 AR Path="/5362BBC7/531FE94B" Ref="C91"  Part="1"
-F 0 "C91" H 4300 3350 40  0000 L CNN
+F 0 "C56" H 4300 3350 40  0000 L CNN
 F 1 "1p" H 4306 3165 40  0000 L CNN
 F 2 "~" H 4338 3100 30  0000 C CNN
@@
 $EndComp
 $Comp
-L GND #PWR73
+L GND #PWR075
 U 1 1 53598F2E
 P 4300 3500
-AR Path="/5355C3A0/53598F2E" Ref="#PWR73"  Part="1"
-AR Path="/5362BBC7/53598F2E" Ref="#PWR112"  Part="1"
-F 0 "#PWR112" H 4300 3500 30  0001 C CNN
+AR Path="/5355C3A0/53598F2E" Ref="#PWR075"  Part="1"
+AR Path="/5362BBC7/53598F2E" Ref="#PWR0114"  Part="1"
+F 0 "#PWR075" H 4300 3500 30  0001 C CNN
 F 1 "GND" H 4300 3430 30  0001 C CNN
 F 2 "" H 4300 3500 60  0000 C CNN

Commit message: [pid] update
Changed lines of the file:
@@
 Sheet 23 53
 Title ""
-Date "19 may 2014"
+Date "28 may 2014"
 Rev ""
 Comp ""
@@
 AR Path="/5355C3A0/531EACE1" Ref="R99"  Part="1"
 AR Path="/5362BBC7/531EACE1" Ref="R150"  Part="1"
-F 0 "R99" V 4130 2800 40  0000 C CNN
+F 0 "R150" V 4130 2800 40  0000 C CNN
 F 1 "100" V 4057 2801 40  0000 C CNN
 F 2 "~" V 3980 2800 30  0000 C CNN
@@
 AR Path="/5355C3A0/531EAD57" Ref="U14"  Part="1"
 AR Path="/5362BBC7/531EAD57" Ref="U25"  Part="1"
-F 0 "U14" H 5150 3100 60  0000 C CNN
+F 0 "U25" H 5150 3100 60  0000 C CNN
 F 1 "LM7171" H 4950 2900 60  0000 C CNN
 F 2 "~" H 4850 2900 60  0000 C CNN
@@
 AR Path="/5355C3A0/531EAE22" Ref="R100"  Part="1"
 AR Path="/5362BBC7/531EAE22" Ref="R151"  Part="1"
-F 0 "R100" V 4530 2350 40  0000 C CNN
+F 0 "R151" V 4530 2350 40  0000 C CNN
 F 1 "100" V 4457 2351 40  0000 C CNN
 F 2 "~" V 4380 2350 30  0000 C CNN
@@
 AR Path="/5355C3A0/53598F22" Ref="#PWR072"  Part="1"
 AR Path="/5362BBC7/53598F22" Ref="#PWR0111"  Part="1"
-F 0 "#PWR072" H 4400 3100 30  0001 C CNN
+F 0 "#PWR0111" H 4400 3100 30  0001 C CNN
 F 1 "GND" H 4400 3030 30  0001 C CNN
 F 2 "" H 4400 3100 60  0000 C CNN
@@
 AR Path="/5355C3A0/53598F23" Ref="R101"  Part="1"
 AR Path="/5362BBC7/53598F23" Ref="R152"  Part="1"
-F 0 "R101" V 5930 2650 40  0000 C CNN
+F 0 "R152" V 5930 2650 40  0000 C CNN
 F 1 "200" V 5857 2651 40  0000 C CNN
 F 2 "~" V 5780 2650 30  0000 C CNN
@@
 AR Path="/5355C3A0/53598F24" Ref="RV28"  Part="1"
 AR Path="/5362BBC7/53598F24" Ref="RV42"  Part="1"
-F 0 "RV28" H 5850 2000 50  0000 C CNN
+F 0 "RV42" H 5850 2000 50  0000 C CNN
 F 1 "200" H 5850 2100 50  0000 C CNN
 F 2 "~" H 5850 2100 60  0000 C CNN
@@
 AR Path="/5355C3A0/53598F25" Ref="#PWR073"  Part="1"
 AR Path="/5362BBC7/53598F25" Ref="#PWR0112"  Part="1"
-F 0 "#PWR073" H 6050 1900 30  0001 C CNN
+F 0 "#PWR0112" H 6050 1900 30  0001 C CNN
 F 1 "GND" H 6050 1830 30  0001 C CNN
 F 2 "" H 6050 1900 60  0000 C CNN
@@
 AR Path="/5355C3A0/531EE90B" Ref="C54"  Part="1"
 AR Path="/5362BBC7/531EE90B" Ref="C89"  Part="1"
-F 0 "C54" H 3100 1450 40  0000 L CNN
+F 0 "C89" H 3100 1450 40  0000 L CNN
 F 1 "10u" H 3106 1265 40  0000 L CNN
 F 2 "~" H 3138 1200 30  0000 C CNN
@@
 AR Path="/5355C3A0/531EE911" Ref="C55"  Part="1"
 AR Path="/5362BBC7/531EE911" Ref="C90"  Part="1"
-F 0 "C55" H 3100 1950 40  0000 L CNN
+F 0 "C90" H 3100 1950 40  0000 L CNN
 F 1 "10u" H 3106 1765 40  0000 L CNN
 F 2 "~" H 3138 1700 30  0000 C CNN
@@
 AR Path="/5355C3A0/53598F28" Ref="#PWR074"  Part="1"
 AR Path="/5362BBC7/53598F28" Ref="#PWR0113"  Part="1"
-F 0 "#PWR074" H 3200 1650 30  0001 C CNN
+F 0 "#PWR0113" H 3200 1650 30  0001 C CNN
 F 1 "GND" H 3200 1580 30  0001 C CNN
 F 2 "" H 3200 1650 60  0000 C CNN
@@
 AR Path="/5355C3A0/531FE94B" Ref="C56"  Part="1"
 AR Path="/5362BBC7/531FE94B" Ref="C91"  Part="1"
-F 0 "C56" H 4300 3350 40  0000 L CNN
+F 0 "C91" H 4300 3350 40  0000 L CNN
 F 1 "1p" H 4306 3165 40  0000 L CNN
 F 2 "~" H 4338 3100 30  0000 C CNN
@@
 AR Path="/5355C3A0/53598F2E" Ref="#PWR075"  Part="1"
 AR Path="/5362BBC7/53598F2E" Ref="#PWR0114"  Part="1"
-F 0 "#PWR075" H 4300 3500 30  0001 C CNN
+F 0 "#PWR0114" H 4300 3500 30  0001 C CNN
 F 1 "GND" H 4300 3430 30  0001 C CNN
 F 2 "" H 4300 3500 60  0000 C CNN
