File: pid/Instrumentation.sch (KiCad schematic (older format))
At the start: 6 parts, among them U13 AD8421

Commit message: [pid] -
Parts:
- renumbered R93 to R96, R94 to R97, R95 to R98
Changed lines of the file:
@@
 $Descr A4 11693 8268
 encoding utf-8
-Sheet 21 47
+Sheet 21 53
 Title ""
-Date "1 may 2014"
+Date "2 may 2014"
 Rev ""
 Comp ""
@@
 $EndComp
 $Comp
-L R R95
+L R R98
 U 1 1 5356B2FA
 P 3250 3600
-F 0 "R95" V 3330 3600 40  0000 C CNN
+F 0 "R98" V 3330 3600 40  0000 C CNN
 F 1 "200" V 3257 3601 40  0000 C CNN
 F 2 "~" V 3180 3600 30  0000 C CNN
@@
 In-
 $Comp
-L GND #PWR057
+L GND #PWR062
 U 1 1 5356B703
 P 4200 3950
-F 0 "#PWR057" H 4200 3950 30  0001 C CNN
+F 0 "#PWR062" H 4200 3950 30  0001 C CNN
 F 1 "GND" H 4200 3880 30  0001 C CNN
 F 2 "" H 4200 3950 60  0000 C CNN
@@
 $EndComp
 $Comp
-L GND #PWR058
+L GND #PWR063
 U 1 1 5356BD73
 P 2600 3700
-F 0 "#PWR058" H 2600 3700 30  0001 C CNN
+F 0 "#PWR063" H 2600 3700 30  0001 C CNN
 F 1 "GND" H 2600 3630 30  0001 C CNN
 F 2 "" H 2600 3700 60  0000 C CNN
@@
 $EndComp
 $Comp
-L GND #PWR059
+L GND #PWR064
 U 1 1 5359724B
 P 2900 3650
-F 0 "#PWR059" H 2900 3650 30  0001 C CNN
+F 0 "#PWR064" H 2900 3650 30  0001 C CNN
 F 1 "GND" H 2900 3580 30  0001 C CNN
 F 2 "" H 2900 3650 60  0000 C CNN
@@
 	3050 4400 3000 4400
 $Comp
-L R_DIV R93
+L R_DIV R96
 U 1 1 53597ABD
 P 3050 3200
-F 0 "R93" V 3120 3060 40  0000 C CNN
+F 0 "R96" V 3120 3060 40  0000 C CNN
 F 1 "16.67k" V 2990 3200 40  0000 C CNN
 F 2 "~" V 2980 3000 30  0000 C CNN
@@
 $EndComp
 $Comp
-L R_DIV R94
+L R_DIV R97
 U 1 1 53597AD4
 P 3050 4000
-F 0 "R94" V 3120 3860 40  0000 C CNN
+F 0 "R97" V 3120 3860 40  0000 C CNN
 F 1 "16.67k" V 2990 4000 40  0000 C CNN
 F 2 "~" V 2980 3800 30  0000 C CNN
