File: pid/OffsetAdjust.sch (KiCad schematic (older format))
At the start: 7 parts

Commit message: [pid] -
Parts:
- gave numbers to parts that had none: 7
Changed lines of the file:
@@
 LIBS:rb-0524s
 LIBS:max44251
+LIBS:r_div
 LIBS:pid-cache
 EELAYER 27 0
@@
 $Descr A4 11693 8268
 encoding utf-8
-Sheet 5 27
+Sheet 23 47
 Title ""
-Date "22 apr 2014"
+Date "1 may 2014"
 Rev ""
 Comp ""
@@
 -5V
 $Comp
-L POT RV?
+L POT RV3
 U 1 1 53547B5F
 P 3450 4650
-AR Path="/531E9A87/531E6F48/53548633/53547B5F" Ref="RV?"  Part="1"
-AR Path="/531E9A87/531E6F48/53547A94/53547B5F" Ref="RV?"  Part="1"
-F 0 "RV?" H 3450 4550 50  0000 C CNN
+AR Path="/5355B409/53598F1D/53548633/53547B5F" Ref="RV3"  Part="1"
+AR Path="/5355B409/53598F1D/53547A94/53547B5F" Ref="RV5"  Part="1"
+AR Path="/5355B409/531EB865/53548633/53547B5F" Ref="RV7"  Part="1"
+AR Path="/5355B409/531EB865/53547A94/53547B5F" Ref="RV9"  Part="1"
+AR Path="/53562461/5321AFC5/53548633/53547B5F" Ref="RV17"  Part="1"
+AR Path="/53562461/5321AFC5/53547A94/53547B5F" Ref="RV19"  Part="1"
+AR Path="/53562461/5321AFC7/53548633/53547B5F" Ref="RV21"  Part="1"
+AR Path="/53562461/5321AFC7/53547A94/53547B5F" Ref="RV23"  Part="1"
+AR Path="/5355C3A0/531E6F48/53548633/53547B5F" Ref="RV30"  Part="1"
+AR Path="/5355C3A0/531E6F48/53547A94/53547B5F" Ref="RV32"  Part="1"
+AR Path="/5355C3A0/53598F21/53548633/53547B5F" Ref="RV34"  Part="1"
+AR Path="/5355C3A0/53598F21/53547A94/53547B5F" Ref="RV36"  Part="1"
+F 0 "RV36" H 3450 4550 50  0000 C CNN
 F 1 "10k" H 3450 4650 50  0000 C CNN
 F 2 "~" H 3450 4650 60  0000 C CNN
@@
 $EndComp
 $Comp
-L POT RV?
+L POT RV2
 U 1 1 53547B6E
 P 2950 4650
-AR Path="/531E9A87/531E6F48/53548633/53547B6E" Ref="RV?"  Part="1"
-AR Path="/531E9A87/531E6F48/53547A94/53547B6E" Ref="RV?"  Part="1"
-F 0 "RV?" H 2950 4550 50  0000 C CNN
+AR Path="/5355B409/53598F1D/53548633/53547B6E" Ref="RV2"  Part="1"
+AR Path="/5355B409/53598F1D/53547A94/53547B6E" Ref="RV4"  Part="1"
+AR Path="/5355B409/531EB865/53548633/53547B6E" Ref="RV6"  Part="1"
+AR Path="/5355B409/531EB865/53547A94/53547B6E" Ref="RV8"  Part="1"
+AR Path="/53562461/5321AFC5/53548633/53547B6E" Ref="RV16"  Part="1"
+AR Path="/53562461/5321AFC5/53547A94/53547B6E" Ref="RV18"  Part="1"
+AR Path="/53562461/5321AFC7/53548633/53547B6E" Ref="RV20"  Part="1"
+AR Path="/53562461/5321AFC7/53547A94/53547B6E" Ref="RV22"  Part="1"
+AR Path="/5355C3A0/531E6F48/53548633/53547B6E" Ref="RV29"  Part="1"
+AR Path="/5355C3A0/531E6F48/53547A94/53547B6E" Ref="RV31"  Part="1"
+AR Path="/5355C3A0/53598F21/53548633/53547B6E" Ref="RV33"  Part="1"
+AR Path="/5355C3A0/53598F21/53547A94/53547B6E" Ref="RV35"  Part="1"
+F 0 "RV35" H 2950 4550 50  0000 C CNN
 F 1 "100k" H 2950 4650 50  0000 C CNN
 F 2 "~" H 2950 4650 60  0000 C CNN
@@
 $EndComp
 $Comp
-L R R?
+L R R19
 U 1 1 53547B7D
 P 3450 5250
-AR Path="/531E9A87/531E6F48/53548633/53547B7D" Ref="R?"  Part="1"
-AR Path="/531E9A87/531E6F48/53547A94/53547B7D" Ref="R?"  Part="1"
-F 0 "R?" V 3530 5250 40  0000 C CNN
+AR Path="/5355B409/53598F1D/53548633/53547B7D" Ref="R19"  Part="1"
+AR Path="/5355B409/53598F1D/53547A94/53547B7D" Ref="R23"  Part="1"
+AR Path="/5355B409/531EB865/53548633/53547B7D" Ref="R32"  Part="1"
+AR Path="/5355B409/531EB865/53547A94/53547B7D" Ref="R36"  Part="1"
+AR Path="/53562461/5321AFC5/53548633/53547B7D" Ref="R65"  Part="1"
+AR Path="/53562461/5321AFC5/53547A94/53547B7D" Ref="R69"  Part="1"
+AR Path="/53562461/5321AFC7/53548633/53547B7D" Ref="R78"  Part="1"
+AR Path="/53562461/5321AFC7/53547A94/53547B7D" Ref="R82"  Part="1"
+AR Path="/5355C3A0/531E6F48/53548633/53547B7D" Ref="R107"  Part="1"
+AR Path="/5355C3A0/531E6F48/53547A94/53547B7D" Ref="R111"  Part="1"
+AR Path="/5355C3A0/53598F21/53548633/53547B7D" Ref="R120"  Part="1"
+AR Path="/5355C3A0/53598F21/53547A94/53547B7D" Ref="R124"  Part="1"
+F 0 "R124" V 3530 5250 40  0000 C CNN
 F 1 "2k" V 3457 5251 40  0000 C CNN
 F 2 "~" V 3380 5250 30  0000 C CNN
@@
 $EndComp
 $Comp
-L R R?
+L R R18
 U 1 1 53547B8C
 P 3450 4050
-AR Path="/531E9A87/531E6F48/53548633/53547B8C" Ref="R?"  Part="1"
-AR Path="/531E9A87/531E6F48/53547A94/53547B8C" Ref="R?"  Part="1"
-F 0 "R?" V 3530 4050 40  0000 C CNN
+AR Path="/5355B409/53598F1D/53548633/53547B8C" Ref="R18"  Part="1"
+AR Path="/5355B409/53598F1D/53547A94/53547B8C" Ref="R22"  Part="1"
+AR Path="/5355B409/531EB865/53548633/53547B8C" Ref="R31"  Part="1"
+AR Path="/5355B409/531EB865/53547A94/53547B8C" Ref="R35"  Part="1"
+AR Path="/53562461/5321AFC5/53548633/53547B8C" Ref="R64"  Part="1"
+AR Path="/53562461/5321AFC5/53547A94/53547B8C" Ref="R68"  Part="1"
+AR Path="/53562461/5321AFC7/53548633/53547B8C" Ref="R77"  Part="1"
+AR Path="/53562461/5321AFC7/53547A94/53547B8C" Ref="R81"  Part="1"
+AR Path="/5355C3A0/531E6F48/53548633/53547B8C" Ref="R106"  Part="1"
+AR Path="/5355C3A0/531E6F48/53547A94/53547B8C" Ref="R110"  Part="1"
+AR Path="/5355C3A0/53598F21/53548633/53547B8C" Ref="R119"  Part="1"
+AR Path="/5355C3A0/53598F21/53547A94/53547B8C" Ref="R123"  Part="1"
+F 0 "R123" V 3530 4050 40  0000 C CNN
 F 1 "2k" V 3457 4051 40  0000 C CNN
 F 2 "~" V 3380 4050 30  0000 C CNN
@@
 $EndComp
 $Comp
-L R R?
+L R R16
 U 1 1 53547B9E
 P 2950 4050
-AR Path="/531E9A87/531E6F48/53548633/53547B9E" Ref="R?"  Part="1"
-AR Path="/531E9A87/531E6F48/53547A94/53547B9E" Ref="R?"  Part="1"
-F 0 "R?" V 3030 4050 40  0000 C CNN
+AR Path="/5355B409/53598F1D/53548633/53547B9E" Ref="R16"  Part="1"
+AR Path="/5355B409/53598F1D/53547A94/53547B9E" Ref="R20"  Part="1"
+AR Path="/5355B409/531EB865/53548633/53547B9E" Ref="R29"  Part="1"
+AR Path="/5355B409/531EB865/53547A94/53547B9E" Ref="R33"  Part="1"
+AR Path="/53562461/5321AFC5/53548633/53547B9E" Ref="R62"  Part="1"
+AR Path="/53562461/5321AFC5/53547A94/53547B9E" Ref="R66"  Part="1"
+AR Path="/53562461/5321AFC7/53548633/53547B9E" Ref="R75"  Part="1"
+AR Path="/53562461/5321AFC7/53547A94/53547B9E" Ref="R79"  Part="1"
+AR Path="/5355C3A0/531E6F48/53548633/53547B9E" Ref="R104"  Part="1"
+AR Path="/5355C3A0/531E6F48/53547A94/53547B9E" Ref="R108"  Part="1"
+AR Path="/5355C3A0/53598F21/53548633/53547B9E" Ref="R117"  Part="1"
+AR Path="/5355C3A0/53598F21/53547A94/53547B9E" Ref="R121"  Part="1"
+F 0 "R121" V 3030 4050 40  0000 C CNN
 F 1 "100k" V 2957 4051 40  0000 C CNN
 F 2 "~" V 2880 4050 30  0000 C CNN
@@
 $EndComp
 $Comp
-L R R?
+L R R17
 U 1 1 53547BA4
 P 2950 5250
-AR Path="/531E9A87/531E6F48/53548633/53547BA4" Ref="R?"  Part="1"
-AR Path="/531E9A87/531E6F48/53547A94/53547BA4" Ref="R?"  Part="1"
-F 0 "R?" V 3030 5250 40  0000 C CNN
+AR Path="/5355B409/53598F1D/53548633/53547BA4" Ref="R17"  Part="1"
+AR Path="/5355B409/53598F1D/53547A94/53547BA4" Ref="R21"  Part="1"
+AR Path="/5355B409/531EB865/53548633/53547BA4" Ref="R30"  Part="1"
+AR Path="/5355B409/531EB865/53547A94/53547BA4" Ref="R34"  Part="1"
+AR Path="/53562461/5321AFC5/53548633/53547BA4" Ref="R63"  Part="1"
+AR Path="/53562461/5321AFC5/53547A94/53547BA4" Ref="R67"  Part="1"
+AR Path="/53562461/5321AFC7/53548633/53547BA4" Ref="R76"  Part="1"
+AR Path="/53562461/5321AFC7/53547A94/53547BA4" Ref="R80"  Part="1"
+AR Path="/5355C3A0/531E6F48/53548633/53547BA4" Ref="R105"  Part="1"
+AR Path="/5355C3A0/531E6F48/53547A94/53547BA4" Ref="R109"  Part="1"
+AR Path="/5355C3A0/53598F21/53548633/53547BA4" Ref="R118"  Part="1"
+AR Path="/5355C3A0/53598F21/53547A94/53547BA4" Ref="R122"  Part="1"
+F 0 "R122" V 3030 5250 40  0000 C CNN
 F 1 "100k" V 2957 5251 40  0000 C CNN
 F 2 "~" V 2880 5250 30  0000 C CNN
@@
 Connection ~ 3200 4650
 $Comp
-L C C?
+L C C9
 U 1 1 53553A48
 P 3200 4950
-AR Path="/531E9A87/531E6F48/53547A94/53553A48" Ref="C?"  Part="1"
-AR Path="/531E9A87/531E6F48/53548633/53553A48" Ref="C?"  Part="1"
-F 0 "C?" H 3200 5050 40  0000 L CNN
+AR Path="/5355B409/53598F1D/53548633/53553A48" Ref="C9"  Part="1"
+AR Path="/5355B409/53598F1D/53547A94/53553A48" Ref="C10"  Part="1"
+AR Path="/5355B409/531EB865/53548633/53553A48" Ref="C14"  Part="1"
+AR Path="/5355B409/531EB865/53547A94/53553A48" Ref="C15"  Part="1"
+AR Path="/53562461/5321AFC5/53548633/53553A48" Ref="C34"  Part="1"
+AR Path="/53562461/5321AFC5/53547A94/53553A48" Ref="C35"  Part="1"
+AR Path="/53562461/5321AFC7/53548633/53553A48" Ref="C39"  Part="1"
+AR Path="/53562461/5321AFC7/53547A94/53553A48" Ref="C40"  Part="1"
+AR Path="/5355C3A0/531E6F48/53548633/53553A48" Ref="C60"  Part="1"
+AR Path="/5355C3A0/531E6F48/53547A94/53553A48" Ref="C61"  Part="1"
+AR Path="/5355C3A0/53598F21/53548633/53553A48" Ref="C65"  Part="1"
+AR Path="/5355C3A0/53598F21/53547A94/53553A48" Ref="C66"  Part="1"
+F 0 "C66" H 3200 5050 40  0000 L CNN
 F 1 "10u" H 3206 4865 40  0000 L CNN
 F 2 "~" H 3238 4800 30  0000 C CNN
@@
 $EndComp
 $Comp
-L GND #PWR?
+L GND #PWR013
 U 1 1 53553A57
 P 3200 5250
-AR Path="/531E9A87/531E6F48/53547A94/53553A57" Ref="#PWR?"  Part="1"
-AR Path="/531E9A87/531E6F48/53548633/53553A57" Ref="#PWR?"  Part="1"
-F 0 "#PWR?" H 3200 5250 30  0001 C CNN
+AR Path="/5355B409/53598F1D/53548633/53553A57" Ref="#PWR013"  Part="1"
+AR Path="/5355B409/53598F1D/53547A94/53553A57" Ref="#PWR014"  Part="1"
+AR Path="/5355B409/531EB865/53548633/53553A57" Ref="#PWR019"  Part="1"
+AR Path="/5355B409/531EB865/53547A94/53553A57" Ref="#PWR020"  Part="1"
+AR Path="/53562461/5321AFC5/53548633/53553A57" Ref="#PWR038"  Part="1"
+AR Path="/53562461/5321AFC5/53547A94/53553A57" Ref="#PWR039"  Part="1"
+AR Path="/53562461/5321AFC7/53548633/53553A57" Ref="#PWR044"  Part="1"
+AR Path="/53562461/5321AFC7/53547A94/53553A57" Ref="#PWR045"  Part="1"
+AR Path="/5355C3A0/531E6F48/53548633/53553A57" Ref="#PWR069"  Part="1"
+AR Path="/5355C3A0/531E6F48/53547A94/53553A57" Ref="#PWR070"  Part="1"
+AR Path="/5355C3A0/53598F21/53548633/53553A57" Ref="#PWR075"  Part="1"
+AR Path="/5355C3A0/53598F21/53547A94/53553A57" Ref="#PWR076"  Part="1"
+F 0 "#PWR076" H 3200 5250 30  0001 C CNN
 F 1 "GND" H 3200 5180 30  0001 C CNN
 F 2 "" H 3200 5250 60  0000 C CNN

Commit message: [pid] -
Parts:
- renumbered R16 to R19, R17 to R20, R18 to R21, R19 to R22

Commit message: [pid] layout
Changed lines of the file:
@@
 $Descr A4 11693 8268
 encoding utf-8
-Sheet 29 53
+Sheet 12 53
 Title ""
-Date "2 may 2014"
+Date "5 may 2014"
 Rev ""
 Comp ""
@@
 AR Path="/5362BBC7/53598F21/53548633/53547B5F" Ref="RV48"  Part="1"
 AR Path="/5362BBC7/53598F21/53547A94/53547B5F" Ref="RV50"  Part="1"
-F 0 "RV50" H 3450 4550 50  0000 C CNN
+F 0 "RV17" H 3450 4550 50  0000 C CNN
 F 1 "10k" H 3450 4650 50  0000 C CNN
 F 2 "~" H 3450 4650 60  0000 C CNN
@@
 AR Path="/5362BBC7/53598F21/53548633/53547B6E" Ref="RV47"  Part="1"
 AR Path="/5362BBC7/53598F21/53547A94/53547B6E" Ref="RV49"  Part="1"
-F 0 "RV49" H 2950 4550 50  0000 C CNN
+F 0 "RV16" H 2950 4550 50  0000 C CNN
 F 1 "100k" H 2950 4650 50  0000 C CNN
 F 2 "~" H 2950 4650 60  0000 C CNN
@@
 AR Path="/5362BBC7/53598F21/53548633/53547B7D" Ref="R174"  Part="1"
 AR Path="/5362BBC7/53598F21/53547A94/53547B7D" Ref="R178"  Part="1"
-F 0 "R178" V 3530 5250 40  0000 C CNN
+F 0 "R68" V 3530 5250 40  0000 C CNN
 F 1 "2k" V 3457 5251 40  0000 C CNN
 F 2 "~" V 3380 5250 30  0000 C CNN
@@
 AR Path="/5362BBC7/53598F21/53548633/53547B8C" Ref="R173"  Part="1"
 AR Path="/5362BBC7/53598F21/53547A94/53547B8C" Ref="R177"  Part="1"
-F 0 "R177" V 3530 4050 40  0000 C CNN
+F 0 "R67" V 3530 4050 40  0000 C CNN
 F 1 "2k" V 3457 4051 40  0000 C CNN
 F 2 "~" V 3380 4050 30  0000 C CNN
@@
 AR Path="/5362BBC7/53598F21/53548633/53547B9E" Ref="R171"  Part="1"
 AR Path="/5362BBC7/53598F21/53547A94/53547B9E" Ref="R175"  Part="1"
-F 0 "R175" V 3030 4050 40  0000 C CNN
+F 0 "R65" V 3030 4050 40  0000 C CNN
 F 1 "100k" V 2957 4051 40  0000 C CNN
 F 2 "~" V 2880 4050 30  0000 C CNN
@@
 AR Path="/5362BBC7/53598F21/53548633/53547BA4" Ref="R172"  Part="1"
 AR Path="/5362BBC7/53598F21/53547A94/53547BA4" Ref="R176"  Part="1"
-F 0 "R176" V 3030 5250 40  0000 C CNN
+F 0 "R66" V 3030 5250 40  0000 C CNN
 F 1 "100k" V 2957 5251 40  0000 C CNN
 F 2 "~" V 2880 5250 30  0000 C CNN
@@
 AR Path="/5362BBC7/53598F21/53548633/53553A48" Ref="C100"  Part="1"
 AR Path="/5362BBC7/53598F21/53547A94/53553A48" Ref="C101"  Part="1"
-F 0 "C101" H 3200 5050 40  0000 L CNN
+F 0 "C34" H 3200 5050 40  0000 L CNN
 F 1 "10u" H 3206 4865 40  0000 L CNN
 F 2 "~" H 3238 4800 30  0000 C CNN
@@
 $EndComp
 $Comp
-L GND #PWR22
+L GND #PWR022
 U 1 1 53553A57
 P 3200 5250
-AR Path="/5355B409/53598F1D/53548633/53553A57" Ref="#PWR22"  Part="1"
-AR Path="/5355B409/53598F1D/53547A94/53553A57" Ref="#PWR23"  Part="1"
-AR Path="/5355B409/531EB865/53548633/53553A57" Ref="#PWR28"  Part="1"
-AR Path="/5355B409/531EB865/53547A94/53553A57" Ref="#PWR29"  Part="1"
-AR Path="/53562461/5321AFC5/53548633/53553A57" Ref="#PWR48"  Part="1"
-AR Path="/53562461/5321AFC5/53547A94/53553A57" Ref="#PWR49"  Part="1"
-AR Path="/53562461/5321AFC7/53548633/53553A57" Ref="#PWR54"  Part="1"
-AR Path="/53562461/5321AFC7/53547A94/53553A57" Ref="#PWR55"  Part="1"
-AR Path="/5355C3A0/531E6F48/53548633/53553A57" Ref="#PWR80"  Part="1"
-AR Path="/5355C3A0/531E6F48/53547A94/53553A57" Ref="#PWR81"  Part="1"
-AR Path="/5355C3A0/53598F21/53548633/53553A57" Ref="#PWR86"  Part="1"
-AR Path="/5355C3A0/53598F21/53547A94/53553A57" Ref="#PWR87"  Part="1"
-AR Path="/5362BBC7/531E6F48/53548633/53553A57" Ref="#PWR119"  Part="1"
-AR Path="/5362BBC7/531E6F48/53547A94/53553A57" Ref="#PWR120"  Part="1"
-AR Path="/5362BBC7/53598F21/53548633/53553A57" Ref="#PWR125"  Part="1"
-AR Path="/5362BBC7/53598F21/53547A94/53553A57" Ref="#PWR126"  Part="1"
-F 0 "#PWR126" H 3200 5250 30  0001 C CNN
+AR Path="/5355B409/53598F1D/53548633/53553A57" Ref="#PWR022"  Part="1"
+AR Path="/5355B409/53598F1D/53547A94/53553A57" Ref="#PWR023"  Part="1"
+AR Path="/5355B409/531EB865/53548633/53553A57" Ref="#PWR028"  Part="1"
+AR Path="/5355B409/531EB865/53547A94/53553A57" Ref="#PWR029"  Part="1"
+AR Path="/53562461/5321AFC5/53548633/53553A57" Ref="#PWR048"  Part="1"
+AR Path="/53562461/5321AFC5/53547A94/53553A57" Ref="#PWR049"  Part="1"
+AR Path="/53562461/5321AFC7/53548633/53553A57" Ref="#PWR054"  Part="1"
+AR Path="/53562461/5321AFC7/53547A94/53553A57" Ref="#PWR055"  Part="1"
+AR Path="/5355C3A0/531E6F48/53548633/53553A57" Ref="#PWR080"  Part="1"
+AR Path="/5355C3A0/531E6F48/53547A94/53553A57" Ref="#PWR081"  Part="1"
+AR Path="/5355C3A0/53598F21/53548633/53553A57" Ref="#PWR086"  Part="1"
+AR Path="/5355C3A0/53598F21/53547A94/53553A57" Ref="#PWR087"  Part="1"
+AR Path="/5362BBC7/531E6F48/53548633/53553A57" Ref="#PWR0119"  Part="1"
+AR Path="/5362BBC7/531E6F48/53547A94/53553A57" Ref="#PWR0120"  Part="1"
+AR Path="/5362BBC7/53598F21/53548633/53553A57" Ref="#PWR0125"  Part="1"
+AR Path="/5362BBC7/53598F21/53547A94/53553A57" Ref="#PWR0126"  Part="1"
+F 0 "#PWR048" H 3200 5250 30  0001 C CNN
 F 1 "GND" H 3200 5180 30  0001 C CNN
 F 2 "" H 3200 5250 60  0000 C CNN
