File: pid/SMA.sch (KiCad schematic (older format))
At the start: 1 part, among them P3 SMA

Commit message: [pid] -
Parts:
- renumbered P3 to P2
Changed lines of the file:
@@
 $Descr A4 11693 8268
 encoding utf-8
-Sheet 22 47
+Sheet 22 53
 Title ""
-Date "1 may 2014"
+Date "2 may 2014"
 Rev ""
 Comp ""
@@
 $EndDescr
 $Comp
-L SMA P3
+L SMA P2
 U 1 1 5357E7C8
 P 3300 4400
-F 0 "P3" H 3300 4450 60  0000 C CNN
+AR Path="/5357E647/5357E7C8" Ref="P2"  Part="1"
+AR Path="/536425B8/5357E7C8" Ref="P3"  Part="1"
+AR Path="/5364286A/5357E7C8" Ref="P4"  Part="1"
+AR Path="/5364286D/5357E7C8" Ref="P5"  Part="1"
+AR Path="/53642A89/5357E7C8" Ref="P6"  Part="1"
+F 0 "P6" H 3300 4450 60  0000 C CNN
 F 1 "SMA" H 3300 4350 60  0000 C CNN
 F 2 "" H 3300 4400 60  0000 C CNN
@@
 $EndComp
 $Comp
-L GND #PWR060
+L GND #PWR065
 U 1 1 5357E7CE
 P 3050 4900
-F 0 "#PWR060" H 3050 4900 30  0001 C CNN
+AR Path="/5357E647/5357E7CE" Ref="#PWR065"  Part="1"
+AR Path="/536425B8/5357E7CE" Ref="#PWR0142"  Part="1"
+AR Path="/5364286A/5357E7CE" Ref="#PWR0143"  Part="1"
+AR Path="/5364286D/5357E7CE" Ref="#PWR0144"  Part="1"
+AR Path="/53642A89/5357E7CE" Ref="#PWR0145"  Part="1"
+F 0 "#PWR0145" H 3050 4900 30  0001 C CNN
 F 1 "GND" H 3050 4830 30  0001 C CNN
 F 2 "" H 3050 4900 60  0000 C CNN
