File: pid/ScaleError.sch (KiCad schematic (older format))
At the start: 15 parts, among them U18 LM7171, U19 LM7171

Commit message: [pid] -
Parts:
- removed R135: 1k, ~, symbol R
- added R138: 1k, ~, symbol R
- R141: renamed from R138; value 51 -> 100
- renumbered R136 to R139, R137 to R140, R139 to R142, R140 to R143
Connections:
- net In: now also R138.1
- net at RV41.1: now also R138.2
Changed lines of the file:
@@
 $Descr A4 11693 8268
 encoding utf-8
-Sheet 31 35
+Sheet 31 53
 Title ""
-Date "30 apr 2014"
+Date "2 may 2014"
 Rev ""
 Comp ""
@@
 $EndDescr
 $Comp
-L R R135
-U 1 1 53584771
+L R R138
+U 1 1 5364DD9C
 P 3450 3150
-F 0 "R135" V 3530 3150 40  0000 C CNN
+F 0 "R138" V 3530 3150 40  0000 C CNN
 F 1 "1k" V 3457 3151 40  0000 C CNN
 F 2 "~" V 3380 3150 30  0000 C CNN
@@
 $EndComp
 $Comp
-L GND #PWR082
-U 1 1 5358477D
+L GND #PWR087
+U 1 1 5364DD9D
 P 3450 4100
-F 0 "#PWR082" H 3450 4100 30  0001 C CNN
+F 0 "#PWR087" H 3450 4100 30  0001 C CNN
 F 1 "GND" H 3450 4030 30  0001 C CNN
 F 2 "" H 3450 4100 60  0000 C CNN
@@
 $Comp
 L LM7171 U18
-U 1 1 5358478D
+U 1 1 5364DD9E
 P 4100 3850
 F 0 "U18" H 4400 4050 60  0000 C CNN
@@
 	4200 4350 4100 4350
 $Comp
-L R R137
+L R R140
 U 1 1 535847B6
 P 4200 4550
-F 0 "R137" V 4280 4550 40  0000 C CNN
+F 0 "R140" V 4280 4550 40  0000 C CNN
 F 1 "510" V 4207 4551 40  0000 C CNN
 F 2 "~" V 4130 4550 30  0000 C CNN
@@
 $EndComp
 $Comp
-L R R136
+L R R139
 U 1 1 535847C5
 P 3700 4900
-F 0 "R136" V 3780 4900 40  0000 C CNN
+F 0 "R139" V 3780 4900 40  0000 C CNN
 F 1 "510" V 3707 4901 40  0000 C CNN
 F 2 "~" V 3630 4900 30  0000 C CNN
@@
 $EndComp
 $Comp
-L GND #PWR083
-U 1 1 535847E3
+L GND #PWR088
+U 1 1 5364DDA3
 P 3700 5250
-F 0 "#PWR083" H 3700 5250 30  0001 C CNN
+F 0 "#PWR088" H 3700 5250 30  0001 C CNN
 F 1 "GND" H 3700 5180 30  0001 C CNN
 F 2 "" H 3700 5250 60  0000 C CNN
@@
 $EndComp
 $Comp
-L GND #PWR084
+L GND #PWR089
 U 1 1 53584AA9
 P 2150 4100
-F 0 "#PWR084" H 2150 4100 30  0001 C CNN
+F 0 "#PWR089" H 2150 4100 30  0001 C CNN
 F 1 "GND" H 2150 4030 30  0001 C CNN
 F 2 "" H 2150 4100 60  0000 C CNN
@@
 $Comp
 L C C72
-U 1 1 53584CC6
+U 1 1 5364DDA4
 P 1600 3800
 F 0 "C72" H 1600 3900 40  0000 L CNN
@@
 $Comp
 L C C73
-U 1 1 53584CCC
+U 1 1 5364DDA6
 P 1600 4300
 F 0 "C73" H 1600 4400 40  0000 L CNN
@@
 $EndComp
 $Comp
-L GND #PWR085
-U 1 1 53584CD2
+L GND #PWR090
+U 1 1 5364DDA8
 P 1700 4100
-F 0 "#PWR085" H 1700 4100 30  0001 C CNN
+F 0 "#PWR090" H 1700 4100 30  0001 C CNN
 F 1 "GND" H 1700 4030 30  0001 C CNN
 F 2 "" H 1700 4100 60  0000 C CNN
@@
 	6150 3650 6050 3650
 $Comp
-L R R139
+L R R142
 U 1 1 53584D04
 P 6150 3850
-F 0 "R139" V 6230 3850 40  0000 C CNN
+F 0 "R142" V 6230 3850 40  0000 C CNN
 F 1 "510" V 6157 3851 40  0000 C CNN
 F 2 "~" V 6080 3850 30  0000 C CNN
@@
 $EndComp
 $Comp
-L R R138
+L R R141
 U 1 1 53584D0A
 P 5650 4200
-F 0 "R138" V 5730 4200 40  0000 C CNN
-F 1 "51" V 5657 4201 40  0000 C CNN
+F 0 "R141" V 5730 4200 40  0000 C CNN
+F 1 "100" V 5657 4201 40  0000 C CNN
 F 2 "~" V 5580 4200 30  0000 C CNN
 F 3 "~" H 5650 4200 30  0000 C CNN
@@
 $EndComp
 $Comp
-L GND #PWR086
+L GND #PWR091
 U 1 1 53584D16
 P 5650 4550
-F 0 "#PWR086" H 5650 4550 30  0001 C CNN
+F 0 "#PWR091" H 5650 4550 30  0001 C CNN
 F 1 "GND" H 5650 4480 30  0001 C CNN
 F 2 "" H 5650 4550 60  0000 C CNN
@@
 Connection ~ 3650 3750
 $Comp
-L R R140
+L R R143
 U 1 1 5358635A
 P 7100 3150
-F 0 "R140" V 7180 3150 40  0000 C CNN
+F 0 "R143" V 7180 3150 40  0000 C CNN
 F 1 "51" V 7107 3151 40  0000 C CNN
 F 2 "~" V 7030 3150 30  0000 C CNN
