File: pid/ScaleFeedForward.sch (KiCad schematic (older format))
At the start: 10 parts, among them U18 LM7171

Commit message: [pid] -
Parts:
- removed C73: 10u, ~, symbol C
- removed C76: 10p, ~, symbol C
- removed R136, R137: 510, ~, symbol R
- added C84: 10p, ~, symbol C
- added C86: 10u, ~, symbol C
- added R146, R149: 510, ~, symbol R
- gave numbers to parts that had none: 3
- renumbered C72 to C85, R135 to R147, U18 to U23
Connections:
- net -5V: now also C86.2
- net GND: now also C84.2, C86.1, R146.2
- net Out: now also R149.2
- net at U23.2 (-In): now also C84.1, R146.1, R149.1
Changed lines of the file:
@@
 $Descr A4 11693 8268
 encoding utf-8
-Sheet 37 47
+Sheet 35 53
 Title ""
-Date "1 may 2014"
+Date "2 may 2014"
 Rev ""
 Comp ""
@@
 $EndDescr
 $Comp
-L R R135
+L R R147
 U 1 1 53584771
 P 5650 2850
-AR Path="/535846D4/53584771" Ref="R135"  Part="1"
-AR Path="/536270FD/53584771" Ref="R135"  Part="1"
-F 0 "R135" V 5730 2850 40  0000 C CNN
+F 0 "R147" V 5730 2850 40  0000 C CNN
 F 1 "200k" V 5657 2851 40  0000 C CNN
 F 2 "~" V 5580 2850 30  0000 C CNN
@@
 $EndComp
 $Comp
-L GND #PWR082
+L GND #PWR098
 U 1 1 5358477D
 P 5650 3900
-AR Path="/535846D4/5358477D" Ref="#PWR082"  Part="1"
-AR Path="/536270FD/5358477D" Ref="#PWR082"  Part="1"
-F 0 "#PWR082" H 5650 3900 30  0001 C CNN
+F 0 "#PWR098" H 5650 3900 30  0001 C CNN
 F 1 "GND" H 5650 3830 30  0001 C CNN
 F 2 "" H 5650 3900 60  0000 C CNN
@@
 In1
 $Comp
-L LM7171 U18
+L LM7171 U23
 U 1 1 5358478D
 P 6000 4300
-AR Path="/535846D4/5358478D" Ref="U18"  Part="1"
-AR Path="/536270FD/5358478D" Ref="U18"  Part="1"
-F 0 "U18" H 6300 4500 60  0000 C CNN
+F 0 "U23" H 6300 4500 60  0000 C CNN
 F 1 "LM7171" H 6350 4050 60  0000 C CNN
 F 2 "~" H 6000 4300 60  0000 C CNN
@@
 	6100 4800 6000 4800
 $Comp
-L R R137
-U 1 1 535847B6
+L R R149
+U 1 1 5364DDA0
 P 6100 5000
-AR Path="/535846D4/535847B6" Ref="R137"  Part="1"
-AR Path="/536270FD/535847B6" Ref="R137"  Part="1"
-F 0 "R137" V 6180 5000 40  0000 C CNN
+F 0 "R149" V 6180 5000 40  0000 C CNN
 F 1 "510" V 6107 5001 40  0000 C CNN
 F 2 "~" V 6030 5000 30  0000 C CNN
@@
 $EndComp
 $Comp
-L R R136
-U 1 1 535847C5
+L R R146
+U 1 1 5364DDA1
 P 5600 5350
-AR Path="/535846D4/535847C5" Ref="R136"  Part="1"
-AR Path="/536270FD/535847C5" Ref="R136"  Part="1"
-F 0 "R136" V 5680 5350 40  0000 C CNN
+F 0 "R146" V 5680 5350 40  0000 C CNN
 F 1 "510" V 5607 5351 40  0000 C CNN
 F 2 "~" V 5530 5350 30  0000 C CNN
@@
 $EndComp
 $Comp
-L C C76
-U 1 1 535847D4
+L C C84
+U 1 1 5364DDA2
 P 5350 5350
-AR Path="/535846D4/535847D4" Ref="C76"  Part="1"
-AR Path="/536270FD/535847D4" Ref="C76"  Part="1"
-F 0 "C76" H 5350 5450 40  0000 L CNN
+F 0 "C84" H 5350 5450 40  0000 L CNN
 F 1 "10p" H 5356 5265 40  0000 L CNN
 F 2 "~" H 5388 5200 30  0000 C CNN
@@
 $EndComp
 $Comp
-L GND #PWR083
+L GND #PWR099
 U 1 1 535847E3
 P 5600 5700
-AR Path="/535846D4/535847E3" Ref="#PWR083"  Part="1"
-AR Path="/536270FD/535847E3" Ref="#PWR083"  Part="1"
-F 0 "#PWR083" H 5600 5700 30  0001 C CNN
+F 0 "#PWR099" H 5600 5700 30  0001 C CNN
 F 1 "GND" H 5600 5630 30  0001 C CNN
 F 2 "" H 5600 5700 60  0000 C CNN
@@
 -5V
 $Comp
-L C C72
+L C C85
 U 1 1 53584CC6
 P 6500 2800
-AR Path="/535846D4/53584CC6" Ref="C72"  Part="1"
-AR Path="/536270FD/53584CC6" Ref="C72"  Part="1"
-F 0 "C72" H 6500 2900 40  0000 L CNN
+F 0 "C85" H 6500 2900 40  0000 L CNN
 F 1 "10u" H 6506 2715 40  0000 L CNN
 F 2 "~" H 6538 2650 30  0000 C CNN
@@
 $EndComp
 $Comp
-L C C73
-U 1 1 53584CCC
+L C C86
+U 1 1 5364DDA7
 P 6500 3300
-AR Path="/535846D4/53584CCC" Ref="C73"  Part="1"
-AR Path="/536270FD/53584CCC" Ref="C73"  Part="1"
-F 0 "C73" H 6500 3400 40  0000 L CNN
+F 0 "C86" H 6500 3400 40  0000 L CNN
 F 1 "10u" H 6506 3215 40  0000 L CNN
 F 2 "~" H 6538 3150 30  0000 C CNN
@@
 $EndComp
 $Comp
-L GND #PWR085
-U 1 1 53584CD2
+L GND #PWR0100
+U 1 1 5364DDA9
 P 6600 3100
-AR Path="/535846D4/53584CD2" Ref="#PWR085"  Part="1"
-AR Path="/536270FD/53584CD2" Ref="#PWR085"  Part="1"
-F 0 "#PWR085" H 6600 3100 30  0001 C CNN
+F 0 "#PWR0100" H 6600 3100 30  0001 C CNN
 F 1 "GND" H 6600 3030 30  0001 C CNN
 F 2 "" H 6600 3100 60  0000 C CNN
@@
 	6500 3550 6550 3550
 $Comp
-L R R?
+L R R148
 U 1 1 5362768F
 P 5650 3550
-F 0 "R?" V 5730 3550 40  0000 C CNN
+F 0 "R148" V 5730 3550 40  0000 C CNN
 F 1 "5k" V 5657 3551 40  0000 C CNN
 F 2 "~" V 5580 3550 30  0000 C CNN
@@
 	5650 3800 5650 3900
 $Comp
-L R R?
+L R R144
 U 1 1 53627ACF
 P 5050 2850
-F 0 "R?" V 5130 2850 40  0000 C CNN
+F 0 "R144" V 5130 2850 40  0000 C CNN
 F 1 "200k" V 5057 2851 40  0000 C CNN
 F 2 "~" V 4980 2850 30  0000 C CNN
@@
 $EndComp
 $Comp
-L GND #PWR?
+L GND #PWR0101
 U 1 1 53627AD5
 P 5050 3900
-F 0 "#PWR?" H 5050 3900 30  0001 C CNN
+F 0 "#PWR0101" H 5050 3900 30  0001 C CNN
 F 1 "GND" H 5050 3830 30  0001 C CNN
 F 2 "" H 5050 3900 60  0000 C CNN
@@
 In2
 $Comp
-L R R?
+L R R145
 U 1 1 53627ADD
 P 5050 3550
-F 0 "R?" V 5130 3550 40  0000 C CNN
+F 0 "R145" V 5130 3550 40  0000 C CNN
 F 1 "5k" V 5057 3551 40  0000 C CNN
 F 2 "~" V 4980 3550 30  0000 C CNN
@@
 	5400 4100 5400 4200
 Wire Wire Line
-	5400 4200 5500 4200
+	5400 4200 5600 4200
 Wire Wire Line
 	5300 4100 5300 4200
 Wire Wire Line
 	5300 4200 5200 4200
-Wire Wire Line
-	5500 4200 5600 4200
 $Sheet
 S 5250 3500 200  600
