File: pid/Switch_NO.sch (KiCad schematic (older format))
At the start: 3 parts, among them U8 DG468

Commit message: [pid] -
Parts:
- renumbered C34 to C43, C35 to C44, U8 to U10
Changed lines of the file:
@@
 LIBS:rb-0524s
 LIBS:max44251
+LIBS:r_div
 LIBS:pid-cache
 EELAYER 27 0
@@
 $Descr A4 11693 8268
 encoding utf-8
-Sheet 17 27
+Sheet 17 47
 Title ""
-Date "22 apr 2014"
+Date "1 may 2014"
 Rev ""
 Comp ""
@@
 -15V
 $Comp
-L GND #PWR039
+L GND #PWR048
 U 1 1 531F2E67
 P 5700 4600
-AR Path="/531F388D/531F2E5F/531F2E67" Ref="#PWR039"  Part="1"
-AR Path="/531FB8C2/5321AFC9/531F2E67" Ref="#PWR060"  Part="1"
-F 0 "#PWR039" H 5700 4600 30  0001 C CNN
+AR Path="/53562461/5321AFC9/531F2E67" Ref="#PWR048"  Part="1"
+AR Path="/53562461/53581115/531F2E67" Ref="#PWR055"  Part="1"
+F 0 "#PWR055" H 5700 4600 30  0001 C CNN
 F 1 "GND" H 5700 4530 30  0001 C CNN
 F 2 "" H 5700 4600 60  0000 C CNN
@@
 -15V
 $Comp
-L C C34
+L C C43
 U 1 1 531F2E78
 P 4200 3750
-AR Path="/531F388D/531F2E5F/531F2E78" Ref="C34"  Part="1"
-AR Path="/531FB8C2/5321AFC9/531F2E78" Ref="C56"  Part="1"
-F 0 "C34" H 4200 3850 40  0000 L CNN
+AR Path="/53562461/5321AFC9/531F2E78" Ref="C43"  Part="1"
+AR Path="/53562461/53581115/531F2E78" Ref="C50"  Part="1"
+F 0 "C50" H 4200 3850 40  0000 L CNN
 F 1 "10u" H 4206 3665 40  0000 L CNN
 F 2 "~" H 4238 3600 30  0000 C CNN
@@
 $EndComp
 $Comp
-L C C35
+L C C44
 U 1 1 531F2E7E
 P 4200 4250
-AR Path="/531F388D/531F2E5F/531F2E7E" Ref="C35"  Part="1"
-AR Path="/531FB8C2/5321AFC9/531F2E7E" Ref="C57"  Part="1"
-F 0 "C35" H 4200 4350 40  0000 L CNN
+AR Path="/53562461/5321AFC9/531F2E7E" Ref="C44"  Part="1"
+AR Path="/53562461/53581115/531F2E7E" Ref="C51"  Part="1"
+F 0 "C51" H 4200 4350 40  0000 L CNN
 F 1 "10u" H 4206 4165 40  0000 L CNN
 F 2 "~" H 4238 4100 30  0000 C CNN
@@
 $EndComp
 $Comp
-L GND #PWR040
+L GND #PWR049
 U 1 1 531F2E84
 P 4300 4050
-AR Path="/531F388D/531F2E5F/531F2E84" Ref="#PWR040"  Part="1"
-AR Path="/531FB8C2/5321AFC9/531F2E84" Ref="#PWR061"  Part="1"
-F 0 "#PWR040" H 4300 4050 30  0001 C CNN
+AR Path="/53562461/5321AFC9/531F2E84" Ref="#PWR049"  Part="1"
+AR Path="/53562461/53581115/531F2E84" Ref="#PWR056"  Part="1"
+F 0 "#PWR056" H 4300 4050 30  0001 C CNN
 F 1 "GND" H 4300 3980 30  0001 C CNN
 F 2 "" H 4300 4050 60  0000 C CNN
@@
 	6300 3850 6350 3850
 $Comp
-L DG468 U8
+L DG468 U10
 U 1 1 531F2E9A
 P 5800 3950
-AR Path="/531F388D/531F2E5F/531F2E9A" Ref="U8"  Part="1"
-AR Path="/531FB8C2/5321AFC9/531F2E9A" Ref="U14"  Part="1"
-F 0 "U8" H 6000 4350 60  0000 C CNN
+AR Path="/53562461/5321AFC9/531F2E9A" Ref="U10"  Part="1"
+AR Path="/53562461/53581115/531F2E9A" Ref="U12"  Part="1"
+F 0 "U12" H 6000 4350 60  0000 C CNN
 F 1 "DG468" H 6100 3600 60  0000 C CNN
 F 2 "~" H 5800 3950 60  0000 C CNN

Commit message: [pid] -
Changed lines of the file:
@@
 $Descr A4 11693 8268
 encoding utf-8
-Sheet 17 47
+Sheet 17 53
 Title ""
-Date "1 may 2014"
+Date "2 may 2014"
 Rev ""
 Comp ""
@@
 -15V
 $Comp
-L GND #PWR048
+L GND #PWR053
 U 1 1 531F2E67
 P 5700 4600
-AR Path="/53562461/5321AFC9/531F2E67" Ref="#PWR048"  Part="1"
-AR Path="/53562461/53581115/531F2E67" Ref="#PWR055"  Part="1"
-F 0 "#PWR055" H 5700 4600 30  0001 C CNN
+AR Path="/53562461/5364DD9B/531F2E67" Ref="#PWR053"  Part="1"
+AR Path="/53562461/53581115/531F2E67" Ref="#PWR060"  Part="1"
+AR Path="/5321AFC9/531F2E67" Ref="#PWR0140"  Part="1"
+F 0 "#PWR0140" H 5700 4600 30  0001 C CNN
 F 1 "GND" H 5700 4530 30  0001 C CNN
 F 2 "" H 5700 4600 60  0000 C CNN
@@
 U 1 1 531F2E78
 P 4200 3750
-AR Path="/53562461/5321AFC9/531F2E78" Ref="C43"  Part="1"
+AR Path="/53562461/5364DD9B/531F2E78" Ref="C43"  Part="1"
 AR Path="/53562461/53581115/531F2E78" Ref="C50"  Part="1"
-F 0 "C50" H 4200 3850 40  0000 L CNN
+AR Path="/5321AFC9/531F2E78" Ref="C122"  Part="1"
+F 0 "C122" H 4200 3850 40  0000 L CNN
 F 1 "10u" H 4206 3665 40  0000 L CNN
 F 2 "~" H 4238 3600 30  0000 C CNN
@@
 U 1 1 531F2E7E
 P 4200 4250
-AR Path="/53562461/5321AFC9/531F2E7E" Ref="C44"  Part="1"
+AR Path="/53562461/5364DD9B/531F2E7E" Ref="C44"  Part="1"
 AR Path="/53562461/53581115/531F2E7E" Ref="C51"  Part="1"
-F 0 "C51" H 4200 4350 40  0000 L CNN
+AR Path="/5321AFC9/531F2E7E" Ref="C123"  Part="1"
+F 0 "C123" H 4200 4350 40  0000 L CNN
 F 1 "10u" H 4206 4165 40  0000 L CNN
 F 2 "~" H 4238 4100 30  0000 C CNN
@@
 $EndComp
 $Comp
-L GND #PWR049
+L GND #PWR054
 U 1 1 531F2E84
 P 4300 4050
-AR Path="/53562461/5321AFC9/531F2E84" Ref="#PWR049"  Part="1"
-AR Path="/53562461/53581115/531F2E84" Ref="#PWR056"  Part="1"
-F 0 "#PWR056" H 4300 4050 30  0001 C CNN
+AR Path="/53562461/5364DD9B/531F2E84" Ref="#PWR054"  Part="1"
+AR Path="/53562461/53581115/531F2E84" Ref="#PWR061"  Part="1"
+AR Path="/5321AFC9/531F2E84" Ref="#PWR0141"  Part="1"
+F 0 "#PWR0141" H 4300 4050 30  0001 C CNN
 F 1 "GND" H 4300 3980 30  0001 C CNN
 F 2 "" H 4300 4050 60  0000 C CNN
@@
 U 1 1 531F2E9A
 P 5800 3950
-AR Path="/53562461/5321AFC9/531F2E9A" Ref="U10"  Part="1"
+AR Path="/53562461/5364DD9B/531F2E9A" Ref="U10"  Part="1"
 AR Path="/53562461/53581115/531F2E9A" Ref="U12"  Part="1"
-F 0 "U12" H 6000 4350 60  0000 C CNN
+AR Path="/5321AFC9/531F2E9A" Ref="U34"  Part="1"
+F 0 "U34" H 6000 4350 60  0000 C CNN
 F 1 "DG468" H 6100 3600 60  0000 C CNN
 F 2 "~" H 5800 3950 60  0000 C CNN

Commit message: [pid] layout
Changed lines of the file:
@@
 $Descr A4 11693 8268
 encoding utf-8
-Sheet 49 53
+Sheet 20 53
 Title ""
-Date "2 may 2014"
+Date "5 may 2014"
 Rev ""
 Comp ""
@@
 -15V
 $Comp
-L GND #PWR59
+L GND #PWR058
 U 1 1 531F2E67
 P 5700 4600
-AR Path="/53562461/5364DD9B/531F2E67" Ref="#PWR59"  Part="1"
-AR Path="/53562461/53581115/531F2E67" Ref="#PWR67"  Part="1"
-AR Path="/5321AFC9/531F2E67" Ref="#PWR149"  Part="1"
-F 0 "#PWR149" H 5700 4600 30  0001 C CNN
+AR Path="/53562461/5364DD9B/531F2E67" Ref="#PWR058"  Part="1"
+AR Path="/53562461/53581115/531F2E67" Ref="#PWR066"  Part="1"
+AR Path="/5321AFC9/531F2E67" Ref="#PWR0148"  Part="1"
+F 0 "#PWR066" H 5700 4600 30  0001 C CNN
 F 1 "GND" H 5700 4530 30  0001 C CNN
 F 2 "" H 5700 4600 60  0000 C CNN
@@
 AR Path="/53562461/53581115/531F2E78" Ref="C50"  Part="1"
 AR Path="/5321AFC9/531F2E78" Ref="C122"  Part="1"
-F 0 "C122" H 4200 3850 40  0000 L CNN
+F 0 "C50" H 4200 3850 40  0000 L CNN
 F 1 "10u" H 4206 3665 40  0000 L CNN
 F 2 "~" H 4238 3600 30  0000 C CNN
@@
 AR Path="/53562461/53581115/531F2E7E" Ref="C51"  Part="1"
 AR Path="/5321AFC9/531F2E7E" Ref="C123"  Part="1"
-F 0 "C123" H 4200 4350 40  0000 L CNN
+F 0 "C51" H 4200 4350 40  0000 L CNN
 F 1 "10u" H 4206 4165 40  0000 L CNN
 F 2 "~" H 4238 4100 30  0000 C CNN
@@
 $EndComp
 $Comp
-L GND #PWR58
+L GND #PWR059
 U 1 1 531F2E84
 P 4300 4050
-AR Path="/53562461/5364DD9B/531F2E84" Ref="#PWR58"  Part="1"
-AR Path="/53562461/53581115/531F2E84" Ref="#PWR66"  Part="1"
-AR Path="/5321AFC9/531F2E84" Ref="#PWR148"  Part="1"
-F 0 "#PWR148" H 4300 4050 30  0001 C CNN
+AR Path="/53562461/5364DD9B/531F2E84" Ref="#PWR059"  Part="1"
+AR Path="/53562461/53581115/531F2E84" Ref="#PWR067"  Part="1"
+AR Path="/5321AFC9/531F2E84" Ref="#PWR0149"  Part="1"
+F 0 "#PWR067" H 4300 4050 30  0001 C CNN
 F 1 "GND" H 4300 3980 30  0001 C CNN
 F 2 "" H 4300 4050 60  0000 C CNN
@@
 AR Path="/53562461/53581115/531F2E9A" Ref="U12"  Part="1"
 AR Path="/5321AFC9/531F2E9A" Ref="U34"  Part="1"
-F 0 "U34" H 6000 4350 60  0000 C CNN
+F 0 "U12" H 6000 4350 60  0000 C CNN
 F 1 "DG468" H 6100 3600 60  0000 C CNN
 F 2 "~" H 5800 3950 60  0000 C CNN

Commit message: [pid] update
Changed lines of the file:
@@
 $Descr A4 11693 8268
 encoding utf-8
-Sheet 20 53
+Sheet 49 53
 Title ""
-Date "19 may 2014"
+Date "28 may 2014"
 Rev ""
 Comp ""
@@
 AR Path="/53562461/53581115/531F2E67" Ref="#PWR066"  Part="1"
 AR Path="/5321AFC9/531F2E67" Ref="#PWR0148"  Part="1"
-F 0 "#PWR066" H 5700 4600 30  0001 C CNN
+F 0 "#PWR0148" H 5700 4600 30  0001 C CNN
 F 1 "GND" H 5700 4530 30  0001 C CNN
 F 2 "" H 5700 4600 60  0000 C CNN
@@
 AR Path="/53562461/53581115/531F2E78" Ref="C50"  Part="1"
 AR Path="/5321AFC9/531F2E78" Ref="C122"  Part="1"
-F 0 "C50" H 4200 3850 40  0000 L CNN
+F 0 "C122" H 4200 3850 40  0000 L CNN
 F 1 "10u" H 4206 3665 40  0000 L CNN
 F 2 "~" H 4238 3600 30  0000 C CNN
@@
 AR Path="/53562461/53581115/531F2E7E" Ref="C51"  Part="1"
 AR Path="/5321AFC9/531F2E7E" Ref="C123"  Part="1"
-F 0 "C51" H 4200 4350 40  0000 L CNN
+F 0 "C123" H 4200 4350 40  0000 L CNN
 F 1 "10u" H 4206 4165 40  0000 L CNN
 F 2 "~" H 4238 4100 30  0000 C CNN
@@
 AR Path="/53562461/53581115/531F2E84" Ref="#PWR067"  Part="1"
 AR Path="/5321AFC9/531F2E84" Ref="#PWR0149"  Part="1"
-F 0 "#PWR067" H 4300 4050 30  0001 C CNN
+F 0 "#PWR0149" H 4300 4050 30  0001 C CNN
 F 1 "GND" H 4300 3980 30  0001 C CNN
 F 2 "" H 4300 4050 60  0000 C CNN
@@
 AR Path="/53562461/53581115/531F2E9A" Ref="U12"  Part="1"
 AR Path="/5321AFC9/531F2E9A" Ref="U34"  Part="1"
-F 0 "U12" H 6000 4350 60  0000 C CNN
+F 0 "U34" H 6000 4350 60  0000 C CNN
 F 1 "DG468" H 6100 3600 60  0000 C CNN
 F 2 "~" H 5800 3950 60  0000 C CNN
