File: pid/Switch_SPDT.sch (KiCad schematic (older format))
At the start: 3 parts, among them U9 DG467

Commit message: [pid] -
Parts:
- removed C41, C42: 10u, ~, symbol C
- removed U9: DG467, ~, symbol DG467
- added C78, C79: 10u, ~, symbol C
- added U20: DG469, ~, symbol DG469
Connections:
- net +15V: now also C78.1, U20.4 (V+)
- net -15V: now also C79.2, U20.7 (V-)
- net COM: now also U20.1 (COM)
- net GND: now also C78.2, C79.1, U20.3 (GND)
- net IN: now also U20.6 (IN)
- net NC: now also U20.2 (NC)
- new net NO: U20.8 (NO)
Changed lines of the file:
@@
 $Descr A4 11693 8268
 encoding utf-8
-Sheet 17 47
+Sheet 33 47
 Title ""
 Date "1 may 2014"
@@
 -15V
 $Comp
-L GND #PWR046
-U 1 1 53598F29
+L GND #PWR087
+U 1 1 531F2734
 P 4700 4550
-F 0 "#PWR046" H 4700 4550 30  0001 C CNN
+AR Path="/5358A076/531F2734" Ref="#PWR087"  Part="1"
+AR Path="/5358D04C/531F2734" Ref="#PWR089"  Part="1"
+AR Path="/5358D353/531F2734" Ref="#PWR091"  Part="1"
+F 0 "#PWR091" H 4700 4550 30  0001 C CNN
 F 1 "GND" H 4700 4480 30  0001 C CNN
 F 2 "" H 4700 4550 60  0000 C CNN
 F 3 "" H 4700 4550 60  0000 C CNN
 	1    4700 4550
-	1    0    0    -1
-$EndComp
-$Comp
-L DG467 U9
-U 1 1 531F273A
-P 4800 3900
-F 0 "U9" H 5000 4300 60  0000 C CNN
-F 1 "DG467" H 5100 3550 60  0000 C CNN
-F 2 "~" H 4800 3900 60  0000 C CNN
-F 3 "~" H 4800 3900 60  0000 C CNN
-	1    4800 3900
 	1    0    0    -1
 $EndComp
@@
 -15V
 $Comp
-L C C41
-U 1 1 531F2780
+L C C78
+U 1 1 53598F2A
 P 3200 3700
-F 0 "C41" H 3200 3800 40  0000 L CNN
+AR Path="/5358A076/53598F2A" Ref="C78"  Part="1"
+AR Path="/5358D04C/53598F2A" Ref="C80"  Part="1"
+AR Path="/5358D353/53598F2A" Ref="C82"  Part="1"
+F 0 "C82" H 3200 3800 40  0000 L CNN
 F 1 "10u" H 3206 3615 40  0000 L CNN
 F 2 "~" H 3238 3550 30  0000 C CNN
@@
 $EndComp
 $Comp
-L C C42
-U 1 1 53598F2B
+L C C79
+U 1 1 531F2786
 P 3200 4200
-F 0 "C42" H 3200 4300 40  0000 L CNN
+AR Path="/5358A076/531F2786" Ref="C79"  Part="1"
+AR Path="/5358D04C/531F2786" Ref="C81"  Part="1"
+AR Path="/5358D353/531F2786" Ref="C83"  Part="1"
+F 0 "C83" H 3200 4300 40  0000 L CNN
 F 1 "10u" H 3206 4115 40  0000 L CNN
 F 2 "~" H 3238 4050 30  0000 C CNN
@@
 $EndComp
 $Comp
-L GND #PWR047
-U 1 1 53598F2C
+L GND #PWR088
+U 1 1 531F278C
 P 3300 4000
-F 0 "#PWR047" H 3300 4000 30  0001 C CNN
+AR Path="/5358A076/531F278C" Ref="#PWR088"  Part="1"
+AR Path="/5358D04C/531F278C" Ref="#PWR090"  Part="1"
+AR Path="/5358D353/531F278C" Ref="#PWR092"  Part="1"
+F 0 "#PWR092" H 3300 4000 30  0001 C CNN
 F 1 "GND" H 3300 3930 30  0001 C CNN
 F 2 "" H 3300 4000 60  0000 C CNN
@@
 Wire Wire Line
 	3200 4450 3250 4450
-Text HLabel 4250 3800 0    60   Input ~ 0
+Text HLabel 4250 3900 0    60   Input ~ 0
 NC
 Text HLabel 4250 4100 0    60   Input ~ 0
@@
 COM
 Wire Wire Line
-	4250 3800 4300 3800
+	4250 3900 4300 3900
 Wire Wire Line
 	4300 4100 4250 4100
 Wire Wire Line
 	5300 3800 5350 3800
+$Comp
+L DG469 U20
+U 1 1 5358A139
+P 4800 3900
+AR Path="/5358A076/5358A139" Ref="U20"  Part="1"
+AR Path="/5358D04C/5358A139" Ref="U21"  Part="1"
+AR Path="/5358D353/5358A139" Ref="U22"  Part="1"
+F 0 "U22" H 5000 4300 60  0000 C CNN
+F 1 "DG469" H 5100 3550 60  0000 C CNN
+F 2 "~" H 4800 3900 60  0000 C CNN
+F 3 "~" H 4800 3900 60  0000 C CNN
+	1    4800 3900
+	1    0    0    -1
+$EndComp
+Text HLabel 4250 3700 0    60   Input ~ 0
+NO
+Wire Wire Line
+	4250 3700 4300 3700
 $EndSCHEMATC

Commit message: [pid] -
Changed lines of the file:
@@
 $Descr A4 11693 8268
 encoding utf-8
-Sheet 33 47
+Sheet 33 53
 Title ""
-Date "1 may 2014"
+Date "2 may 2014"
 Rev ""
 Comp ""
@@
 -15V
 $Comp
-L GND #PWR087
+L GND #PWR092
 U 1 1 531F2734
 P 4700 4550
-AR Path="/5358A076/531F2734" Ref="#PWR087"  Part="1"
-AR Path="/5358D04C/531F2734" Ref="#PWR089"  Part="1"
-AR Path="/5358D353/531F2734" Ref="#PWR091"  Part="1"
-F 0 "#PWR091" H 4700 4550 30  0001 C CNN
+AR Path="/5358D04C/531F2734" Ref="#PWR092"  Part="1"
+AR Path="/5358D353/531F2734" Ref="#PWR094"  Part="1"
+AR Path="/5358A076/531F2734" Ref="#PWR096"  Part="1"
+AR Path="/536270FD/5359A966/531F2734" Ref="#PWR0102"  Part="1"
+AR Path="/5362D599/531F2734" Ref="#PWR0125"  Part="1"
+AR Path="/536303B9/5364DDAA/531F2734" Ref="#PWR0136"  Part="1"
+AR Path="/536303B9/53635F8D/531F2734" Ref="#PWR0138"  Part="1"
+F 0 "#PWR092" H 4700 4550 30  0001 C CNN
 F 1 "GND" H 4700 4480 30  0001 C CNN
 F 2 "" H 4700 4550 60  0000 C CNN
@@
 U 1 1 53598F2A
 P 3200 3700
-AR Path="/5358A076/53598F2A" Ref="C78"  Part="1"
-AR Path="/5358D04C/53598F2A" Ref="C80"  Part="1"
-AR Path="/5358D353/53598F2A" Ref="C82"  Part="1"
-F 0 "C82" H 3200 3800 40  0000 L CNN
+AR Path="/5358D04C/53598F2A" Ref="C78"  Part="1"
+AR Path="/5358D353/53598F2A" Ref="C80"  Part="1"
+AR Path="/5358A076/53598F2A" Ref="C82"  Part="1"
+AR Path="/536270FD/5359A966/53598F2A" Ref="C87"  Part="1"
+AR Path="/5362D599/53598F2A" Ref="C107"  Part="1"
+AR Path="/536303B9/5364DDAA/53598F2A" Ref="C118"  Part="1"
+AR Path="/536303B9/53635F8D/53598F2A" Ref="C120"  Part="1"
+F 0 "C78" H 3200 3800 40  0000 L CNN
 F 1 "10u" H 3206 3615 40  0000 L CNN
 F 2 "~" H 3238 3550 30  0000 C CNN
@@
 U 1 1 531F2786
 P 3200 4200
-AR Path="/5358A076/531F2786" Ref="C79"  Part="1"
-AR Path="/5358D04C/531F2786" Ref="C81"  Part="1"
-AR Path="/5358D353/531F2786" Ref="C83"  Part="1"
-F 0 "C83" H 3200 4300 40  0000 L CNN
+AR Path="/5358D04C/531F2786" Ref="C79"  Part="1"
+AR Path="/5358D353/531F2786" Ref="C81"  Part="1"
+AR Path="/5358A076/531F2786" Ref="C83"  Part="1"
+AR Path="/536270FD/5359A966/531F2786" Ref="C88"  Part="1"
+AR Path="/5362D599/531F2786" Ref="C108"  Part="1"
+AR Path="/536303B9/5364DDAA/531F2786" Ref="C119"  Part="1"
+AR Path="/536303B9/53635F8D/531F2786" Ref="C121"  Part="1"
+F 0 "C79" H 3200 4300 40  0000 L CNN
 F 1 "10u" H 3206 4115 40  0000 L CNN
 F 2 "~" H 3238 4050 30  0000 C CNN
@@
 $EndComp
 $Comp
-L GND #PWR088
+L GND #PWR093
 U 1 1 531F278C
 P 3300 4000
-AR Path="/5358A076/531F278C" Ref="#PWR088"  Part="1"
-AR Path="/5358D04C/531F278C" Ref="#PWR090"  Part="1"
-AR Path="/5358D353/531F278C" Ref="#PWR092"  Part="1"
-F 0 "#PWR092" H 3300 4000 30  0001 C CNN
+AR Path="/5358D04C/531F278C" Ref="#PWR093"  Part="1"
+AR Path="/5358D353/531F278C" Ref="#PWR095"  Part="1"
+AR Path="/5358A076/531F278C" Ref="#PWR097"  Part="1"
+AR Path="/536270FD/5359A966/531F278C" Ref="#PWR0103"  Part="1"
+AR Path="/5362D599/531F278C" Ref="#PWR0126"  Part="1"
+AR Path="/536303B9/5364DDAA/531F278C" Ref="#PWR0137"  Part="1"
+AR Path="/536303B9/53635F8D/531F278C" Ref="#PWR0139"  Part="1"
+F 0 "#PWR093" H 3300 4000 30  0001 C CNN
 F 1 "GND" H 3300 3930 30  0001 C CNN
 F 2 "" H 3300 4000 60  0000 C CNN
@@
 U 1 1 5358A139
 P 4800 3900
-AR Path="/5358A076/5358A139" Ref="U20"  Part="1"
-AR Path="/5358D04C/5358A139" Ref="U21"  Part="1"
-AR Path="/5358D353/5358A139" Ref="U22"  Part="1"
-F 0 "U22" H 5000 4300 60  0000 C CNN
+AR Path="/5358D04C/5358A139" Ref="U20"  Part="1"
+AR Path="/5358D353/5358A139" Ref="U21"  Part="1"
+AR Path="/5358A076/5358A139" Ref="U22"  Part="1"
+AR Path="/536270FD/5359A966/5358A139" Ref="U24"  Part="1"
+AR Path="/5362D599/5358A139" Ref="U29"  Part="1"
+AR Path="/536303B9/5364DDAA/5358A139" Ref="U32"  Part="1"
+AR Path="/536303B9/53635F8D/5358A139" Ref="U33"  Part="1"
+F 0 "U20" H 5000 4300 60  0000 C CNN
 F 1 "DG469" H 5100 3550 60  0000 C CNN
 F 2 "~" H 4800 3900 60  0000 C CNN

Commit message: [pid] net list
Changed lines of the file:
@@
 -15V
 $Comp
-L GND #PWR092
+L GND #PWR096
 U 1 1 531F2734
 P 4700 4550
-AR Path="/5358D04C/531F2734" Ref="#PWR092"  Part="1"
-AR Path="/5358D353/531F2734" Ref="#PWR094"  Part="1"
-AR Path="/5358A076/531F2734" Ref="#PWR096"  Part="1"
-AR Path="/536270FD/5359A966/531F2734" Ref="#PWR0102"  Part="1"
-AR Path="/5362D599/531F2734" Ref="#PWR0125"  Part="1"
-AR Path="/536303B9/5364DDAA/531F2734" Ref="#PWR0136"  Part="1"
-AR Path="/536303B9/53635F8D/531F2734" Ref="#PWR0138"  Part="1"
-F 0 "#PWR092" H 4700 4550 30  0001 C CNN
+AR Path="/5358D04C/531F2734" Ref="#PWR096"  Part="1"
+AR Path="/5358D353/531F2734" Ref="#PWR098"  Part="1"
+AR Path="/5358A076/531F2734" Ref="#PWR0100"  Part="1"
+AR Path="/536270FD/5359A966/531F2734" Ref="#PWR0106"  Part="1"
+AR Path="/5362D599/531F2734" Ref="#PWR0129"  Part="1"
+AR Path="/536303B9/5364DDAA/531F2734" Ref="#PWR0140"  Part="1"
+AR Path="/536303B9/53635F8D/531F2734" Ref="#PWR0142"  Part="1"
+F 0 "#PWR0142" H 4700 4550 30  0001 C CNN
 F 1 "GND" H 4700 4480 30  0001 C CNN
 F 2 "" H 4700 4550 60  0000 C CNN
@@
 AR Path="/536303B9/5364DDAA/53598F2A" Ref="C118"  Part="1"
 AR Path="/536303B9/53635F8D/53598F2A" Ref="C120"  Part="1"
-F 0 "C78" H 3200 3800 40  0000 L CNN
+F 0 "C120" H 3200 3800 40  0000 L CNN
 F 1 "10u" H 3206 3615 40  0000 L CNN
 F 2 "~" H 3238 3550 30  0000 C CNN
@@
 AR Path="/536303B9/5364DDAA/531F2786" Ref="C119"  Part="1"
 AR Path="/536303B9/53635F8D/531F2786" Ref="C121"  Part="1"
-F 0 "C79" H 3200 4300 40  0000 L CNN
+F 0 "C121" H 3200 4300 40  0000 L CNN
 F 1 "10u" H 3206 4115 40  0000 L CNN
 F 2 "~" H 3238 4050 30  0000 C CNN
@@
 $EndComp
 $Comp
-L GND #PWR093
+L GND #PWR097
 U 1 1 531F278C
 P 3300 4000
-AR Path="/5358D04C/531F278C" Ref="#PWR093"  Part="1"
-AR Path="/5358D353/531F278C" Ref="#PWR095"  Part="1"
-AR Path="/5358A076/531F278C" Ref="#PWR097"  Part="1"
-AR Path="/536270FD/5359A966/531F278C" Ref="#PWR0103"  Part="1"
-AR Path="/5362D599/531F278C" Ref="#PWR0126"  Part="1"
-AR Path="/536303B9/5364DDAA/531F278C" Ref="#PWR0137"  Part="1"
-AR Path="/536303B9/53635F8D/531F278C" Ref="#PWR0139"  Part="1"
-F 0 "#PWR093" H 3300 4000 30  0001 C CNN
+AR Path="/5358D04C/531F278C" Ref="#PWR097"  Part="1"
+AR Path="/5358D353/531F278C" Ref="#PWR099"  Part="1"
+AR Path="/5358A076/531F278C" Ref="#PWR0101"  Part="1"
+AR Path="/536270FD/5359A966/531F278C" Ref="#PWR0107"  Part="1"
+AR Path="/5362D599/531F278C" Ref="#PWR0130"  Part="1"
+AR Path="/536303B9/5364DDAA/531F278C" Ref="#PWR0141"  Part="1"
+AR Path="/536303B9/53635F8D/531F278C" Ref="#PWR0143"  Part="1"
+F 0 "#PWR0143" H 3300 4000 30  0001 C CNN
 F 1 "GND" H 3300 3930 30  0001 C CNN
 F 2 "" H 3300 4000 60  0000 C CNN
@@
 AR Path="/536303B9/5364DDAA/5358A139" Ref="U32"  Part="1"
 AR Path="/536303B9/53635F8D/5358A139" Ref="U33"  Part="1"
-F 0 "U20" H 5000 4300 60  0000 C CNN
+F 0 "U33" H 5000 4300 60  0000 C CNN
 F 1 "DG469" H 5100 3550 60  0000 C CNN
 F 2 "~" H 4800 3900 60  0000 C CNN
