File: pid/VarAmp.sch (KiCad schematic (older format))
At the start: 9 parts, among them U2 LMH6505

Commit message: [pid] -
Parts:
- renumbered C7 to C6, C8 to C7, C9 to C8, R4 to R11, R6 to R12, R5 to R13, R7 to R14, R8 to R15

Commit message: [pid] -
Parts:
- renumbered R11 to R14, R12 to R15, R13 to R16, R14 to R17, R15 to R18

Commit message: [pid] layout
Changed lines of the file:
@@
 $Descr A4 11693 8268
 encoding utf-8
-Sheet 27 53
+Sheet 11 53
 Title ""
-Date "2 may 2014"
+Date "5 may 2014"
 Rev ""
 Comp ""
@@
 $EndDescr
 $Comp
-L GND #PWR18
+L GND #PWR018
 U 1 1 531E3EE5
 P 4050 4400
-AR Path="/5355B409/53598F1D/531E3EE5" Ref="#PWR18"  Part="1"
-AR Path="/5355B409/531EB865/531E3EE5" Ref="#PWR24"  Part="1"
-AR Path="/53562461/5321AFC5/531E3EE5" Ref="#PWR44"  Part="1"
-AR Path="/53562461/5321AFC7/531E3EE5" Ref="#PWR50"  Part="1"
-AR Path="/5355C3A0/531E6F48/531E3EE5" Ref="#PWR76"  Part="1"
-AR Path="/5355C3A0/53598F21/531E3EE5" Ref="#PWR82"  Part="1"
-AR Path="/5362BBC7/531E6F48/531E3EE5" Ref="#PWR115"  Part="1"
-AR Path="/5362BBC7/53598F21/531E3EE5" Ref="#PWR121"  Part="1"
-F 0 "#PWR121" H 4050 4400 30  0001 C CNN
+AR Path="/5355B409/53598F1D/531E3EE5" Ref="#PWR018"  Part="1"
+AR Path="/5355B409/531EB865/531E3EE5" Ref="#PWR024"  Part="1"
+AR Path="/53562461/5321AFC5/531E3EE5" Ref="#PWR044"  Part="1"
+AR Path="/53562461/5321AFC7/531E3EE5" Ref="#PWR050"  Part="1"
+AR Path="/5355C3A0/531E6F48/531E3EE5" Ref="#PWR076"  Part="1"
+AR Path="/5355C3A0/53598F21/531E3EE5" Ref="#PWR082"  Part="1"
+AR Path="/5362BBC7/531E6F48/531E3EE5" Ref="#PWR0115"  Part="1"
+AR Path="/5362BBC7/53598F21/531E3EE5" Ref="#PWR0121"  Part="1"
+F 0 "#PWR044" H 4050 4400 30  0001 C CNN
 F 1 "GND" H 4050 4330 30  0001 C CNN
 F 2 "" H 4050 4400 60  0000 C CNN
@@
 AR Path="/5362BBC7/531E6F48/531E3EEB" Ref="R153"  Part="1"
 AR Path="/5362BBC7/53598F21/531E3EEB" Ref="R166"  Part="1"
-F 0 "R166" V 3780 3700 40  0000 C CNN
+F 0 "R60" V 3780 3700 40  0000 C CNN
 F 1 "10k" V 3707 3701 40  0000 C CNN
 F 2 "~" V 3630 3700 30  0000 C CNN
@@
 AR Path="/5362BBC7/531E6F48/531E3EF1" Ref="R155"  Part="1"
 AR Path="/5362BBC7/53598F21/531E3EF1" Ref="R168"  Part="1"
-F 0 "R168" V 4130 4050 40  0000 C CNN
+F 0 "R62" V 4130 4050 40  0000 C CNN
 F 1 "100" V 4057 4051 40  0000 C CNN
 F 2 "~" V 3980 4050 30  0000 C CNN
@@
 AR Path="/5362BBC7/531E6F48/531E3EF7" Ref="U26"  Part="1"
 AR Path="/5362BBC7/53598F21/531E3EF7" Ref="U27"  Part="1"
-F 0 "U27" H 4800 3850 60  0000 C CNN
+F 0 "U7" H 4800 3850 60  0000 C CNN
 F 1 "LMH6505" H 4500 3600 60  0000 C CNN
 F 2 "~" H 4450 3600 60  0000 C CNN
@@
 $EndComp
 $Comp
-L GND #PWR20
+L GND #PWR019
 U 1 1 531E3EFE
 P 4450 4050
-AR Path="/5355B409/53598F1D/531E3EFE" Ref="#PWR20"  Part="1"
-AR Path="/5355B409/531EB865/531E3EFE" Ref="#PWR26"  Part="1"
-AR Path="/53562461/5321AFC5/531E3EFE" Ref="#PWR46"  Part="1"
-AR Path="/53562461/5321AFC7/531E3EFE" Ref="#PWR52"  Part="1"
-AR Path="/5355C3A0/531E6F48/531E3EFE" Ref="#PWR78"  Part="1"
-AR Path="/5355C3A0/53598F21/531E3EFE" Ref="#PWR84"  Part="1"
-AR Path="/5362BBC7/531E6F48/531E3EFE" Ref="#PWR117"  Part="1"
-AR Path="/5362BBC7/53598F21/531E3EFE" Ref="#PWR123"  Part="1"
-F 0 "#PWR123" H 4450 4050 30  0001 C CNN
+AR Path="/5355B409/53598F1D/531E3EFE" Ref="#PWR019"  Part="1"
+AR Path="/5355B409/531EB865/531E3EFE" Ref="#PWR025"  Part="1"
+AR Path="/53562461/5321AFC5/531E3EFE" Ref="#PWR045"  Part="1"
+AR Path="/53562461/5321AFC7/531E3EFE" Ref="#PWR051"  Part="1"
+AR Path="/5355C3A0/531E6F48/531E3EFE" Ref="#PWR077"  Part="1"
+AR Path="/5355C3A0/53598F21/531E3EFE" Ref="#PWR083"  Part="1"
+AR Path="/5362BBC7/531E6F48/531E3EFE" Ref="#PWR0116"  Part="1"
+AR Path="/5362BBC7/53598F21/531E3EFE" Ref="#PWR0122"  Part="1"
+F 0 "#PWR045" H 4450 4050 30  0001 C CNN
 F 1 "GND" H 4450 3980 30  0001 C CNN
 F 2 "" H 4450 4050 60  0000 C CNN
@@
 AR Path="/5362BBC7/531E6F48/531E3F04" Ref="R156"  Part="1"
 AR Path="/5362BBC7/53598F21/531E3F04" Ref="R169"  Part="1"
-F 0 "R169" V 5130 3300 40  0000 C CNN
+F 0 "R63" V 5130 3300 40  0000 C CNN
 F 1 "1k" V 5057 3301 40  0000 C CNN
 F 2 "~" V 4980 3300 30  0000 C CNN
@@
 AR Path="/5362BBC7/531E6F48/531E3F0A" Ref="R157"  Part="1"
 AR Path="/5362BBC7/53598F21/531E3F0A" Ref="R170"  Part="1"
-F 0 "R170" V 5480 2850 40  0000 C CNN
+F 0 "R64" V 5480 2850 40  0000 C CNN
 F 1 "10k" V 5407 2851 40  0000 C CNN
 F 2 "~" V 5330 2850 30  0000 C CNN
@@
 AR Path="/5362BBC7/531E6F48/531EE565" Ref="C93"  Part="1"
 AR Path="/5362BBC7/53598F21/531EE565" Ref="C98"  Part="1"
-F 0 "C98" H 5050 1700 40  0000 L CNN
+F 0 "C32" H 5050 1700 40  0000 L CNN
 F 1 "10u" H 5056 1515 40  0000 L CNN
 F 2 "~" H 5088 1450 30  0000 C CNN
@@
 AR Path="/5362BBC7/531E6F48/531EE56B" Ref="C94"  Part="1"
 AR Path="/5362BBC7/53598F21/531EE56B" Ref="C99"  Part="1"
-F 0 "C99" H 5050 2200 40  0000 L CNN
+F 0 "C33" H 5050 2200 40  0000 L CNN
 F 1 "10u" H 5056 2015 40  0000 L CNN
 F 2 "~" H 5088 1950 30  0000 C CNN
@@
 $EndComp
 $Comp
-L GND #PWR21
+L GND #PWR020
 U 1 1 531EE575
 P 5150 1900
-AR Path="/5355B409/53598F1D/531EE575" Ref="#PWR21"  Part="1"
-AR Path="/5355B409/531EB865/531EE575" Ref="#PWR27"  Part="1"
-AR Path="/53562461/5321AFC5/531EE575" Ref="#PWR47"  Part="1"
-AR Path="/53562461/5321AFC7/531EE575" Ref="#PWR53"  Part="1"
-AR Path="/5355C3A0/531E6F48/531EE575" Ref="#PWR79"  Part="1"
-AR Path="/5355C3A0/53598F21/531EE575" Ref="#PWR85"  Part="1"
-AR Path="/5362BBC7/531E6F48/531EE575" Ref="#PWR118"  Part="1"
-AR Path="/5362BBC7/53598F21/531EE575" Ref="#PWR124"  Part="1"
-F 0 "#PWR124" H 5150 1900 30  0001 C CNN
+AR Path="/5355B409/53598F1D/531EE575" Ref="#PWR020"  Part="1"
+AR Path="/5355B409/531EB865/531EE575" Ref="#PWR026"  Part="1"
+AR Path="/53562461/5321AFC5/531EE575" Ref="#PWR046"  Part="1"
+AR Path="/53562461/5321AFC7/531EE575" Ref="#PWR052"  Part="1"
+AR Path="/5355C3A0/531E6F48/531EE575" Ref="#PWR078"  Part="1"
+AR Path="/5355C3A0/53598F21/531EE575" Ref="#PWR084"  Part="1"
+AR Path="/5362BBC7/531E6F48/531EE575" Ref="#PWR0117"  Part="1"
+AR Path="/5362BBC7/53598F21/531EE575" Ref="#PWR0123"  Part="1"
+F 0 "#PWR046" H 5150 1900 30  0001 C CNN
 F 1 "GND" H 5150 1830 30  0001 C CNN
 F 2 "" H 5150 1900 60  0000 C CNN
@@
 AR Path="/5362BBC7/531E6F48/53215335" Ref="R154"  Part="1"
 AR Path="/5362BBC7/53598F21/53215335" Ref="R167"  Part="1"
-F 0 "R167" V 4030 2850 40  0000 C CNN
+F 0 "R61" V 4030 2850 40  0000 C CNN
 F 1 "5k" V 3957 2851 40  0000 C CNN
 F 2 "~" V 3880 2850 30  0000 C CNN
@@
 AR Path="/5362BBC7/531E6F48/5321533D" Ref="C92"  Part="1"
 AR Path="/5362BBC7/53598F21/5321533D" Ref="C97"  Part="1"
-F 0 "C97" H 4250 3200 40  0000 L CNN
+F 0 "C31" H 4250 3200 40  0000 L CNN
 F 1 "10u" H 4256 3015 40  0000 L CNN
 F 2 "~" H 4288 2950 30  0000 C CNN
@@
 $EndComp
 $Comp
-L GND #PWR19
+L GND #PWR021
 U 1 1 5321535B
 P 4250 3350
-AR Path="/5355B409/53598F1D/5321535B" Ref="#PWR19"  Part="1"
-AR Path="/5355B409/531EB865/5321535B" Ref="#PWR25"  Part="1"
-AR Path="/53562461/5321AFC5/5321535B" Ref="#PWR45"  Part="1"
-AR Path="/53562461/5321AFC7/5321535B" Ref="#PWR51"  Part="1"
-AR Path="/5355C3A0/531E6F48/5321535B" Ref="#PWR77"  Part="1"
-AR Path="/5355C3A0/53598F21/5321535B" Ref="#PWR83"  Part="1"
-AR Path="/5362BBC7/531E6F48/5321535B" Ref="#PWR116"  Part="1"
-AR Path="/5362BBC7/53598F21/5321535B" Ref="#PWR122"  Part="1"
-F 0 "#PWR122" H 4250 3350 30  0001 C CNN
+AR Path="/5355B409/53598F1D/5321535B" Ref="#PWR021"  Part="1"
+AR Path="/5355B409/531EB865/5321535B" Ref="#PWR027"  Part="1"
+AR Path="/53562461/5321AFC5/5321535B" Ref="#PWR047"  Part="1"
+AR Path="/53562461/5321AFC7/5321535B" Ref="#PWR053"  Part="1"
+AR Path="/5355C3A0/531E6F48/5321535B" Ref="#PWR079"  Part="1"
+AR Path="/5355C3A0/53598F21/5321535B" Ref="#PWR085"  Part="1"
+AR Path="/5362BBC7/531E6F48/5321535B" Ref="#PWR0118"  Part="1"
+AR Path="/5362BBC7/53598F21/5321535B" Ref="#PWR0124"  Part="1"
+F 0 "#PWR047" H 4250 3350 30  0001 C CNN
 F 1 "GND" H 4250 3280 30  0001 C CNN
 F 2 "" H 4250 3350 60  0000 C CNN

Commit message: [pid] update
Changed lines of the file:
@@
 Sheet 11 53
 Title ""
-Date "19 may 2014"
+Date "28 may 2014"
 Rev ""
 Comp ""
@@
 AR Path="/5362BBC7/531E6F48/531E3EE5" Ref="#PWR0115"  Part="1"
 AR Path="/5362BBC7/53598F21/531E3EE5" Ref="#PWR0121"  Part="1"
-F 0 "#PWR044" H 4050 4400 30  0001 C CNN
+F 0 "#PWR0121" H 4050 4400 30  0001 C CNN
 F 1 "GND" H 4050 4330 30  0001 C CNN
 F 2 "" H 4050 4400 60  0000 C CNN
@@
 AR Path="/5362BBC7/531E6F48/531E3EEB" Ref="R153"  Part="1"
 AR Path="/5362BBC7/53598F21/531E3EEB" Ref="R166"  Part="1"
-F 0 "R60" V 3780 3700 40  0000 C CNN
+F 0 "R166" V 3780 3700 40  0000 C CNN
 F 1 "10k" V 3707 3701 40  0000 C CNN
 F 2 "~" V 3630 3700 30  0000 C CNN
@@
 AR Path="/5362BBC7/531E6F48/531E3EF1" Ref="R155"  Part="1"
 AR Path="/5362BBC7/53598F21/531E3EF1" Ref="R168"  Part="1"
-F 0 "R62" V 4130 4050 40  0000 C CNN
+F 0 "R168" V 4130 4050 40  0000 C CNN
 F 1 "100" V 4057 4051 40  0000 C CNN
 F 2 "~" V 3980 4050 30  0000 C CNN
@@
 AR Path="/5362BBC7/531E6F48/531E3EF7" Ref="U26"  Part="1"
 AR Path="/5362BBC7/53598F21/531E3EF7" Ref="U27"  Part="1"
-F 0 "U7" H 4800 3850 60  0000 C CNN
+F 0 "U27" H 4800 3850 60  0000 C CNN
 F 1 "LMH6505" H 4500 3600 60  0000 C CNN
 F 2 "~" H 4450 3600 60  0000 C CNN
@@
 AR Path="/5362BBC7/531E6F48/531E3EFE" Ref="#PWR0116"  Part="1"
 AR Path="/5362BBC7/53598F21/531E3EFE" Ref="#PWR0122"  Part="1"
-F 0 "#PWR045" H 4450 4050 30  0001 C CNN
+F 0 "#PWR0122" H 4450 4050 30  0001 C CNN
 F 1 "GND" H 4450 3980 30  0001 C CNN
 F 2 "" H 4450 4050 60  0000 C CNN
@@
 AR Path="/5362BBC7/531E6F48/531E3F04" Ref="R156"  Part="1"
 AR Path="/5362BBC7/53598F21/531E3F04" Ref="R169"  Part="1"
-F 0 "R63" V 5130 3300 40  0000 C CNN
+F 0 "R169" V 5130 3300 40  0000 C CNN
 F 1 "1k" V 5057 3301 40  0000 C CNN
 F 2 "~" V 4980 3300 30  0000 C CNN
@@
 AR Path="/5362BBC7/531E6F48/531E3F0A" Ref="R157"  Part="1"
 AR Path="/5362BBC7/53598F21/531E3F0A" Ref="R170"  Part="1"
-F 0 "R64" V 5480 2850 40  0000 C CNN
+F 0 "R170" V 5480 2850 40  0000 C CNN
 F 1 "10k" V 5407 2851 40  0000 C CNN
 F 2 "~" V 5330 2850 30  0000 C CNN
@@
 AR Path="/5362BBC7/531E6F48/531EE565" Ref="C93"  Part="1"
 AR Path="/5362BBC7/53598F21/531EE565" Ref="C98"  Part="1"
-F 0 "C32" H 5050 1700 40  0000 L CNN
+F 0 "C98" H 5050 1700 40  0000 L CNN
 F 1 "10u" H 5056 1515 40  0000 L CNN
 F 2 "~" H 5088 1450 30  0000 C CNN
@@
 AR Path="/5362BBC7/531E6F48/531EE56B" Ref="C94"  Part="1"
 AR Path="/5362BBC7/53598F21/531EE56B" Ref="C99"  Part="1"
-F 0 "C33" H 5050 2200 40  0000 L CNN
+F 0 "C99" H 5050 2200 40  0000 L CNN
 F 1 "10u" H 5056 2015 40  0000 L CNN
 F 2 "~" H 5088 1950 30  0000 C CNN
@@
 AR Path="/5362BBC7/531E6F48/531EE575" Ref="#PWR0117"  Part="1"
 AR Path="/5362BBC7/53598F21/531EE575" Ref="#PWR0123"  Part="1"
-F 0 "#PWR046" H 5150 1900 30  0001 C CNN
+F 0 "#PWR0123" H 5150 1900 30  0001 C CNN
 F 1 "GND" H 5150 1830 30  0001 C CNN
 F 2 "" H 5150 1900 60  0000 C CNN
@@
 AR Path="/5362BBC7/531E6F48/53215335" Ref="R154"  Part="1"
 AR Path="/5362BBC7/53598F21/53215335" Ref="R167"  Part="1"
-F 0 "R61" V 4030 2850 40  0000 C CNN
+F 0 "R167" V 4030 2850 40  0000 C CNN
 F 1 "5k" V 3957 2851 40  0000 C CNN
 F 2 "~" V 3880 2850 30  0000 C CNN
@@
 AR Path="/5362BBC7/531E6F48/5321533D" Ref="C92"  Part="1"
 AR Path="/5362BBC7/53598F21/5321533D" Ref="C97"  Part="1"
-F 0 "C31" H 4250 3200 40  0000 L CNN
+F 0 "C97" H 4250 3200 40  0000 L CNN
 F 1 "10u" H 4256 3015 40  0000 L CNN
 F 2 "~" H 4288 2950 30  0000 C CNN
@@
 AR Path="/5362BBC7/531E6F48/5321535B" Ref="#PWR0118"  Part="1"
 AR Path="/5362BBC7/53598F21/5321535B" Ref="#PWR0124"  Part="1"
-F 0 "#PWR047" H 4250 3350 30  0001 C CNN
+F 0 "#PWR0124" H 4250 3350 30  0001 C CNN
 F 1 "GND" H 4250 3280 30  0001 C CNN
 F 2 "" H 4250 3350 60  0000 C CNN
