File: pid-tweak/GainCtrl.sch (KiCad schematic (older format))
At the start: 2 parts, among them K3 CONN_3, P7 CONN_2

Commit message: [pid-tweak] layout
Changed lines of the file:
@@
 Sheet 9 21
 Title ""
-Date "12 may 2014"
+Date "13 may 2014"
 Rev ""
 Comp ""
@@
 AR Path="/5370EBF3/536EEF0B" Ref="K8"  Part="1"
 AR Path="/5370EBF6/536EEF0B" Ref="K9"  Part="1"
-F 0 "K8" V 3900 2650 50  0000 C CNN
+F 0 "K9" V 3900 2650 50  0000 C CNN
 F 1 "CONN_3" V 4000 2650 40  0000 C CNN
 F 2 "~" H 3950 2650 60  0000 C CNN
@@
 AR Path="/5370EBF3/536EEF1A" Ref="P8"  Part="1"
 AR Path="/5370EBF6/536EEF1A" Ref="P9"  Part="1"
-F 0 "P8" V 3900 3100 40  0000 C CNN
+F 0 "P9" V 3900 3100 40  0000 C CNN
 F 1 "CONN_2" V 4000 3100 40  0000 C CNN
 F 2 "~" H 3950 3100 60  0000 C CNN
@@
 AR Path="/5370EBF3/536EEF3F" Ref="#PWR031"  Part="1"
 AR Path="/5370EBF6/536EEF3F" Ref="#PWR032"  Part="1"
-F 0 "#PWR031" H 4400 3250 30  0001 C CNN
+F 0 "#PWR032" H 4400 3250 30  0001 C CNN
 F 1 "GND" H 4400 3180 30  0001 C CNN
 F 2 "" H 4400 3250 60  0000 C CNN
