File: pid-tweak/LimitIn.sch (KiCad schematic (older format))
At the start: 6 parts, among them K2 CONN_3, K3 CONN_3, P4 CONN_2

Commit message: [pid-tweak] layout
Changed lines of the file:
@@
 $Descr A4 11693 8268
 encoding utf-8
-Sheet 6 21
+Sheet 7 21
 Title ""
-Date "12 may 2014"
+Date "13 may 2014"
 Rev ""
 Comp ""
@@
 AR Path="/5370F380/537150CF" Ref="K11"  Part="1"
 AR Path="/5370F3EE/537150CF" Ref="K13"  Part="1"
-F 0 "K4" V 3850 2800 50  0000 C CNN
+F 0 "K6" V 3850 2800 50  0000 C CNN
 F 1 "CONN_3" V 3950 2800 40  0000 C CNN
 F 2 "~" H 3900 2800 60  0000 C CNN
@@
 AR Path="/5370F380/5370DEDC" Ref="P10"  Part="1"
 AR Path="/5370F3EE/5370DEDC" Ref="P11"  Part="1"
-F 0 "P5" V 3000 3800 40  0000 C CNN
+F 0 "P6" V 3000 3800 40  0000 C CNN
 F 1 "CONN_2" V 3100 3800 40  0000 C CNN
 F 2 "~" H 3050 3800 60  0000 C CNN
@@
 AR Path="/5370F380/5370C167" Ref="K12"  Part="1"
 AR Path="/5370F3EE/5370C167" Ref="K14"  Part="1"
-F 0 "K5" V 3850 3350 50  0000 C CNN
+F 0 "K7" V 3850 3350 50  0000 C CNN
 F 1 "CONN_3" V 3950 3350 40  0000 C CNN
 F 2 "~" H 3900 3350 60  0000 C CNN
@@
 AR Path="/5370F380/5370DEDE" Ref="#PWR038"  Part="1"
 AR Path="/5370F3EE/5370DEDE" Ref="#PWR040"  Part="1"
-F 0 "#PWR026" H 3500 4000 30  0001 C CNN
+F 0 "#PWR028" H 3500 4000 30  0001 C CNN
 F 1 "GND" H 3500 3930 30  0001 C CNN
 F 2 "" H 3500 4000 60  0000 C CNN
@@
 AR Path="/5370F380/5370C195" Ref="R24"  Part="1"
 AR Path="/5370F3EE/5370C195" Ref="R26"  Part="1"
-F 0 "R17" V 4780 4050 40  0000 C CNN
+F 0 "R19" V 4780 4050 40  0000 C CNN
 F 1 "10k" V 4707 4051 40  0000 C CNN
 F 2 "~" V 4630 4050 30  0000 C CNN
@@
 AR Path="/5370F380/536EF582" Ref="R23"  Part="1"
 AR Path="/5370F3EE/536EF582" Ref="R25"  Part="1"
-F 0 "R16" V 3830 3700 40  0000 C CNN
+F 0 "R18" V 3830 3700 40  0000 C CNN
 F 1 "2k" V 3757 3701 40  0000 C CNN
 F 2 "~" V 3680 3700 30  0000 C CNN
@@
 AR Path="/5370F380/5370C1B3" Ref="RV8"  Part="1"
 AR Path="/5370F3EE/5370C1B3" Ref="RV9"  Part="1"
-F 0 "RV6" H 4350 3600 50  0000 C CNN
+F 0 "RV7" H 4350 3600 50  0000 C CNN
 F 1 "POT" H 4350 3700 50  0000 C CNN
 F 2 "~" H 4350 3700 60  0000 C CNN
@@
 AR Path="/5370F380/5370C24B" Ref="#PWR039"  Part="1"
 AR Path="/5370F3EE/5370C24B" Ref="#PWR041"  Part="1"
-F 0 "#PWR027" H 4700 4400 30  0001 C CNN
+F 0 "#PWR029" H 4700 4400 30  0001 C CNN
 F 1 "GND" H 4700 4330 30  0001 C CNN
 F 2 "" H 4700 4400 60  0000 C CNN
