File: pid-tweak/pid-tweak.sch (KiCad schematic (older format))
At the start: 38 parts, among them P1 CONN_13X2, P2 CONN_5X2, U1 TPS7A49, U2 TPS7A49, U3 TPS7A30, U4 TPS7A30

Commit message: [pid-tweak] layout
Parts:
- added P21, P22, P23, P24: CONN_1, ~, symbol CONN_1
Changed lines of the file:
@@
 Sheet 1 21
 Title "PID Controller"
-Date "12 may 2014"
+Date "13 may 2014"
 Rev "1"
 Comp "MIT BEC5"
@@
 Wire Wire Line
 	10150 4050 10250 4050
+$Comp
+L CONN_1 P21
+U 1 1 537189E9
+P 6050 4900
+F 0 "P21" H 6130 4900 40  0000 L CNN
+F 1 "CONN_1" H 6050 4955 30  0001 C CNN
+F 2 "~" H 6050 4900 60  0000 C CNN
+F 3 "~" H 6050 4900 60  0000 C CNN
+	1    6050 4900
+	1    0    0    -1
+$EndComp
+$Comp
+L CONN_1 P22
+U 1 1 53718AE6
+P 6050 5050
+F 0 "P22" H 6130 5050 40  0000 L CNN
+F 1 "CONN_1" H 6050 5105 30  0001 C CNN
+F 2 "~" H 6050 5050 60  0000 C CNN
+F 3 "~" H 6050 5050 60  0000 C CNN
+	1    6050 5050
+	1    0    0    -1
+$EndComp
+$Comp
+L CONN_1 P23
+U 1 1 53718AEC
+P 6050 5200
+F 0 "P23" H 6130 5200 40  0000 L CNN
+F 1 "CONN_1" H 6050 5255 30  0001 C CNN
+F 2 "~" H 6050 5200 60  0000 C CNN
+F 3 "~" H 6050 5200 60  0000 C CNN
+	1    6050 5200
+	1    0    0    -1
+$EndComp
+$Comp
+L CONN_1 P24
+U 1 1 53718AF2
+P 6050 5350
+F 0 "P24" H 6130 5350 40  0000 L CNN
+F 1 "CONN_1" H 6050 5405 30  0001 C CNN
+F 2 "~" H 6050 5350 60  0000 C CNN
+F 3 "~" H 6050 5350 60  0000 C CNN
+	1    6050 5350
+	1    0    0    -1
+$EndComp
 $EndSCHEMATC
